File: PEE50_MPPT/DC_DC.sch (KiCad schematic (older format))
At the start: 6 parts

Commit message: redelijk ver met de DC/DC schakeling overnemen
Parts:
- added C4, C5, C?: 100n, symbol Device:C
- added C?: 4u7, symbol Device:C
- added C? (x2): 10u, symbol Device:C
- added C? (x2): 39u, symbol Device:C
- added L1: 6u8, AudioProject:SER2915L-153KL, symbol pspice:INDUCTOR
- added R5, R7: 1, symbol Device:R
- added R6: 66.5k, symbol Device:R
- added R?: 21k, symbol Device:R
- added R?: 13k, symbol Device:R
- added R? (x2): 100k, symbol Device:R
- added U2: CSD18514Q5A, Robin_Lib:DQJ0008A, symbol Robin_lib:CSD18514Q5A
- added U3: CSD18543Q3A, Robin_Lib:DNH0008A, symbol Robin_lib:CSD18543Q3A
- U1: renamed from U?; footprint RPM0026A-MFG -> Robin_Lib:RPM0026A-MFG
- gave numbers to parts that had none: 5
Connections:
- net labels added: GND, ISN, ISP
- wire segments 18 -> 82

Commit message: microcontroller ingevoegd, current sense ingevoegd
Parts:
- gave numbers to parts that had none: 10
Changed lines of the file:
@@
 $Descr A4 11693 8268
 encoding utf-8
-Sheet 2 2
+Sheet 2 5
 Title ""
 Date ""
@@
 	4450 4050 4750 4050
 $Comp
-L Device:R R?
+L Device:R R12
 U 1 1 6089DC5E
 P 6900 4750
-F 0 "R?" H 6970 4796 50  0000 L CNN
+F 0 "R12" H 6970 4796 50  0000 L CNN
 F 1 "21k" H 6970 4705 50  0000 L CNN
 F 2 "" V 6830 4750 50  0001 C CNN
@@
 	6900 4550 6550 4550
 $Comp
-L power:GND #PWR?
+L power:GND #PWR0106
 U 1 1 6089E83E
 P 6900 4950
-F 0 "#PWR?" H 6900 4700 50  0001 C CNN
+F 0 "#PWR0106" H 6900 4700 50  0001 C CNN
 F 1 "GND" H 6905 4777 50  0000 C CNN
 F 2 "" H 6900 4950 50  0001 C CNN
@@
 	6900 4950 6900 4900
 $Comp
-L Device:C C?
+L Device:C C9
 U 1 1 6089F657
 P 7450 4500
-F 0 "C?" H 7565 4546 50  0000 L CNN
+F 0 "C9" H 7565 4546 50  0000 L CNN
 F 1 "100n" H 7565 4455 50  0000 L CNN
 F 2 "" H 7488 4350 50  0001 C CNN
@@
 $EndComp
 $Comp
-L Device:R R?
+L Device:R R13
 U 1 1 6089F6A9
 P 7450 4800
-F 0 "R?" H 7520 4846 50  0000 L CNN
+F 0 "R13" H 7520 4846 50  0000 L CNN
 F 1 "13k" H 7520 4755 50  0000 L CNN
 F 2 "" V 7380 4800 50  0001 C CNN
@@
 $EndComp
 $Comp
-L power:GND #PWR?
+L power:GND #PWR0107
 U 1 1 6089F6E5
 P 7450 5000
-F 0 "#PWR?" H 7450 4750 50  0001 C CNN
+F 0 "#PWR0107" H 7450 4750 50  0001 C CNN
 F 1 "GND" H 7455 4827 50  0000 C CNN
 F 2 "" H 7450 5000 50  0001 C CNN
@@
 Connection ~ 6550 4350
 $Comp
-L Device:C C?
+L Device:C C6
 U 1 1 608A52E7
 P 6850 4150
-F 0 "C?" H 6965 4196 50  0000 L CNN
+F 0 "C6" H 6965 4196 50  0000 L CNN
 F 1 "4u7" H 6965 4105 50  0000 L CNN
 F 2 "" H 6888 4000 50  0001 C CNN
@@
 	6550 4150 6700 4150
 $Comp
-L power:GND #PWR?
+L power:GND #PWR0108
 U 1 1 608A610D
 P 7100 4150
-F 0 "#PWR?" H 7100 3900 50  0001 C CNN
+F 0 "#PWR0108" H 7100 3900 50  0001 C CNN
 F 1 "GND" V 7105 4022 50  0000 R CNN
 F 2 "" H 7100 4150 50  0001 C CNN
@@
 	7000 4150 7100 4150
 $Comp
-L Device:C C?
+L Device:C C7
 U 1 1 608A80BD
 P 6900 3250
-F 0 "C?" H 7015 3296 50  0000 L CNN
+F 0 "C7" H 7015 3296 50  0000 L CNN
 F 1 "10u" H 7015 3205 50  0000 L CNN
 F 2 "" H 6938 3100 50  0001 C CNN
@@
 Connection ~ 6550 3050
 $Comp
-L power:GND #PWR?
+L power:GND #PWR0109
 U 1 1 608A9E4B
 P 6900 3450
-F 0 "#PWR?" H 6900 3200 50  0001 C CNN
+F 0 "#PWR0109" H 6900 3200 50  0001 C CNN
 F 1 "GND" H 6905 3277 50  0000 C CNN
 F 2 "" H 6900 3450 50  0001 C CNN
@@
 	6900 3400 6900 3450
 $Comp
-L Device:C C?
+L Device:C C8
 U 1 1 608AAE9E
 P 7250 3250
-F 0 "C?" H 7365 3296 50  0000 L CNN
+F 0 "C8" H 7365 3296 50  0000 L CNN
 F 1 "10u" H 7365 3205 50  0000 L CNN
 F 2 "" H 7288 3100 50  0001 C CNN
@@
 $EndComp
 $Comp
-L Device:C C?
+L Device:C C10
 U 1 1 608AAEE2
 P 7650 3250
-F 0 "C?" H 7765 3296 50  0000 L CNN
+F 0 "C10" H 7765 3296 50  0000 L CNN
 F 1 "39u" H 7765 3205 50  0000 L CNN
 F 2 "" H 7688 3100 50  0001 C CNN
@@
 $EndComp
 $Comp
-L Device:C C?
+L Device:C C11
 U 1 1 608AAF26
 P 8000 3250
-F 0 "C?" H 8115 3296 50  0000 L CNN
+F 0 "C11" H 8115 3296 50  0000 L CNN
 F 1 "39u" H 8115 3205 50  0000 L CNN
 F 2 "" H 8038 3100 50  0001 C CNN
@@
 	6550 3750 6600 3750
 $Comp
-L Device:R R?
+L Device:R R11
 U 1 1 608B2601
 P 4450 3800
-F 0 "R?" H 4520 3846 50  0000 L CNN
+F 0 "R11" H 4520 3846 50  0000 L CNN
 F 1 "100k" H 4520 3755 50  0000 L CNN
 F 2 "" V 4380 3800 50  0001 C CNN
@@
 $EndComp
 $Comp
-L Device:R R?
+L Device:R R10
 U 1 1 608B265F
 P 4200 3800
-F 0 "R?" H 4270 3846 50  0000 L CNN
+F 0 "R10" H 4270 3846 50  0000 L CNN
 F 1 "100k" H 4270 3755 50  0000 L CNN
 F 2 "" V 4130 3800 50  0001 C CNN
@@
 	4200 3450 4200 3650
 $Comp
-L power:GND #PWR?
+L power:GND #PWR0110
 U 1 1 608B53CB
 P 4200 4050
-F 0 "#PWR?" H 4200 3800 50  0001 C CNN
+F 0 "#PWR0110" H 4200 3800 50  0001 C CNN
 F 1 "GND" H 4205 3877 50  0000 C CNN
 F 2 "" H 4200 4050 50  0001 C CNN

Commit message: verschil gemaakt tussen Agnd en Pgnd
Connections:
- net labels added: Pgnd
- wire segments 82 -> 87
Changed lines of the file:
@@
 $EndComp
 Wire Wire Line
-	3550 3300 3050 3300
+	3550 3300 3350 3300
 Wire Wire Line
 	3050 3300 3050 2950
@@
 AR Path="/608C70E4/60894C33" Ref="#PWR0150"  Part="1"
 AR Path="/608DD92B/60894C33" Ref="#PWR0166"  Part="1"
-F 0 "#PWR0166" H 4850 1300 50  0001 C CNN
+F 0 "#PWR0103" H 4850 1300 50  0001 C CNN
 F 1 "GND" H 4855 1377 50  0000 C CNN
 F 2 "" H 4850 1550 50  0001 C CNN
@@
 	6900 2400 7400 2400
 Wire Wire Line
-	6550 3350 6550 3450
+	6550 3350 6550 3400
 $Comp
 L Device:R R6
@@
 AR Path="/608C70E4/6089AA95" Ref="#PWR0151"  Part="1"
 AR Path="/608DD92B/6089AA95" Ref="#PWR0167"  Part="1"
-F 0 "#PWR0167" H 4350 4650 50  0001 C CNN
+F 0 "#PWR0104" H 4350 4650 50  0001 C CNN
 F 1 "GND" H 4355 4727 50  0000 C CNN
 F 2 "" H 4350 4900 50  0001 C CNN
@@
 AR Path="/608C70E4/6089C9A3" Ref="#PWR0152"  Part="1"
 AR Path="/608DD92B/6089C9A3" Ref="#PWR0168"  Part="1"
-F 0 "#PWR0168" H 4450 3800 50  0001 C CNN
+F 0 "#PWR0105" H 4450 3800 50  0001 C CNN
 F 1 "GND" H 4455 3877 50  0000 C CNN
 F 2 "" H 4450 4050 50  0001 C CNN
@@
 AR Path="/608C70E4/6089E83E" Ref="#PWR0153"  Part="1"
 AR Path="/608DD92B/6089E83E" Ref="#PWR0169"  Part="1"
-F 0 "#PWR0169" H 6900 4700 50  0001 C CNN
+F 0 "#PWR0106" H 6900 4700 50  0001 C CNN
 F 1 "GND" H 6905 4777 50  0000 C CNN
 F 2 "" H 6900 4950 50  0001 C CNN
@@
 AR Path="/608C70E4/6089F6E5" Ref="#PWR0154"  Part="1"
 AR Path="/608DD92B/6089F6E5" Ref="#PWR0170"  Part="1"
-F 0 "#PWR0170" H 7450 4750 50  0001 C CNN
+F 0 "#PWR0107" H 7450 4750 50  0001 C CNN
 F 1 "GND" H 7455 4827 50  0000 C CNN
 F 2 "" H 7450 5000 50  0001 C CNN
@@
 AR Path="/608C70E4/608A610D" Ref="#PWR0155"  Part="1"
 AR Path="/608DD92B/608A610D" Ref="#PWR0171"  Part="1"
-F 0 "#PWR0171" H 7100 3900 50  0001 C CNN
+F 0 "#PWR0108" H 7100 3900 50  0001 C CNN
 F 1 "GND" V 7105 4022 50  0000 R CNN
 F 2 "" H 7100 4150 50  0001 C CNN
@@
 AR Path="/608C70E4/608A9E4B" Ref="#PWR0156"  Part="1"
 AR Path="/608DD92B/608A9E4B" Ref="#PWR0172"  Part="1"
-F 0 "#PWR0172" H 6900 3200 50  0001 C CNN
+F 0 "#PWR0109" H 6900 3200 50  0001 C CNN
 F 1 "GND" H 6905 3277 50  0000 C CNN
 F 2 "" H 6900 3450 50  0001 C CNN
@@
 AR Path="/608C70E4/608B53CB" Ref="#PWR0157"  Part="1"
 AR Path="/608DD92B/608B53CB" Ref="#PWR0173"  Part="1"
-F 0 "#PWR0173" H 4200 3800 50  0001 C CNN
+F 0 "#PWR0110" H 4200 3800 50  0001 C CNN
 F 1 "GND" H 4205 3877 50  0000 C CNN
 F 2 "" H 4200 4050 50  0001 C CNN
@@
 	4450 3950 4450 4050
 Connection ~ 4450 4050
+Wire Wire Line
+	6550 4950 6900 4950
+Connection ~ 6900 4950
+Text HLabel 6600 3400 2    50   BiDi ~ 0
+Pgnd
+Wire Wire Line
+	6600 3400 6550 3400
+Connection ~ 6550 3400
+Wire Wire Line
+	6550 3400 6550 3450
+$Comp
+L power:GND #PWR?
+U 1 1 60947EAA
+P 3350 3400
+AR Path="/6085EB29/60947EAA" Ref="#PWR?"  Part="1"
+AR Path="/608C3AEC/60947EAA" Ref="#PWR?"  Part="1"
+AR Path="/608C70E4/60947EAA" Ref="#PWR?"  Part="1"
+AR Path="/608DD92B/60947EAA" Ref="#PWR?"  Part="1"
+F 0 "#PWR?" H 3350 3150 50  0001 C CNN
+F 1 "GND" H 3355 3227 50  0000 C CNN
+F 2 "" H 3350 3400 50  0001 C CNN
+F 3 "" H 3350 3400 50  0001 C CNN
+	1    3350 3400
+	1    0    0    -1
+$EndComp
+Wire Wire Line
+	3350 3400 3350 3300
+Connection ~ 3350 3300
+Wire Wire Line
+	3350 3300 3050 3300
 $EndSCHEMATC

Commit message: toch maar wel Pgnd en Agnd verbonden met ontkoppel C
Connections:
- wire segments 87 -> 89
Changed lines of the file:
@@
 Wire Wire Line
 	3350 3300 3050 3300
+Wire Wire Line
+	6550 3350 6900 3350
+Wire Wire Line
+	6900 3350 6900 3400
+Connection ~ 6550 3350
+Connection ~ 6900 3400
 $EndSCHEMATC
