File: PEE50_MPPT/PEE50_MPPT.sch (KiCad schematic (older format))
At the start: 4 parts

Commit message: redelijk ver met de DC/DC schakeling overnemen
Parts:
- gave numbers to parts that had none: 4
Changed lines of the file:
@@
 $EndDescr
 $Comp
-L Connector:Conn_01x02_Female J?
+L Connector:Conn_01x02_Female J1
 U 1 1 6085EA1A
 P 1250 2000
-F 0 "J?" H 1144 1675 50  0000 C CNN
+F 0 "J1" H 1144 1675 50  0000 C CNN
 F 1 "PV_IN1" H 1144 1766 50  0000 C CNN
 F 2 "" H 1250 2000 50  0001 C CNN
@@
 	3050 1900 3350 1900
 $Comp
-L Device:R R?
+L Device:R R1
 U 1 1 6085EC5A
 P 3350 2100
-F 0 "R?" H 3420 2146 50  0000 L CNN
+F 0 "R1" H 3420 2146 50  0000 L CNN
 F 1 "R" H 3420 2055 50  0000 L CNN
 F 2 "" V 3280 2100 50  0001 C CNN
@@
 	3350 1950 3350 1900
 $Comp
-L Transistor_BJT:BC547 Q?
+L Transistor_BJT:BC547 Q1
 U 1 1 6085ED32
 P 3250 2750
-F 0 "Q?" H 3441 2796 50  0000 L CNN
+F 0 "Q1" H 3441 2796 50  0000 L CNN
 F 1 "BC547" H 3441 2705 50  0000 L CNN
 F 2 "Package_TO_SOT_THT:TO-92_Inline" H 3450 2675 50  0001 L CIN
@@
 	3350 2350 3350 2550
 $Comp
-L Device:R R?
+L Device:R R2
 U 1 1 6085EE2A
 P 3350 3150
-F 0 "R?" H 3420 3196 50  0000 L CNN
+F 0 "R2" H 3420 3196 50  0000 L CNN
 F 1 "R" H 3420 3105 50  0000 L CNN
 F 2 "" V 3280 3150 50  0001 C CNN
@@
 	3350 2950 3350 3000
 $Comp
-L power:GND #PWR?
+L power:GND #PWR0101
 U 1 1 6085EF47
 P 3350 3350
-F 0 "#PWR?" H 3350 3100 50  0001 C CNN
+F 0 "#PWR0101" H 3350 3100 50  0001 C CNN
 F 1 "GND" H 3355 3177 50  0000 C CNN
 F 2 "" H 3350 3350 50  0001 C CNN
@@
 	3350 3300 3350 3350
 $Comp
-L power:GND #PWR?
+L power:GND #PWR0102
 U 1 1 6085F011
 P 1750 2200
-F 0 "#PWR?" H 1750 1950 50  0001 C CNN
+F 0 "#PWR0102" H 1750 1950 50  0001 C CNN
 F 1 "GND" H 1755 2027 50  0000 C CNN
 F 2 "" H 1750 2200 50  0001 C CNN

Commit message: microcontroller ingevoegd, current sense ingevoegd
Parts:
- added J?: Conn_01x02_Female, symbol Connector:Conn_01x02_Female
- added R8, R9, R? (x2): R, symbol Device:R
Connections:
- wire segments 16 -> 33
Changed lines of the file:
@@
 $Descr A4 11693 8268
 encoding utf-8
-Sheet 1 2
+Sheet 1 5
 Title ""
 Date ""
@@
 L Connector:Conn_01x02_Female J1
 U 1 1 6085EA1A
-P 1250 2000
-F 0 "J1" H 1144 1675 50  0000 C CNN
-F 1 "PV_IN1" H 1144 1766 50  0000 C CNN
-F 2 "" H 1250 2000 50  0001 C CNN
-F 3 "~" H 1250 2000 50  0001 C CNN
-	1    1250 2000
+P 1150 2000
+F 0 "J1" H 1044 1675 50  0000 C CNN
+F 1 "PV_IN1" H 1044 1766 50  0000 C CNN
+F 2 "" H 1150 2000 50  0001 C CNN
+F 3 "~" H 1150 2000 50  0001 C CNN
+	1    1150 2000
 	-1   0    0    1
 $EndComp
 Wire Wire Line
-	1450 1900 1750 1900
-Wire Wire Line
 	1750 1900 1750 1750
 Wire Wire Line
 	1750 1750 1900 1750
 Wire Wire Line
-	1450 2000 1750 2000
-Wire Wire Line
 	1750 2000 1750 2150
-Wire Wire Line
-	3050 1900 3350 1900
 $Comp
 L Device:R R1
@@
 F5 "Vout" O R 3050 1900 50
 $EndSheet
+$Sheet
+S 1950 2700 950  600
+U 608BCBF7
+F0 "uC_MPPT" 50
+F1 "uC.sch" 50
+$EndSheet
+$Sheet
+S 1300 1050 400  500
+U 608BDD43
+F0 "current_Sense" 50
+F1 "current_sense.sch" 50
+F2 "R+" I B 1400 1550 50
+F3 "R-" I B 1600 1550 50
+F4 "out" O T 1500 1050 50
+$EndSheet
+$Comp
+L Device:R R8
+U 1 1 608BE8A7
+P 1600 1900
+F 0 "R8" V 1500 1850 50  0000 C CNN
+F 1 "R" V 1600 1900 50  0000 C CNN
+F 2 "" V 1530 1900 50  0001 C CNN
+F 3 "~" H 1600 1900 50  0001 C CNN
+	1    1600 1900
+	0    1    1    0
+$EndComp
+Wire Wire Line
+	1350 1900 1400 1900
+Wire Wire Line
+	1350 2000 1750 2000
+Wire Wire Line
+	1400 1900 1400 1550
+Connection ~ 1400 1900
+Wire Wire Line
+	1400 1900 1450 1900
+Wire Wire Line
+	1750 1750 1600 1750
+Wire Wire Line
+	1600 1750 1600 1550
+Connection ~ 1750 1750
+$Sheet
+S 3700 1150 400  500
+U 608BF482
+F0 "current_sense2" 50
+F1 "current_sense.sch" 50
+F2 "R+" I B 3800 1650 50
+F3 "R-" I B 4000 1650 50
+F4 "out" O T 3900 1150 50
+$EndSheet
+$Comp
+L Device:R R9
+U 1 1 608BF638
+P 3900 1900
+F 0 "R9" V 3800 1850 50  0000 C CNN
+F 1 "R" V 3900 1900 50  0000 C CNN
+F 2 "" V 3830 1900 50  0001 C CNN
+F 3 "~" H 3900 1900 50  0001 C CNN
+	1    3900 1900
+	0    1    1    0
+$EndComp
+Wire Wire Line
+	3750 1900 3750 1700
+Wire Wire Line
+	3750 1700 3800 1700
+Wire Wire Line
+	3800 1700 3800 1650
+Wire Wire Line
+	4050 1900 4050 1700
+Wire Wire Line
+	4050 1700 4000 1700
+Wire Wire Line
+	4000 1700 4000 1650
+Wire Wire Line
+	3050 1900 3350 1900
+Connection ~ 3750 1900
+Connection ~ 3350 1900
+Wire Wire Line
+	3350 1900 3750 1900
+Connection ~ 4050 1900
+$Comp
+L Connector:Conn_01x02_Female J?
+U 1 1 608C1F5B
+P 5050 1900
+F 0 "J?" H 5077 1876 50  0000 L CNN
+F 1 "Conn_01x02_Female" H 5077 1785 50  0000 L CNN
+F 2 "" H 5050 1900 50  0001 C CNN
+F 3 "~" H 5050 1900 50  0001 C CNN
+	1    5050 1900
+	1    0    0    -1
+$EndComp
+Wire Wire Line
+	4050 1900 4850 1900
+$Comp
+L power:GND #PWR?
+U 1 1 608C22E4
+P 4800 2050
+F 0 "#PWR?" H 4800 1800 50  0001 C CNN
+F 1 "GND" H 4805 1877 50  0000 C CNN
+F 2 "" H 4800 2050 50  0001 C CNN
+F 3 "" H 4800 2050 50  0001 C CNN
+	1    4800 2050
+	1    0    0    -1
+$EndComp
+Wire Wire Line
+	4800 2050 4800 2000
+Wire Wire Line
+	4800 2000 4850 2000
+$Comp
+L Device:R R?
+U 1 1 608C27BC
+P 1400 2200
+F 0 "R?" H 1470 2246 50  0000 L CNN
+F 1 "R" H 1470 2155 50  0000 L CNN
+F 2 "" V 1330 2200 50  0001 C CNN
+F 3 "~" H 1400 2200 50  0001 C CNN
+	1    1400 2200
+	1    0    0    -1
+$EndComp
+$Comp
+L Device:R R?
+U 1 1 608C27F8
+P 1400 2550
+F 0 "R?" H 1470 2596 50  0000 L CNN
+F 1 "R" H 1470 2505 50  0000 L CNN
+F 2 "" V 1330 2550 50  0001 C CNN
+F 3 "~" H 1400 2550 50  0001 C CNN
+	1    1400 2550
+	1    0    0    -1
+$EndComp
+$Comp
+L power:GND #PWR?
+U 1 1 608C2820
+P 1400 2750
+F 0 "#PWR?" H 1400 2500 50  0001 C CNN
+F 1 "GND" H 1405 2577 50  0000 C CNN
+F 2 "" H 1400 2750 50  0001 C CNN
+F 3 "" H 1400 2750 50  0001 C CNN
+	1    1400 2750
+	1    0    0    -1
+$EndComp
+Wire Wire Line
+	1400 2750 1400 2700
+Wire Wire Line
+	1400 2400 1400 2350
+Wire Wire Line
+	1400 2050 1400 1900
 $EndSCHEMATC

Commit message: copy + pasten van schakeling
Parts:
- added J? (x2): PV_IN2, symbol Connector:Conn_01x02_Female
- added Q? (x2): BC547, Package_TO_SOT_THT:TO-92_Inline, symbol Transistor_BJT:BC547
- added R? (x17): R, symbol Device:R
Connections:
- wire segments 33 -> 110

Commit message: mux ingevoegd en geintegreerd
Parts:
- added J?: PV_IN3, symbol Connector:Conn_01x02_Female
- added Q?: BC547, Package_TO_SOT_THT:TO-92_Inline, symbol Transistor_BJT:BC547
- added R? (x7): R, symbol Device:R
- J?: value PV_IN2 -> PV_IN4
Connections:
- net labels added: DAC1, DAC2, DAC3, DAC4, Vpv1, Vpv2, Vpv3, Vpv4
- wire segments 110 -> 155

Commit message: meetsignalen doorgevoerd naar mux
Connections:
- net labels added: Imppt1, Imppt2, Imppt3, Imppt4, Ipv1, Ipv2, Ipv3, Ipv4
- wire segments 155 -> 176
Changed lines of the file:
@@
 Wire Wire Line
 	4900 6100 4800 6100
+Wire Wire Line
+	800  2250 950  2250
+Connection ~ 950  2250
+Text GLabel 4200 6850 0    50   Input ~ 0
+Vpv1
+Wire Wire Line
+	4250 5350 4300 5350
+Text GLabel 1050 800  1    50   Input ~ 0
+Ipv1
+Wire Wire Line
+	1050 800  1050 900
+Text GLabel 1150 3900 1    50   Input ~ 0
+Ipv2
+Text GLabel 9050 3850 1    50   Input ~ 0
+Ipv3
+Text GLabel 9050 800  1    50   Input ~ 0
+Ipv4
+Wire Wire Line
+	1150 3900 1150 3950
+Wire Wire Line
+	9050 3850 9050 3950
+Wire Wire Line
+	9050 900  9050 800
+Text GLabel 4200 6400 0    50   Input ~ 0
+Ipv2
+Text GLabel 4200 6700 0    50   Input ~ 0
+Ipv1
+Wire Wire Line
+	4250 5450 4300 5450
+Text GLabel 4200 6550 0    50   Input ~ 0
+Vpv2
+Wire Wire Line
+	4250 5550 4300 5550
+Wire Wire Line
+	4250 5650 4300 5650
+Text GLabel 4200 6100 0    50   Input ~ 0
+Ipv3
+Text GLabel 4200 6250 0    50   Input ~ 0
+Vpv3
+Text GLabel 4200 5950 0    50   Input ~ 0
+Vpv4
+Text GLabel 4200 5800 0    50   Input ~ 0
+Ipv4
+Text GLabel 3450 900  1    50   Input ~ 0
+Imppt1
+Wire Wire Line
+	3450 900  3450 1000
+Text GLabel 3550 3950 1    50   Input ~ 0
+Imppt2
+Text GLabel 6650 4000 1    50   Input ~ 0
+Imppt3
+Text GLabel 6650 900  1    50   Input ~ 0
+Imppt4
+Wire Wire Line
+	6650 900  6650 1000
+Wire Wire Line
+	6650 4000 6650 4050
+Wire Wire Line
+	3550 3950 3550 4050
+Text GLabel 4250 5650 0    50   Input ~ 0
+Imppt1
+Text GLabel 4250 5450 0    50   Input ~ 0
+Imppt3
+Text GLabel 4250 5350 0    50   Input ~ 0
+Imppt4
+Text GLabel 4250 5550 0    50   Input ~ 0
+Imppt2
+Wire Wire Line
+	4200 6850 4300 6850
+Wire Wire Line
+	4200 6700 4300 6700
+Wire Wire Line
+	4200 6550 4300 6550
+Wire Wire Line
+	4200 6400 4300 6400
+Wire Wire Line
+	4200 6250 4300 6250
+Wire Wire Line
+	4200 6100 4300 6100
+Wire Wire Line
+	4200 5950 4300 5950
+Wire Wire Line
+	4200 5800 4300 5800
 $EndSCHEMATC

Commit message: laatste spanning bijgevoegd (was vergeten)
Connections:
- net labels added: Vout
- wire segments 176 -> 178
Changed lines of the file:
@@
 F17 "S12" I L 4300 5350 50
 F18 "out" O R 4800 6100 50
+F19 "S13" I R 4800 5400 50
 $EndSheet
 Wire Wire Line
@@
 Wire Wire Line
 	4200 5800 4300 5800
+Text GLabel 4250 3450 0    50   Input ~ 0
+Vout
+Wire Wire Line
+	4250 3450 4350 3450
+Connection ~ 4350 3450
+Text GLabel 4900 5400 2    50   Input ~ 0
+Vout
+Wire Wire Line
+	4900 5400 4800 5400
 $EndSCHEMATC

Commit message: verschil gemaakt tussen Agnd en Pgnd
Connections:
- net labels added: Pgnd
- wire segments 178 -> 198
Changed lines of the file:
@@
 F4 "FB" I R 2600 2050 50
 F5 "Vout" O R 2600 1750 50
+F6 "ISP" I R 2600 1950 50
+F7 "ISN" I R 2600 1850 50
+F8 "Pgnd" B R 2600 1500 50
 $EndSheet
 $Sheet
@@
 	1    0    0    -1
 $EndComp
-$Comp
-L power:GND #PWR0121
-U 1 1 608C22E4
-P 4600 3200
-F 0 "#PWR0121" H 4600 2950 50  0001 C CNN
-F 1 "GND" H 4605 3027 50  0000 C CNN
-F 2 "" H 4600 3200 50  0001 C CNN
-F 3 "" H 4600 3200 50  0001 C CNN
-	1    4600 3200
-	1    0    0    -1
-$EndComp
 Wire Wire Line
 	4600 3200 4600 3150
@@
 F4 "FB" I R 2700 5100 50
 F5 "Vout" O R 2700 4800 50
+F6 "ISP" I R 2700 4900 50
+F7 "ISN" I R 2700 5000 50
+F8 "Pgnd" B R 2700 4550 50
 $EndSheet
 $Sheet
@@
 F4 "FB" I L 7500 2050 50
 F5 "Vout" O L 7500 1750 50
+F6 "ISP" I L 7500 1850 50
+F7 "ISN" I L 7500 1950 50
+F8 "Pgnd" B L 7500 1600 50
 $EndSheet
 $Sheet
@@
 F4 "FB" I L 7500 5100 50
 F5 "Vout" O L 7500 4800 50
+F6 "ISP" I L 7500 4900 50
+F7 "ISN" I L 7500 5000 50
+F8 "Pgnd" B L 7500 4650 50
 $EndSheet
 $Sheet
@@
 Wire Wire Line
 	4900 5400 4800 5400
+Text GLabel 4600 3200 3    50   Input ~ 0
+Pgnd
+Wire Wire Line
+	2600 1850 3600 1850
+Wire Wire Line
+	3600 1850 3600 1750
+Wire Wire Line
+	2600 1950 3300 1950
+Wire Wire Line
+	3300 1950 3300 1750
+Wire Wire Line
+	2700 4900 3400 4900
+Wire Wire Line
+	3400 4900 3400 4800
+Wire Wire Line
+	2700 5000 3700 5000
+Wire Wire Line
+	3700 5000 3700 4800
+Text GLabel 2750 4550 2    50   Input ~ 0
+Pgnd
+Wire Wire Line
+	2750 4550 2700 4550
+Text GLabel 2650 1500 2    50   Input ~ 0
+Pgnd
+Wire Wire Line
+	2650 1500 2600 1500
+Wire Wire Line
+	7500 1850 6800 1850
+Wire Wire Line
+	6800 1850 6800 1750
+Wire Wire Line
+	7500 1950 6500 1950
+Wire Wire Line
+	6500 1950 6500 1750
+Text GLabel 7400 1600 0    50   Input ~ 0
+Pgnd
+Wire Wire Line
+	7400 1600 7500 1600
+Wire Wire Line
+	7500 4900 6800 4900
+Wire Wire Line
+	6800 4900 6800 4800
+Wire Wire Line
+	7500 5000 6500 5000
+Wire Wire Line
+	6500 5000 6500 4800
+Text GLabel 7450 4650 0    50   Input ~ 0
+Pgnd
+Wire Wire Line
+	7450 4650 7500 4650
 $EndSCHEMATC

Commit message: schakeling klaar (denk ik)
Parts:
- added C1, C?: 1u, symbol Device:C
- added C2, C?: 100n, symbol Device:C
- added J3: Conn_01x02_Female, symbol Connector:Conn_01x02_Female
- added JP1: Jumper_NC_Dual, symbol Device:Jumper_NC_Dual
- added U1: LM3480-3.3, Package_TO_SOT_SMD:SOT-23, symbol Regulator_Linear:LM3480-3.3
- gave numbers to parts that had none: 33
- renumbered R2 to R10, R9 to R13, R8 to R5, R1 to R9
Connections:
- net labels added: +12V, +3.3V
- wire segments 198 -> 219
