File: PEE50_MPPT/current_sense8.sch (KiCad schematic (older format))
At the start: 2 parts, among them U21 MAX44284FAUT+T

Commit message: best veel footprints ingevoegd
Parts:
- C54: footprint (none) -> Capacitor_SMD:C_1206_3216Metric_Pad1.42x1.75mm_HandSolder
Changed lines of the file:
@@
 EESchema Schematic File Version 4
-LIBS:PEE50_MPPT-cache
-EELAYER 26 0
+EELAYER 30 0
 EELAYER END
 $Descr A4 11693 8268
 encoding utf-8
-Sheet 4 15
+Sheet 13 15
 Title ""
 Date ""
@@
 F 0 "C54" V 4098 3100 50  0000 C CNN
 F 1 "100n" V 4189 3100 50  0000 C CNN
-F 2 "" H 4388 2950 50  0001 C CNN
+F 2 "Capacitor_SMD:C_1206_3216Metric_Pad1.42x1.75mm_HandSolder" H 4388 2950 50  0001 C CNN
 F 3 "~" H 4350 3100 50  0001 C CNN
 	1    4350 3100

Commit message: footprints gemapt + 10x10 pcb rand getekend
Parts:
- U21: footprint 21-0058I_MXM -> AudioProject:MAX44284FAUT&plus_T
Changed lines of the file:
@@
 EESchema Schematic File Version 4
-EELAYER 30 0
+LIBS:PEE50_MPPT-cache
+EELAYER 26 0
 EELAYER END
 $Descr A4 11693 8268
@@
 F 0 "U21" H 5500 3487 60  0000 C CNN
 F 1 "MAX44284FAUT+T" H 5500 3381 60  0000 C CNN
-F 2 "21-0058I_MXM" H 5500 3340 60  0001 C CNN
+F 2 "AudioProject:MAX44284FAUT&plus_T" H 5500 3340 60  0001 C CNN
 F 3 "" H 4700 3100 60  0000 C CNN
 	1    4700 3100
