File: PEE50_MPPT/DC_DC0.sch (KiCad schematic (older format))
At the start: 24 parts, among them U1 TPS552882QRPMRQ1, U2 CSD18514Q5A, U3 CSD18543Q3A

Commit message: schakeling klaar (denk ik)
Parts:
- removed C1, C2: 150u, symbol Device:C
- removed C7: 10u, symbol Device:C
- removed R10, R11, R4: 100k, symbol Device:R
- removed R13: 13k, symbol Device:R
- removed R3: 383k, symbol Device:R
- removed R5, R7: 1, symbol Device:R
- removed R6: 66.5k, symbol Device:R
- removed U1: TPS552882QRPMRQ1, Robin_Lib:RPM0026A-MFG, symbol Robin_lib:TPS552882QRPMRQ1
- added C12, C13: 39u, symbol Device:C
- added C6: 100n, symbol Device:C
- added R31: 383k, symbol Device:R
- added R32, R34, R36: 100k, symbol Device:R
- added R33, R37: 1, symbol Device:R
- added R35: 66.5k, symbol Device:R
- added R39: 13k, symbol Device:R
- added U4: TPS552882QRPMRQ1, Robin_Lib:RPM0026A-MFG, symbol Robin_lib:TPS552882QRPMRQ1
- C10: value 39u -> 10u
- C11: value 39u -> 100n
- C3: value 10u -> 150u
- C4: value 100n -> 150u
- C5, C9: value 100n -> 10u
- C8: value 10u -> 100n
- renumbered C6 to C7, R12 to R38
Connections:
- net FB: now also U4.14 (FB)
- net GND: now also C4.2, C5.2, C9.2, C12.2, C13.2, R32.2, R34.2, R35.2, R36.2, R39.2, U4.10 (AGND), U4.15 (MODE), U4.24 (PGND), U4.7 (DITH_SYNC), U4.9 (PGND); no longer C11.2, C8.2
- net ISN: now also U4.13 (ISN)
- net ISP: now also U4.12 (ISP)
- net PVin+: now also C4.1, C5.1, R31.1, U4.3 (VIN)
- net Vout: now also C9.1, C12.1, C13.1, U4.11 (VOUT), U4.26 (VOUT); no longer C11.1, C8.1
- net at R38.1: now also U4.17 (ILIM)
- net at C7.1: now also U4.19 (VCC)
- net at L1.2: now also C8.2, U4.21 (SW2), U4.25 (SW2); no longer C5.2
- net at L1.1, U2.1 (S), U2.2 (S)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: now also C6.1, U4.23 (SW1); no longer C4.1
- net at U2.4 (G): now also R33.1
- net at U3.4 (G): now also R37.1
- new net: R37.2, U4.1 (DR1L)
- new net: C11.2, U4.18 (COMP)
- new net: R33.2, U4.2 (DR1H)
- new net: C8.1, U4.20 (BOOT2)
- new net: C6.2, U4.22 (BOOT1)
- new net: R31.2, R32.1, U4.4 (EN)
- new net: R34.1, U4.5 (PG)
- new net: R36.1, U4.6 (CC_N)
- new net: R35.1, U4.8 (FSW)
- new net: C11.1, R39.1

Commit message: best veel footprints ingevoegd
Parts:
- C10, C11, C12, C13, C3, C4, C5, C6, C7, C8, C9: footprint (none) -> Capacitor_SMD:C_1206_3216Metric_Pad1.42x1.75mm_HandSolder
- R31, R32, R33, R34, R35, R36, R37, R38, R39: footprint (none) -> Resistor_SMD:R_1206_3216Metric_Pad1.42x1.75mm_HandSolder
Changed lines of the file:
@@
 EESchema Schematic File Version 4
-LIBS:PEE50_MPPT-cache
-EELAYER 26 0
+EELAYER 30 0
 EELAYER END
 $Descr A4 11693 8268
@@
 F 0 "C3" H 2365 2846 50  0000 L CNN
 F 1 "150u" H 2365 2755 50  0000 L CNN
-F 2 "" H 2288 2650 50  0001 C CNN
+F 2 "Capacitor_SMD:C_1206_3216Metric_Pad1.42x1.75mm_HandSolder" H 2288 2650 50  0001 C CNN
 F 3 "~" H 2250 2800 50  0001 C CNN
 	1    2250 2800
@@
 F 0 "C5" H 3165 2846 50  0000 L CNN
 F 1 "10u" H 3165 2755 50  0000 L CNN
-F 2 "" H 3088 2650 50  0001 C CNN
+F 2 "Capacitor_SMD:C_1206_3216Metric_Pad1.42x1.75mm_HandSolder" H 3088 2650 50  0001 C CNN
 F 3 "~" H 3050 2800 50  0001 C CNN
 	1    3050 2800
@@
 F 0 "C4" H 2765 2846 50  0000 L CNN
 F 1 "150u" H 2765 2755 50  0000 L CNN
-F 2 "" H 2688 2650 50  0001 C CNN
+F 2 "Capacitor_SMD:C_1206_3216Metric_Pad1.42x1.75mm_HandSolder" H 2688 2650 50  0001 C CNN
 F 3 "~" H 2650 2800 50  0001 C CNN
 	1    2650 2800
@@
 F 0 "R31" H 3620 2846 50  0000 L CNN
 F 1 "383k" H 3620 2755 50  0000 L CNN
-F 2 "" V 3480 2800 50  0001 C CNN
+F 2 "Resistor_SMD:R_1206_3216Metric_Pad1.42x1.75mm_HandSolder" V 3480 2800 50  0001 C CNN
 F 3 "~" H 3550 2800 50  0001 C CNN
 	1    3550 2800
@@
 F 0 "R32" H 3620 3196 50  0000 L CNN
 F 1 "100k" H 3620 3105 50  0000 L CNN
-F 2 "" V 3480 3150 50  0001 C CNN
+F 2 "Resistor_SMD:R_1206_3216Metric_Pad1.42x1.75mm_HandSolder" V 3480 3150 50  0001 C CNN
 F 3 "~" H 3550 3150 50  0001 C CNN
 	1    3550 3150
@@
 F 0 "R33" H 3820 1846 50  0000 L CNN
 F 1 "1" H 3820 1755 50  0000 L CNN
-F 2 "" V 3680 1800 50  0001 C CNN
+F 2 "Resistor_SMD:R_1206_3216Metric_Pad1.42x1.75mm_HandSolder" V 3680 1800 50  0001 C CNN
 F 3 "~" H 3750 1800 50  0001 C CNN
 	1    3750 1800
@@
 F 0 "R37" H 4570 1546 50  0000 L CNN
 F 1 "1" H 4570 1455 50  0000 L CNN
-F 2 "" V 4430 1500 50  0001 C CNN
+F 2 "Resistor_SMD:R_1206_3216Metric_Pad1.42x1.75mm_HandSolder" V 4430 1500 50  0001 C CNN
 F 3 "~" H 4500 1500 50  0001 C CNN
 	1    4500 1500
@@
 F 0 "C6" H 6715 1346 50  0000 L CNN
 F 1 "100n" H 6715 1255 50  0000 L CNN
-F 2 "" H 6638 1150 50  0001 C CNN
+F 2 "Capacitor_SMD:C_1206_3216Metric_Pad1.42x1.75mm_HandSolder" H 6638 1150 50  0001 C CNN
 F 3 "~" H 6600 1300 50  0001 C CNN
 	1    6600 1300
@@
 F 0 "C8" H 7015 2646 50  0000 L CNN
 F 1 "100n" H 7015 2555 50  0000 L CNN
-F 2 "" H 6938 2450 50  0001 C CNN
+F 2 "Capacitor_SMD:C_1206_3216Metric_Pad1.42x1.75mm_HandSolder" H 6938 2450 50  0001 C CNN
 F 3 "~" H 6900 2600 50  0001 C CNN
 	1    6900 2600
@@
 F 0 "R35" H 4270 4546 50  0000 L CNN
 F 1 "66.5k" H 4270 4455 50  0000 L CNN
-F 2 "" V 4130 4500 50  0001 C CNN
+F 2 "Resistor_SMD:R_1206_3216Metric_Pad1.42x1.75mm_HandSolder" V 4130 4500 50  0001 C CNN
 F 3 "~" H 4200 4500 50  0001 C CNN
 	1    4200 4500
@@
 F 0 "R38" H 6970 4796 50  0000 L CNN
 F 1 "21k" H 6970 4705 50  0000 L CNN
-F 2 "" V 6830 4750 50  0001 C CNN
+F 2 "Resistor_SMD:R_1206_3216Metric_Pad1.42x1.75mm_HandSolder" V 6830 4750 50  0001 C CNN
 F 3 "~" H 6900 4750 50  0001 C CNN
 	1    6900 4750
@@
 F 0 "C11" H 7565 4546 50  0000 L CNN
 F 1 "100n" H 7565 4455 50  0000 L CNN
-F 2 "" H 7488 4350 50  0001 C CNN
+F 2 "Capacitor_SMD:C_1206_3216Metric_Pad1.42x1.75mm_HandSolder" H 7488 4350 50  0001 C CNN
 F 3 "~" H 7450 4500 50  0001 C CNN
 	1    7450 4500
@@
 F 0 "R39" H 7520 4846 50  0000 L CNN
 F 1 "13k" H 7520 4755 50  0000 L CNN
-F 2 "" V 7380 4800 50  0001 C CNN
+F 2 "Resistor_SMD:R_1206_3216Metric_Pad1.42x1.75mm_HandSolder" V 7380 4800 50  0001 C CNN
 F 3 "~" H 7450 4800 50  0001 C CNN
 	1    7450 4800
@@
 F 0 "C7" H 6965 4196 50  0000 L CNN
 F 1 "4u7" H 6965 4105 50  0000 L CNN
-F 2 "" H 6888 4000 50  0001 C CNN
+F 2 "Capacitor_SMD:C_1206_3216Metric_Pad1.42x1.75mm_HandSolder" H 6888 4000 50  0001 C CNN
 F 3 "~" H 6850 4150 50  0001 C CNN
 	1    6850 4150
@@
 F 0 "C9" H 7015 3296 50  0000 L CNN
 F 1 "10u" H 7015 3205 50  0000 L CNN
-F 2 "" H 6938 3100 50  0001 C CNN
+F 2 "Capacitor_SMD:C_1206_3216Metric_Pad1.42x1.75mm_HandSolder" H 6938 3100 50  0001 C CNN
 F 3 "~" H 6900 3250 50  0001 C CNN
 	1    6900 3250
@@
 F 0 "C10" H 7365 3296 50  0000 L CNN
 F 1 "10u" H 7365 3205 50  0000 L CNN
-F 2 "" H 7288 3100 50  0001 C CNN
+F 2 "Capacitor_SMD:C_1206_3216Metric_Pad1.42x1.75mm_HandSolder" H 7288 3100 50  0001 C CNN
 F 3 "~" H 7250 3250 50  0001 C CNN
 	1    7250 3250
@@
 F 0 "C12" H 7765 3296 50  0000 L CNN
 F 1 "39u" H 7765 3205 50  0000 L CNN
-F 2 "" H 7688 3100 50  0001 C CNN
+F 2 "Capacitor_SMD:C_1206_3216Metric_Pad1.42x1.75mm_HandSolder" H 7688 3100 50  0001 C CNN
 F 3 "~" H 7650 3250 50  0001 C CNN
 	1    7650 3250
@@
 F 0 "C13" H 8115 3296 50  0000 L CNN
 F 1 "39u" H 8115 3205 50  0000 L CNN
-F 2 "" H 8038 3100 50  0001 C CNN
+F 2 "Capacitor_SMD:C_1206_3216Metric_Pad1.42x1.75mm_HandSolder" H 8038 3100 50  0001 C CNN
 F 3 "~" H 8000 3250 50  0001 C CNN
 	1    8000 3250
@@
 F 0 "R36" H 4520 3846 50  0000 L CNN
 F 1 "100k" H 4520 3755 50  0000 L CNN
-F 2 "" V 4380 3800 50  0001 C CNN
+F 2 "Resistor_SMD:R_1206_3216Metric_Pad1.42x1.75mm_HandSolder" V 4380 3800 50  0001 C CNN
 F 3 "~" H 4450 3800 50  0001 C CNN
 	1    4450 3800
@@
 F 0 "R34" H 4270 3846 50  0000 L CNN
 F 1 "100k" H 4270 3755 50  0000 L CNN
-F 2 "" V 4130 3800 50  0001 C CNN
+F 2 "Resistor_SMD:R_1206_3216Metric_Pad1.42x1.75mm_HandSolder" V 4130 3800 50  0001 C CNN
 F 3 "~" H 4200 3800 50  0001 C CNN
 	1    4200 3800

Commit message: footprints gemapt + 10x10 pcb rand getekend
Parts:
- U2: footprint Robin_Lib:DQJ0008A -> AudioProject:CSD18514Q5A
- U3: footprint Robin_Lib:DNH0008A -> AudioProject:CSD18543Q3A
- U4: footprint Robin_Lib:RPM0026A-MFG -> AudioProject:TPS552882QRPMRQ1
Changed lines of the file:
@@
 EESchema Schematic File Version 4
-EELAYER 30 0
+LIBS:PEE50_MPPT-cache
+EELAYER 26 0
 EELAYER END
 $Descr A4 11693 8268
@@
 F 0 "U4" H 5650 5238 60  0000 C CNN
 F 1 "TPS552882QRPMRQ1" H 5650 5132 60  0000 C CNN
-F 2 "Robin_Lib:RPM0026A-MFG" H 5650 3290 60  0001 C CNN
+F 2 "AudioProject:TPS552882QRPMRQ1" H 5650 3290 60  0001 C CNN
 F 3 "" H 5650 3350 60  0000 C CNN
 	1    5650 3350
@@
 F 0 "U2" V 4362 1203 60  0000 C CNN
 F 1 "CSD18514Q5A" V 4256 1203 60  0000 C CNN
-F 2 "Robin_Lib:DQJ0008A" H 4200 1050 60  0001 C CNN
+F 2 "AudioProject:CSD18514Q5A" H 4200 1050 60  0001 C CNN
 F 3 "" H 3750 1250 60  0000 C CNN
 	1    3750 1250
@@
 F 0 "U3" H 5131 1179 60  0000 L CNN
 F 1 "CSD18543Q3A" H 5131 1073 60  0000 L CNN
-F 2 "Robin_Lib:DNH0008A" H 4850 1090 60  0001 C CNN
+F 2 "AudioProject:CSD18543Q3A" H 4850 1090 60  0001 C CNN
 F 3 "" H 4850 1150 60  0000 C CNN
 	1    4850 1150

Commit message: best veel al gedaan voor 1e mppt
Parts:
- U3: footprint AudioProject:CSD18543Q3A -> Robin_Lib:DNH0008A
Changed lines of the file:
@@
 F 0 "U3" H 5131 1179 60  0000 L CNN
 F 1 "CSD18543Q3A" H 5131 1073 60  0000 L CNN
-F 2 "AudioProject:CSD18543Q3A" H 4850 1090 60  0001 C CNN
+F 2 "Robin_Lib:DNH0008A" H 4850 1090 60  0001 C CNN
 F 3 "" H 4850 1150 60  0000 C CNN
 	1    4850 1150
