File: PEE50_MPPT/DC_DC1.sch (KiCad schematic (older format))
At the start: 24 parts, among them U1 TPS552882QRPMRQ1, U2 CSD18514Q5A, U3 CSD18543Q3A

Commit message: schakeling klaar (denk ik)
Parts:
- removed C10, C11: 39u, symbol Device:C
- removed C2: 150u, symbol Device:C
- removed C4, C5, C9: 100n, symbol Device:C
- removed C6: 4u7, symbol Device:C
- removed C7, C8: 10u, symbol Device:C
- removed L1: 6u8, AudioProject:SER2915L-153KL, symbol pspice:INDUCTOR
- removed R11, R4: 100k, symbol Device:R
- removed R12: 21k, symbol Device:R
- removed R13: 13k, symbol Device:R
- removed R3: 383k, symbol Device:R
- removed R6: 66.5k, symbol Device:R
- removed U1: TPS552882QRPMRQ1, Robin_Lib:RPM0026A-MFG, symbol Robin_lib:TPS552882QRPMRQ1
- removed U2: CSD18514Q5A, Robin_Lib:DQJ0008A, symbol Robin_lib:CSD18514Q5A
- removed U3: CSD18543Q3A, Robin_Lib:DNH0008A, symbol Robin_lib:CSD18543Q3A
- added C18: 150u, symbol Device:C
- added C20, C22, C25: 100n, symbol Device:C
- added C21: 4u7, symbol Device:C
- added C23, C24: 10u, symbol Device:C
- added C26, C27: 39u, symbol Device:C
- added L2: 6u8, AudioProject:SER2915L-153KL, symbol pspice:INDUCTOR
- added R40: 383k, symbol Device:R
- added R41, R45: 100k, symbol Device:R
- added R44: 66.5k, symbol Device:R
- added R47: 21k, symbol Device:R
- added R48: 13k, symbol Device:R
- added U10: TPS552882QRPMRQ1, Robin_Lib:RPM0026A-MFG, symbol Robin_lib:TPS552882QRPMRQ1
- added U8: CSD18514Q5A, Robin_Lib:DQJ0008A, symbol Robin_lib:CSD18514Q5A
- added U9: CSD18543Q3A, Robin_Lib:DNH0008A, symbol Robin_lib:CSD18543Q3A
- renumbered C1 to C17, C3 to C19, R5 to R42, R10 to R43, R7 to R46
Connections:
- net FB: now also U10.14 (FB)
- net GND: now also C18.2, C21.2, C23.2, C24.2, C26.2, C27.2, R41.2, R44.2, R45.2, R47.2, R48.2, U10.10 (AGND), U10.15 (MODE), U10.24 (PGND), U10.7 (DITH_SYNC), U10.9 (PGND), U9.1 (S), U9.2 (S), U9.3 (S)
- net ISN: now also U10.13 (ISN)
- net ISP: now also U10.12 (ISP)
- net PVin+: now also C18.1, R40.1, U10.3 (VIN), U8.5 (D), U8.6 (D), U8.7 (D), U8.8 (D), U8.9 (D)
- net Vout: now also C23.1, C24.1, C26.1, C27.1, U10.11 (VOUT), U10.26 (VOUT)
- net at R46.2: now also U10.1 (DR1L)
- net at R42.2: now also U10.2 (DR1H)
- net at R43.1: now also U10.5 (PG)
- net at R42.1: now also U8.4 (G)
- net at R46.1: now also U9.4 (G)
- new net: R47.1, U10.17 (ILIM)
- new net: C25.2, U10.18 (COMP)
- new net: C21.1, U10.19 (VCC)
- new net: C22.1, U10.20 (BOOT2)
- new net: C22.2, L2.2, U10.21 (SW2), U10.25 (SW2)
- new net: C20.2, U10.22 (BOOT1)
- new net: C20.1, L2.1, U10.23 (SW1), U8.1 (S), U8.2 (S), U8.3 (S), U9.5 (D), U9.6 (D), U9.7 (D), U9.8 (D), U9.9 (D)
- new net: R40.2, R41.1, U10.4 (EN)
- new net: R45.1, U10.6 (CC_N)
- new net: R44.1, U10.8 (FSW)
- new net: C25.1, R48.1

Commit message: best veel footprints ingevoegd
Parts:
- C17, C18, C19, C20, C21, C22, C23, C24, C25, C26, C27: footprint (none) -> Capacitor_SMD:C_1206_3216Metric_Pad1.42x1.75mm_HandSolder
- R40, R41, R42, R43, R44, R45, R46, R47, R48: footprint (none) -> Resistor_SMD:R_1206_3216Metric_Pad1.42x1.75mm_HandSolder
Changed lines of the file:
@@
 EESchema Schematic File Version 4
-LIBS:PEE50_MPPT-cache
-EELAYER 26 0
+EELAYER 30 0
 EELAYER END
 $Descr A4 11693 8268
@@
 F 0 "C17" H 2365 2846 50  0000 L CNN
 F 1 "150u" H 2365 2755 50  0000 L CNN
-F 2 "" H 2288 2650 50  0001 C CNN
+F 2 "Capacitor_SMD:C_1206_3216Metric_Pad1.42x1.75mm_HandSolder" H 2288 2650 50  0001 C CNN
 F 3 "~" H 2250 2800 50  0001 C CNN
 	1    2250 2800
@@
 F 0 "C19" H 3165 2846 50  0000 L CNN
 F 1 "10u" H 3165 2755 50  0000 L CNN
-F 2 "" H 3088 2650 50  0001 C CNN
+F 2 "Capacitor_SMD:C_1206_3216Metric_Pad1.42x1.75mm_HandSolder" H 3088 2650 50  0001 C CNN
 F 3 "~" H 3050 2800 50  0001 C CNN
 	1    3050 2800
@@
 F 0 "C18" H 2765 2846 50  0000 L CNN
 F 1 "150u" H 2765 2755 50  0000 L CNN
-F 2 "" H 2688 2650 50  0001 C CNN
+F 2 "Capacitor_SMD:C_1206_3216Metric_Pad1.42x1.75mm_HandSolder" H 2688 2650 50  0001 C CNN
 F 3 "~" H 2650 2800 50  0001 C CNN
 	1    2650 2800
@@
 F 0 "R40" H 3620 2846 50  0000 L CNN
 F 1 "383k" H 3620 2755 50  0000 L CNN
-F 2 "" V 3480 2800 50  0001 C CNN
+F 2 "Resistor_SMD:R_1206_3216Metric_Pad1.42x1.75mm_HandSolder" V 3480 2800 50  0001 C CNN
 F 3 "~" H 3550 2800 50  0001 C CNN
 	1    3550 2800
@@
 F 0 "R41" H 3620 3196 50  0000 L CNN
 F 1 "100k" H 3620 3105 50  0000 L CNN
-F 2 "" V 3480 3150 50  0001 C CNN
+F 2 "Resistor_SMD:R_1206_3216Metric_Pad1.42x1.75mm_HandSolder" V 3480 3150 50  0001 C CNN
 F 3 "~" H 3550 3150 50  0001 C CNN
 	1    3550 3150
@@
 F 0 "R42" H 3820 1846 50  0000 L CNN
 F 1 "1" H 3820 1755 50  0000 L CNN
-F 2 "" V 3680 1800 50  0001 C CNN
+F 2 "Resistor_SMD:R_1206_3216Metric_Pad1.42x1.75mm_HandSolder" V 3680 1800 50  0001 C CNN
 F 3 "~" H 3750 1800 50  0001 C CNN
 	1    3750 1800
@@
 F 0 "R46" H 4570 1546 50  0000 L CNN
 F 1 "1" H 4570 1455 50  0000 L CNN
-F 2 "" V 4430 1500 50  0001 C CNN
+F 2 "Resistor_SMD:R_1206_3216Metric_Pad1.42x1.75mm_HandSolder" V 4430 1500 50  0001 C CNN
 F 3 "~" H 4500 1500 50  0001 C CNN
 	1    4500 1500
@@
 F 0 "C20" H 6715 1346 50  0000 L CNN
 F 1 "100n" H 6715 1255 50  0000 L CNN
-F 2 "" H 6638 1150 50  0001 C CNN
+F 2 "Capacitor_SMD:C_1206_3216Metric_Pad1.42x1.75mm_HandSolder" H 6638 1150 50  0001 C CNN
 F 3 "~" H 6600 1300 50  0001 C CNN
 	1    6600 1300
@@
 F 0 "C22" H 7015 2646 50  0000 L CNN
 F 1 "100n" H 7015 2555 50  0000 L CNN
-F 2 "" H 6938 2450 50  0001 C CNN
+F 2 "Capacitor_SMD:C_1206_3216Metric_Pad1.42x1.75mm_HandSolder" H 6938 2450 50  0001 C CNN
 F 3 "~" H 6900 2600 50  0001 C CNN
 	1    6900 2600
@@
 F 0 "R44" H 4270 4546 50  0000 L CNN
 F 1 "66.5k" H 4270 4455 50  0000 L CNN
-F 2 "" V 4130 4500 50  0001 C CNN
+F 2 "Resistor_SMD:R_1206_3216Metric_Pad1.42x1.75mm_HandSolder" V 4130 4500 50  0001 C CNN
 F 3 "~" H 4200 4500 50  0001 C CNN
 	1    4200 4500
@@
 F 0 "R47" H 6970 4796 50  0000 L CNN
 F 1 "21k" H 6970 4705 50  0000 L CNN
-F 2 "" V 6830 4750 50  0001 C CNN
+F 2 "Resistor_SMD:R_1206_3216Metric_Pad1.42x1.75mm_HandSolder" V 6830 4750 50  0001 C CNN
 F 3 "~" H 6900 4750 50  0001 C CNN
 	1    6900 4750
@@
 F 0 "C25" H 7565 4546 50  0000 L CNN
 F 1 "100n" H 7565 4455 50  0000 L CNN
-F 2 "" H 7488 4350 50  0001 C CNN
+F 2 "Capacitor_SMD:C_1206_3216Metric_Pad1.42x1.75mm_HandSolder" H 7488 4350 50  0001 C CNN
 F 3 "~" H 7450 4500 50  0001 C CNN
 	1    7450 4500
@@
 F 0 "R48" H 7520 4846 50  0000 L CNN
 F 1 "13k" H 7520 4755 50  0000 L CNN
-F 2 "" V 7380 4800 50  0001 C CNN
+F 2 "Resistor_SMD:R_1206_3216Metric_Pad1.42x1.75mm_HandSolder" V 7380 4800 50  0001 C CNN
 F 3 "~" H 7450 4800 50  0001 C CNN
 	1    7450 4800
@@
 F 0 "C21" H 6965 4196 50  0000 L CNN
 F 1 "4u7" H 6965 4105 50  0000 L CNN
-F 2 "" H 6888 4000 50  0001 C CNN
+F 2 "Capacitor_SMD:C_1206_3216Metric_Pad1.42x1.75mm_HandSolder" H 6888 4000 50  0001 C CNN
 F 3 "~" H 6850 4150 50  0001 C CNN
 	1    6850 4150
@@
 F 0 "C23" H 7015 3296 50  0000 L CNN
 F 1 "10u" H 7015 3205 50  0000 L CNN
-F 2 "" H 6938 3100 50  0001 C CNN
+F 2 "Capacitor_SMD:C_1206_3216Metric_Pad1.42x1.75mm_HandSolder" H 6938 3100 50  0001 C CNN
 F 3 "~" H 6900 3250 50  0001 C CNN
 	1    6900 3250
@@
 F 0 "C24" H 7365 3296 50  0000 L CNN
 F 1 "10u" H 7365 3205 50  0000 L CNN
-F 2 "" H 7288 3100 50  0001 C CNN
+F 2 "Capacitor_SMD:C_1206_3216Metric_Pad1.42x1.75mm_HandSolder" H 7288 3100 50  0001 C CNN
 F 3 "~" H 7250 3250 50  0001 C CNN
 	1    7250 3250
@@
 F 0 "C26" H 7765 3296 50  0000 L CNN
 F 1 "39u" H 7765 3205 50  0000 L CNN
-F 2 "" H 7688 3100 50  0001 C CNN
+F 2 "Capacitor_SMD:C_1206_3216Metric_Pad1.42x1.75mm_HandSolder" H 7688 3100 50  0001 C CNN
 F 3 "~" H 7650 3250 50  0001 C CNN
 	1    7650 3250
@@
 F 0 "C27" H 8115 3296 50  0000 L CNN
 F 1 "39u" H 8115 3205 50  0000 L CNN
-F 2 "" H 8038 3100 50  0001 C CNN
+F 2 "Capacitor_SMD:C_1206_3216Metric_Pad1.42x1.75mm_HandSolder" H 8038 3100 50  0001 C CNN
 F 3 "~" H 8000 3250 50  0001 C CNN
 	1    8000 3250
@@
 F 0 "R45" H 4520 3846 50  0000 L CNN
 F 1 "100k" H 4520 3755 50  0000 L CNN
-F 2 "" V 4380 3800 50  0001 C CNN
+F 2 "Resistor_SMD:R_1206_3216Metric_Pad1.42x1.75mm_HandSolder" V 4380 3800 50  0001 C CNN
 F 3 "~" H 4450 3800 50  0001 C CNN
 	1    4450 3800
@@
 F 0 "R43" H 4270 3846 50  0000 L CNN
 F 1 "100k" H 4270 3755 50  0000 L CNN
-F 2 "" V 4130 3800 50  0001 C CNN
+F 2 "Resistor_SMD:R_1206_3216Metric_Pad1.42x1.75mm_HandSolder" V 4130 3800 50  0001 C CNN
 F 3 "~" H 4200 3800 50  0001 C CNN
 	1    4200 3800

Commit message: footprints gemapt + 10x10 pcb rand getekend
Parts:
- U10: footprint Robin_Lib:RPM0026A-MFG -> AudioProject:TPS552882QRPMRQ1
- U8: footprint Robin_Lib:DQJ0008A -> AudioProject:CSD18514Q5A
- U9: footprint Robin_Lib:DNH0008A -> AudioProject:CSD18543Q3A
Changed lines of the file:
@@
 EESchema Schematic File Version 4
-EELAYER 30 0
+LIBS:PEE50_MPPT-cache
+EELAYER 26 0
 EELAYER END
 $Descr A4 11693 8268
@@
 F 0 "U10" H 5650 5238 60  0000 C CNN
 F 1 "TPS552882QRPMRQ1" H 5650 5132 60  0000 C CNN
-F 2 "Robin_Lib:RPM0026A-MFG" H 5650 3290 60  0001 C CNN
+F 2 "AudioProject:TPS552882QRPMRQ1" H 5650 3290 60  0001 C CNN
 F 3 "" H 5650 3350 60  0000 C CNN
 	1    5650 3350
@@
 F 0 "U8" V 4362 1203 60  0000 C CNN
 F 1 "CSD18514Q5A" V 4256 1203 60  0000 C CNN
-F 2 "Robin_Lib:DQJ0008A" H 4200 1050 60  0001 C CNN
+F 2 "AudioProject:CSD18514Q5A" H 4200 1050 60  0001 C CNN
 F 3 "" H 3750 1250 60  0000 C CNN
 	1    3750 1250
@@
 F 0 "U9" H 5131 1179 60  0000 L CNN
 F 1 "CSD18543Q3A" H 5131 1073 60  0000 L CNN
-F 2 "Robin_Lib:DNH0008A" H 4850 1090 60  0001 C CNN
+F 2 "AudioProject:CSD18543Q3A" H 4850 1090 60  0001 C CNN
 F 3 "" H 4850 1150 60  0000 C CNN
 	1    4850 1150

Commit message: best veel al gedaan voor 1e mppt
Parts:
- U9: footprint AudioProject:CSD18543Q3A -> Robin_Lib:DNH0008A
Changed lines of the file:
@@
 F 0 "U9" H 5131 1179 60  0000 L CNN
 F 1 "CSD18543Q3A" H 5131 1073 60  0000 L CNN
-F 2 "AudioProject:CSD18543Q3A" H 4850 1090 60  0001 C CNN
+F 2 "Robin_Lib:DNH0008A" H 4850 1090 60  0001 C CNN
 F 3 "" H 4850 1150 60  0000 C CNN
 	1    4850 1150
