File: PEE50_MPPT/DC_DC2.sch (KiCad schematic (older format))
At the start: 24 parts, among them U1 TPS552882QRPMRQ1, U2 CSD18514Q5A, U3 CSD18543Q3A

Commit message: schakeling klaar (denk ik)
Parts:
- removed C1, C2: 150u, symbol Device:C
- removed C10, C11: 39u, symbol Device:C
- removed C3, C8: 10u, symbol Device:C
- removed C5: 100n, symbol Device:C
- removed C6: 4u7, symbol Device:C
- removed R10: 100k, symbol Device:R
- removed R12: 21k, symbol Device:R
- removed R5, R7: 1, symbol Device:R
- removed U2: CSD18514Q5A, Robin_Lib:DQJ0008A, symbol Robin_lib:CSD18514Q5A
- added C43, C44: 150u, symbol Device:C
- added C45, C50: 10u, symbol Device:C
- added C47: 4u7, symbol Device:C
- added C48: 100n, symbol Device:C
- added C52, C53: 39u, symbol Device:C
- added R60, R64: 1, symbol Device:R
- added R61: 100k, symbol Device:R
- added R65: 21k, symbol Device:R
- added U18: CSD18514Q5A, Robin_Lib:DQJ0008A, symbol Robin_lib:CSD18514Q5A
- renumbered C4 to C46, C7 to C49, C9 to C51, L1 to L4, R3 to R58, R4 to R59, R6 to R62, R11 to R63, R13 to R66, U3 to U19, U1 to U20
Connections:
- net GND: now also C43.2, C44.2, C45.2, C47.2, C50.2, C52.2, C53.2, R61.2, R65.2
- net PVin+: now also C43.1, C44.1, C45.1, U18.5 (D), U18.6 (D), U18.7 (D), U18.8 (D), U18.9 (D)
- net Vout: now also C50.1, C52.1, C53.1
- net at U20.1 (DR1L): now also R64.2
- net at U20.17 (ILIM): now also R65.1
- net at U20.19 (VCC): now also C47.1
- net at U20.2 (DR1H): now also R60.2
- net at U20.20 (BOOT2): now also C48.1
- net at L4.2, U20.21 (SW2), U20.25 (SW2): now also C48.2
- net at C46.1, L4.1, U19.5 (D)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: now also U18.1 (S), U18.2 (S), U18.3 (S)
- net at U20.5 (PG): now also R61.1
- net at U19.4 (G): now also R64.1
- new net: R60.1, U18.4 (G)

Commit message: best veel footprints ingevoegd
Parts:
- C43, C44, C45, C46, C47, C48, C49, C50, C51, C52, C53: footprint (none) -> Capacitor_SMD:C_1206_3216Metric_Pad1.42x1.75mm_HandSolder
- R58, R59, R60, R61, R62, R63, R64, R65, R66: footprint (none) -> Resistor_SMD:R_1206_3216Metric_Pad1.42x1.75mm_HandSolder
Changed lines of the file:
@@
 EESchema Schematic File Version 4
-LIBS:PEE50_MPPT-cache
-EELAYER 26 0
+EELAYER 30 0
 EELAYER END
 $Descr A4 11693 8268
 encoding utf-8
-Sheet 2 15
+Sheet 12 15
 Title ""
 Date ""
@@
 F 0 "C43" H 2365 2846 50  0000 L CNN
 F 1 "150u" H 2365 2755 50  0000 L CNN
-F 2 "" H 2288 2650 50  0001 C CNN
+F 2 "Capacitor_SMD:C_1206_3216Metric_Pad1.42x1.75mm_HandSolder" H 2288 2650 50  0001 C CNN
 F 3 "~" H 2250 2800 50  0001 C CNN
 	1    2250 2800
@@
 F 0 "C45" H 3165 2846 50  0000 L CNN
 F 1 "10u" H 3165 2755 50  0000 L CNN
-F 2 "" H 3088 2650 50  0001 C CNN
+F 2 "Capacitor_SMD:C_1206_3216Metric_Pad1.42x1.75mm_HandSolder" H 3088 2650 50  0001 C CNN
 F 3 "~" H 3050 2800 50  0001 C CNN
 	1    3050 2800
@@
 F 0 "C44" H 2765 2846 50  0000 L CNN
 F 1 "150u" H 2765 2755 50  0000 L CNN
-F 2 "" H 2688 2650 50  0001 C CNN
+F 2 "Capacitor_SMD:C_1206_3216Metric_Pad1.42x1.75mm_HandSolder" H 2688 2650 50  0001 C CNN
 F 3 "~" H 2650 2800 50  0001 C CNN
 	1    2650 2800
@@
 F 0 "R58" H 3620 2846 50  0000 L CNN
 F 1 "383k" H 3620 2755 50  0000 L CNN
-F 2 "" V 3480 2800 50  0001 C CNN
+F 2 "Resistor_SMD:R_1206_3216Metric_Pad1.42x1.75mm_HandSolder" V 3480 2800 50  0001 C CNN
 F 3 "~" H 3550 2800 50  0001 C CNN
 	1    3550 2800
@@
 F 0 "R59" H 3620 3196 50  0000 L CNN
 F 1 "100k" H 3620 3105 50  0000 L CNN
-F 2 "" V 3480 3150 50  0001 C CNN
+F 2 "Resistor_SMD:R_1206_3216Metric_Pad1.42x1.75mm_HandSolder" V 3480 3150 50  0001 C CNN
 F 3 "~" H 3550 3150 50  0001 C CNN
 	1    3550 3150
@@
 F 0 "R60" H 3820 1846 50  0000 L CNN
 F 1 "1" H 3820 1755 50  0000 L CNN
-F 2 "" V 3680 1800 50  0001 C CNN
+F 2 "Resistor_SMD:R_1206_3216Metric_Pad1.42x1.75mm_HandSolder" V 3680 1800 50  0001 C CNN
 F 3 "~" H 3750 1800 50  0001 C CNN
 	1    3750 1800
@@
 F 0 "R64" H 4570 1546 50  0000 L CNN
 F 1 "1" H 4570 1455 50  0000 L CNN
-F 2 "" V 4430 1500 50  0001 C CNN
+F 2 "Resistor_SMD:R_1206_3216Metric_Pad1.42x1.75mm_HandSolder" V 4430 1500 50  0001 C CNN
 F 3 "~" H 4500 1500 50  0001 C CNN
 	1    4500 1500
@@
 F 0 "C46" H 6715 1346 50  0000 L CNN
 F 1 "100n" H 6715 1255 50  0000 L CNN
-F 2 "" H 6638 1150 50  0001 C CNN
+F 2 "Capacitor_SMD:C_1206_3216Metric_Pad1.42x1.75mm_HandSolder" H 6638 1150 50  0001 C CNN
 F 3 "~" H 6600 1300 50  0001 C CNN
 	1    6600 1300
@@
 F 0 "C48" H 7015 2646 50  0000 L CNN
 F 1 "100n" H 7015 2555 50  0000 L CNN
-F 2 "" H 6938 2450 50  0001 C CNN
+F 2 "Capacitor_SMD:C_1206_3216Metric_Pad1.42x1.75mm_HandSolder" H 6938 2450 50  0001 C CNN
 F 3 "~" H 6900 2600 50  0001 C CNN
 	1    6900 2600
@@
 F 0 "R62" H 4270 4546 50  0000 L CNN
 F 1 "66.5k" H 4270 4455 50  0000 L CNN
-F 2 "" V 4130 4500 50  0001 C CNN
+F 2 "Resistor_SMD:R_1206_3216Metric_Pad1.42x1.75mm_HandSolder" V 4130 4500 50  0001 C CNN
 F 3 "~" H 4200 4500 50  0001 C CNN
 	1    4200 4500
@@
 F 0 "R65" H 6970 4796 50  0000 L CNN
 F 1 "21k" H 6970 4705 50  0000 L CNN
-F 2 "" V 6830 4750 50  0001 C CNN
+F 2 "Resistor_SMD:R_1206_3216Metric_Pad1.42x1.75mm_HandSolder" V 6830 4750 50  0001 C CNN
 F 3 "~" H 6900 4750 50  0001 C CNN
 	1    6900 4750
@@
 F 0 "C51" H 7565 4546 50  0000 L CNN
 F 1 "100n" H 7565 4455 50  0000 L CNN
-F 2 "" H 7488 4350 50  0001 C CNN
+F 2 "Capacitor_SMD:C_1206_3216Metric_Pad1.42x1.75mm_HandSolder" H 7488 4350 50  0001 C CNN
 F 3 "~" H 7450 4500 50  0001 C CNN
 	1    7450 4500
@@
 F 0 "R66" H 7520 4846 50  0000 L CNN
 F 1 "13k" H 7520 4755 50  0000 L CNN
-F 2 "" V 7380 4800 50  0001 C CNN
+F 2 "Resistor_SMD:R_1206_3216Metric_Pad1.42x1.75mm_HandSolder" V 7380 4800 50  0001 C CNN
 F 3 "~" H 7450 4800 50  0001 C CNN
 	1    7450 4800
@@
 F 0 "C47" H 6965 4196 50  0000 L CNN
 F 1 "4u7" H 6965 4105 50  0000 L CNN
-F 2 "" H 6888 4000 50  0001 C CNN
+F 2 "Capacitor_SMD:C_1206_3216Metric_Pad1.42x1.75mm_HandSolder" H 6888 4000 50  0001 C CNN
 F 3 "~" H 6850 4150 50  0001 C CNN
 	1    6850 4150
@@
 F 0 "C49" H 7015 3296 50  0000 L CNN
 F 1 "10u" H 7015 3205 50  0000 L CNN
-F 2 "" H 6938 3100 50  0001 C CNN
+F 2 "Capacitor_SMD:C_1206_3216Metric_Pad1.42x1.75mm_HandSolder" H 6938 3100 50  0001 C CNN
 F 3 "~" H 6900 3250 50  0001 C CNN
 	1    6900 3250
@@
 F 0 "C50" H 7365 3296 50  0000 L CNN
 F 1 "10u" H 7365 3205 50  0000 L CNN
-F 2 "" H 7288 3100 50  0001 C CNN
+F 2 "Capacitor_SMD:C_1206_3216Metric_Pad1.42x1.75mm_HandSolder" H 7288 3100 50  0001 C CNN
 F 3 "~" H 7250 3250 50  0001 C CNN
 	1    7250 3250
@@
 F 0 "C52" H 7765 3296 50  0000 L CNN
 F 1 "39u" H 7765 3205 50  0000 L CNN
-F 2 "" H 7688 3100 50  0001 C CNN
+F 2 "Capacitor_SMD:C_1206_3216Metric_Pad1.42x1.75mm_HandSolder" H 7688 3100 50  0001 C CNN
 F 3 "~" H 7650 3250 50  0001 C CNN
 	1    7650 3250
@@
 F 0 "C53" H 8115 3296 50  0000 L CNN
 F 1 "39u" H 8115 3205 50  0000 L CNN
-F 2 "" H 8038 3100 50  0001 C CNN
+F 2 "Capacitor_SMD:C_1206_3216Metric_Pad1.42x1.75mm_HandSolder" H 8038 3100 50  0001 C CNN
 F 3 "~" H 8000 3250 50  0001 C CNN
 	1    8000 3250
@@
 F 0 "R63" H 4520 3846 50  0000 L CNN
 F 1 "100k" H 4520 3755 50  0000 L CNN
-F 2 "" V 4380 3800 50  0001 C CNN
+F 2 "Resistor_SMD:R_1206_3216Metric_Pad1.42x1.75mm_HandSolder" V 4380 3800 50  0001 C CNN
 F 3 "~" H 4450 3800 50  0001 C CNN
 	1    4450 3800
@@
 F 0 "R61" H 4270 3846 50  0000 L CNN
 F 1 "100k" H 4270 3755 50  0000 L CNN
-F 2 "" V 4130 3800 50  0001 C CNN
+F 2 "Resistor_SMD:R_1206_3216Metric_Pad1.42x1.75mm_HandSolder" V 4130 3800 50  0001 C CNN
 F 3 "~" H 4200 3800 50  0001 C CNN
 	1    4200 3800

Commit message: footprints gemapt + 10x10 pcb rand getekend
Parts:
- U18: footprint Robin_Lib:DQJ0008A -> AudioProject:CSD18514Q5A
- U19: footprint Robin_Lib:DNH0008A -> AudioProject:CSD18543Q3A
- U20: footprint Robin_Lib:RPM0026A-MFG -> AudioProject:TPS552882QRPMRQ1
Changed lines of the file:
@@
 EESchema Schematic File Version 4
-EELAYER 30 0
+LIBS:PEE50_MPPT-cache
+EELAYER 26 0
 EELAYER END
 $Descr A4 11693 8268
@@
 F 0 "U20" H 5650 5238 60  0000 C CNN
 F 1 "TPS552882QRPMRQ1" H 5650 5132 60  0000 C CNN
-F 2 "Robin_Lib:RPM0026A-MFG" H 5650 3290 60  0001 C CNN
+F 2 "AudioProject:TPS552882QRPMRQ1" H 5650 3290 60  0001 C CNN
 F 3 "" H 5650 3350 60  0000 C CNN
 	1    5650 3350
@@
 F 0 "U18" V 4362 1203 60  0000 C CNN
 F 1 "CSD18514Q5A" V 4256 1203 60  0000 C CNN
-F 2 "Robin_Lib:DQJ0008A" H 4200 1050 60  0001 C CNN
+F 2 "AudioProject:CSD18514Q5A" H 4200 1050 60  0001 C CNN
 F 3 "" H 3750 1250 60  0000 C CNN
 	1    3750 1250
@@
 F 0 "U19" H 5131 1179 60  0000 L CNN
 F 1 "CSD18543Q3A" H 5131 1073 60  0000 L CNN
-F 2 "Robin_Lib:DNH0008A" H 4850 1090 60  0001 C CNN
+F 2 "AudioProject:CSD18543Q3A" H 4850 1090 60  0001 C CNN
 F 3 "" H 4850 1150 60  0000 C CNN
 	1    4850 1150

Commit message: best veel al gedaan voor 1e mppt
Parts:
- U19: footprint AudioProject:CSD18543Q3A -> Robin_Lib:DNH0008A
Changed lines of the file:
@@
 F 0 "U19" H 5131 1179 60  0000 L CNN
 F 1 "CSD18543Q3A" H 5131 1073 60  0000 L CNN
-F 2 "AudioProject:CSD18543Q3A" H 4850 1090 60  0001 C CNN
+F 2 "Robin_Lib:DNH0008A" H 4850 1090 60  0001 C CNN
 F 3 "" H 4850 1150 60  0000 C CNN
 	1    4850 1150
