File: PEE50_MPPT/DC_DC3.sch (KiCad schematic (older format))
At the start: 24 parts, among them U1 TPS552882QRPMRQ1, U2 CSD18514Q5A, U3 CSD18543Q3A

Commit message: schakeling klaar (denk ik)
Parts:
- removed C1: 150u, symbol Device:C
- removed C3, C7: 10u, symbol Device:C
- removed C4, C9: 100n, symbol Device:C
- removed C6: 4u7, symbol Device:C
- removed L1: 6u8, AudioProject:SER2915L-153KL, symbol pspice:INDUCTOR
- removed R10, R11, R4: 100k, symbol Device:R
- removed R12: 21k, symbol Device:R
- removed R13: 13k, symbol Device:R
- removed R3: 383k, symbol Device:R
- removed R5, R7: 1, symbol Device:R
- removed R6: 66.5k, symbol Device:R
- removed U1: TPS552882QRPMRQ1, Robin_Lib:RPM0026A-MFG, symbol Robin_lib:TPS552882QRPMRQ1
- removed U2: CSD18514Q5A, Robin_Lib:DQJ0008A, symbol Robin_lib:CSD18514Q5A
- removed U3: CSD18543Q3A, Robin_Lib:DNH0008A, symbol Robin_lib:CSD18543Q3A
- added C30: 150u, symbol Device:C
- added C32, C36: 10u, symbol Device:C
- added C33, C38: 100n, symbol Device:C
- added C34: 4u7, symbol Device:C
- added L3: 6u8, AudioProject:SER2915L-153KL, symbol pspice:INDUCTOR
- added R49: 383k, symbol Device:R
- added R50, R52, R54: 100k, symbol Device:R
- added R51, R55: 1, symbol Device:R
- added R53: 66.5k, symbol Device:R
- added R56: 21k, symbol Device:R
- added R57: 13k, symbol Device:R
- added U13: CSD18514Q5A, Robin_Lib:DQJ0008A, symbol Robin_lib:CSD18514Q5A
- added U14: CSD18543Q3A, Robin_Lib:DNH0008A, symbol Robin_lib:CSD18543Q3A
- added U15: TPS552882QRPMRQ1, Robin_Lib:RPM0026A-MFG, symbol Robin_lib:TPS552882QRPMRQ1
- renumbered C2 to C31, C5 to C35, C8 to C37, C10 to C39, C11 to C40
Connections:
- net FB: now also U15.14 (FB)
- net GND: now also C30.2, C32.2, C34.2, C36.2, R50.2, R52.2, R53.2, R54.2, R56.2, R57.2, U14.1 (S), U14.2 (S), U14.3 (S), U15.10 (AGND), U15.15 (MODE), U15.24 (PGND), U15.7 (DITH_SYNC), U15.9 (PGND)
- net ISN: now also U15.13 (ISN)
- net ISP: now also U15.12 (ISP)
- net PVin+: now also C30.1, C32.1, R49.1, U13.5 (D), U13.6 (D), U13.7 (D), U13.8 (D), U13.9 (D), U15.3 (VIN)
- net Vout: now also C36.1, U15.11 (VOUT), U15.26 (VOUT)
- net at C35.1: now also U15.20 (BOOT2)
- net at C35.2: now also L3.2, U15.21 (SW2), U15.25 (SW2)
- new net: R55.2, U15.1 (DR1L)
- new net: R56.1, U15.17 (ILIM)
- new net: C38.2, U15.18 (COMP)
- new net: C34.1, U15.19 (VCC)
- new net: R51.2, U15.2 (DR1H)
- new net: C33.2, U15.22 (BOOT1)
- new net: C33.1, L3.1, U13.1 (S), U13.2 (S), U13.3 (S), U14.5 (D), U14.6 (D), U14.7 (D), U14.8 (D), U14.9 (D), U15.23 (SW1)
- new net: R49.2, R50.1, U15.4 (EN)
- new net: R52.1, U15.5 (PG)
- new net: R54.1, U15.6 (CC_N)
- new net: R53.1, U15.8 (FSW)
- new net: R51.1, U13.4 (G)
- new net: R55.1, U14.4 (G)
- new net: C38.1, R57.1

Commit message: best veel footprints ingevoegd
Parts:
- C30, C31, C32, C33, C34, C35, C36, C37, C38, C39, C40: footprint (none) -> Capacitor_SMD:C_1206_3216Metric_Pad1.42x1.75mm_HandSolder
- R49, R50, R51, R52, R53, R54, R55, R56, R57: footprint (none) -> Resistor_SMD:R_1206_3216Metric_Pad1.42x1.75mm_HandSolder
Changed lines of the file:
@@
 EESchema Schematic File Version 4
-LIBS:PEE50_MPPT-cache
-EELAYER 26 0
+EELAYER 30 0
 EELAYER END
 $Descr A4 11693 8268
@@
 F 0 "C30" H 2365 2846 50  0000 L CNN
 F 1 "150u" H 2365 2755 50  0000 L CNN
-F 2 "" H 2288 2650 50  0001 C CNN
+F 2 "Capacitor_SMD:C_1206_3216Metric_Pad1.42x1.75mm_HandSolder" H 2288 2650 50  0001 C CNN
 F 3 "~" H 2250 2800 50  0001 C CNN
 	1    2250 2800
@@
 F 0 "C32" H 3165 2846 50  0000 L CNN
 F 1 "10u" H 3165 2755 50  0000 L CNN
-F 2 "" H 3088 2650 50  0001 C CNN
+F 2 "Capacitor_SMD:C_1206_3216Metric_Pad1.42x1.75mm_HandSolder" H 3088 2650 50  0001 C CNN
 F 3 "~" H 3050 2800 50  0001 C CNN
 	1    3050 2800
@@
 F 0 "C31" H 2765 2846 50  0000 L CNN
 F 1 "150u" H 2765 2755 50  0000 L CNN
-F 2 "" H 2688 2650 50  0001 C CNN
+F 2 "Capacitor_SMD:C_1206_3216Metric_Pad1.42x1.75mm_HandSolder" H 2688 2650 50  0001 C CNN
 F 3 "~" H 2650 2800 50  0001 C CNN
 	1    2650 2800
@@
 F 0 "R49" H 3620 2846 50  0000 L CNN
 F 1 "383k" H 3620 2755 50  0000 L CNN
-F 2 "" V 3480 2800 50  0001 C CNN
+F 2 "Resistor_SMD:R_1206_3216Metric_Pad1.42x1.75mm_HandSolder" V 3480 2800 50  0001 C CNN
 F 3 "~" H 3550 2800 50  0001 C CNN
 	1    3550 2800
@@
 F 0 "R50" H 3620 3196 50  0000 L CNN
 F 1 "100k" H 3620 3105 50  0000 L CNN
-F 2 "" V 3480 3150 50  0001 C CNN
+F 2 "Resistor_SMD:R_1206_3216Metric_Pad1.42x1.75mm_HandSolder" V 3480 3150 50  0001 C CNN
 F 3 "~" H 3550 3150 50  0001 C CNN
 	1    3550 3150
@@
 F 0 "R51" H 3820 1846 50  0000 L CNN
 F 1 "1" H 3820 1755 50  0000 L CNN
-F 2 "" V 3680 1800 50  0001 C CNN
+F 2 "Resistor_SMD:R_1206_3216Metric_Pad1.42x1.75mm_HandSolder" V 3680 1800 50  0001 C CNN
 F 3 "~" H 3750 1800 50  0001 C CNN
 	1    3750 1800
@@
 F 0 "R55" H 4570 1546 50  0000 L CNN
 F 1 "1" H 4570 1455 50  0000 L CNN
-F 2 "" V 4430 1500 50  0001 C CNN
+F 2 "Resistor_SMD:R_1206_3216Metric_Pad1.42x1.75mm_HandSolder" V 4430 1500 50  0001 C CNN
 F 3 "~" H 4500 1500 50  0001 C CNN
 	1    4500 1500
@@
 F 0 "C33" H 6715 1346 50  0000 L CNN
 F 1 "100n" H 6715 1255 50  0000 L CNN
-F 2 "" H 6638 1150 50  0001 C CNN
+F 2 "Capacitor_SMD:C_1206_3216Metric_Pad1.42x1.75mm_HandSolder" H 6638 1150 50  0001 C CNN
 F 3 "~" H 6600 1300 50  0001 C CNN
 	1    6600 1300
@@
 F 0 "C35" H 7015 2646 50  0000 L CNN
 F 1 "100n" H 7015 2555 50  0000 L CNN
-F 2 "" H 6938 2450 50  0001 C CNN
+F 2 "Capacitor_SMD:C_1206_3216Metric_Pad1.42x1.75mm_HandSolder" H 6938 2450 50  0001 C CNN
 F 3 "~" H 6900 2600 50  0001 C CNN
 	1    6900 2600
@@
 F 0 "R53" H 4270 4546 50  0000 L CNN
 F 1 "66.5k" H 4270 4455 50  0000 L CNN
-F 2 "" V 4130 4500 50  0001 C CNN
+F 2 "Resistor_SMD:R_1206_3216Metric_Pad1.42x1.75mm_HandSolder" V 4130 4500 50  0001 C CNN
 F 3 "~" H 4200 4500 50  0001 C CNN
 	1    4200 4500
@@
 F 0 "R56" H 6970 4796 50  0000 L CNN
 F 1 "21k" H 6970 4705 50  0000 L CNN
-F 2 "" V 6830 4750 50  0001 C CNN
+F 2 "Resistor_SMD:R_1206_3216Metric_Pad1.42x1.75mm_HandSolder" V 6830 4750 50  0001 C CNN
 F 3 "~" H 6900 4750 50  0001 C CNN
 	1    6900 4750
@@
 F 0 "C38" H 7565 4546 50  0000 L CNN
 F 1 "100n" H 7565 4455 50  0000 L CNN
-F 2 "" H 7488 4350 50  0001 C CNN
+F 2 "Capacitor_SMD:C_1206_3216Metric_Pad1.42x1.75mm_HandSolder" H 7488 4350 50  0001 C CNN
 F 3 "~" H 7450 4500 50  0001 C CNN
 	1    7450 4500
@@
 F 0 "R57" H 7520 4846 50  0000 L CNN
 F 1 "13k" H 7520 4755 50  0000 L CNN
-F 2 "" V 7380 4800 50  0001 C CNN
+F 2 "Resistor_SMD:R_1206_3216Metric_Pad1.42x1.75mm_HandSolder" V 7380 4800 50  0001 C CNN
 F 3 "~" H 7450 4800 50  0001 C CNN
 	1    7450 4800
@@
 F 0 "C34" H 6965 4196 50  0000 L CNN
 F 1 "4u7" H 6965 4105 50  0000 L CNN
-F 2 "" H 6888 4000 50  0001 C CNN
+F 2 "Capacitor_SMD:C_1206_3216Metric_Pad1.42x1.75mm_HandSolder" H 6888 4000 50  0001 C CNN
 F 3 "~" H 6850 4150 50  0001 C CNN
 	1    6850 4150
@@
 F 0 "C36" H 7015 3296 50  0000 L CNN
 F 1 "10u" H 7015 3205 50  0000 L CNN
-F 2 "" H 6938 3100 50  0001 C CNN
+F 2 "Capacitor_SMD:C_1206_3216Metric_Pad1.42x1.75mm_HandSolder" H 6938 3100 50  0001 C CNN
 F 3 "~" H 6900 3250 50  0001 C CNN
 	1    6900 3250
@@
 F 0 "C37" H 7365 3296 50  0000 L CNN
 F 1 "10u" H 7365 3205 50  0000 L CNN
-F 2 "" H 7288 3100 50  0001 C CNN
+F 2 "Capacitor_SMD:C_1206_3216Metric_Pad1.42x1.75mm_HandSolder" H 7288 3100 50  0001 C CNN
 F 3 "~" H 7250 3250 50  0001 C CNN
 	1    7250 3250
@@
 F 0 "C39" H 7765 3296 50  0000 L CNN
 F 1 "39u" H 7765 3205 50  0000 L CNN
-F 2 "" H 7688 3100 50  0001 C CNN
+F 2 "Capacitor_SMD:C_1206_3216Metric_Pad1.42x1.75mm_HandSolder" H 7688 3100 50  0001 C CNN
 F 3 "~" H 7650 3250 50  0001 C CNN
 	1    7650 3250
@@
 F 0 "C40" H 8115 3296 50  0000 L CNN
 F 1 "39u" H 8115 3205 50  0000 L CNN
-F 2 "" H 8038 3100 50  0001 C CNN
+F 2 "Capacitor_SMD:C_1206_3216Metric_Pad1.42x1.75mm_HandSolder" H 8038 3100 50  0001 C CNN
 F 3 "~" H 8000 3250 50  0001 C CNN
 	1    8000 3250
@@
 F 0 "R54" H 4520 3846 50  0000 L CNN
 F 1 "100k" H 4520 3755 50  0000 L CNN
-F 2 "" V 4380 3800 50  0001 C CNN
+F 2 "Resistor_SMD:R_1206_3216Metric_Pad1.42x1.75mm_HandSolder" V 4380 3800 50  0001 C CNN
 F 3 "~" H 4450 3800 50  0001 C CNN
 	1    4450 3800
@@
 F 0 "R52" H 4270 3846 50  0000 L CNN
 F 1 "100k" H 4270 3755 50  0000 L CNN
-F 2 "" V 4130 3800 50  0001 C CNN
+F 2 "Resistor_SMD:R_1206_3216Metric_Pad1.42x1.75mm_HandSolder" V 4130 3800 50  0001 C CNN
 F 3 "~" H 4200 3800 50  0001 C CNN
 	1    4200 3800

Commit message: footprints gemapt + 10x10 pcb rand getekend
Parts:
- U13: footprint Robin_Lib:DQJ0008A -> AudioProject:CSD18514Q5A
- U14: footprint Robin_Lib:DNH0008A -> AudioProject:CSD18543Q3A
- U15: footprint Robin_Lib:RPM0026A-MFG -> AudioProject:TPS552882QRPMRQ1
Changed lines of the file:
@@
 EESchema Schematic File Version 4
-EELAYER 30 0
+LIBS:PEE50_MPPT-cache
+EELAYER 26 0
 EELAYER END
 $Descr A4 11693 8268
@@
 F 0 "U15" H 5650 5238 60  0000 C CNN
 F 1 "TPS552882QRPMRQ1" H 5650 5132 60  0000 C CNN
-F 2 "Robin_Lib:RPM0026A-MFG" H 5650 3290 60  0001 C CNN
+F 2 "AudioProject:TPS552882QRPMRQ1" H 5650 3290 60  0001 C CNN
 F 3 "" H 5650 3350 60  0000 C CNN
 	1    5650 3350
@@
 F 0 "U13" V 4362 1203 60  0000 C CNN
 F 1 "CSD18514Q5A" V 4256 1203 60  0000 C CNN
-F 2 "Robin_Lib:DQJ0008A" H 4200 1050 60  0001 C CNN
+F 2 "AudioProject:CSD18514Q5A" H 4200 1050 60  0001 C CNN
 F 3 "" H 3750 1250 60  0000 C CNN
 	1    3750 1250
@@
 F 0 "U14" H 5131 1179 60  0000 L CNN
 F 1 "CSD18543Q3A" H 5131 1073 60  0000 L CNN
-F 2 "Robin_Lib:DNH0008A" H 4850 1090 60  0001 C CNN
+F 2 "AudioProject:CSD18543Q3A" H 4850 1090 60  0001 C CNN
 F 3 "" H 4850 1150 60  0000 C CNN
 	1    4850 1150

Commit message: best veel al gedaan voor 1e mppt
Parts:
- U14: footprint AudioProject:CSD18543Q3A -> Robin_Lib:DNH0008A
Changed lines of the file:
@@
 F 0 "U14" H 5131 1179 60  0000 L CNN
 F 1 "CSD18543Q3A" H 5131 1073 60  0000 L CNN
-F 2 "AudioProject:CSD18543Q3A" H 4850 1090 60  0001 C CNN
+F 2 "Robin_Lib:DNH0008A" H 4850 1090 60  0001 C CNN
 F 3 "" H 4850 1150 60  0000 C CNN
 	1    4850 1150
