File: PEE50_MPPT/multiplexer.sch (KiCad schematic (older format))
At the start: 2 parts

Commit message: laatste spanning bijgevoegd (was vergeten)
Connections:
- net S13: now reaches U?.7 (S13)
Changed lines of the file:
@@
 Wire Wire Line
 	7400 2650 7300 2650
+Text HLabel 5050 3250 0    50   Input ~ 0
+S13
+Wire Wire Line
+	5050 3250 5100 3250
 $EndSCHEMATC

Commit message: schakeling klaar (denk ik)
Parts:
- gave numbers to parts that had none: 2
Changed lines of the file:
@@
 $EndDescr
 $Comp
-L power:+3.3V #PWR0182
+L power:+3.3V #PWR090
 U 1 1 60946E3C
 P 4950 2600
-F 0 "#PWR0182" H 4950 2450 50  0001 C CNN
+F 0 "#PWR090" H 4950 2450 50  0001 C CNN
 F 1 "+3.3V" H 4965 2773 50  0000 C CNN
 F 2 "" H 4950 2600 50  0001 C CNN
@@
 	4950 2650 5100 2650
 $Comp
-L Device:C C?
+L Device:C C56
 U 1 1 60946E6B
 P 4700 2650
-F 0 "C?" V 4448 2650 50  0000 C CNN
+F 0 "C56" V 4448 2650 50  0000 C CNN
 F 1 "100n" V 4539 2650 50  0000 C CNN
 F 2 "" H 4738 2500 50  0001 C CNN
@@
 Connection ~ 4950 2650
 $Comp
-L power:GND #PWR0183
+L power:GND #PWR092
 U 1 1 60946EFE
 P 7350 2750
-F 0 "#PWR0183" H 7350 2500 50  0001 C CNN
+F 0 "#PWR092" H 7350 2500 50  0001 C CNN
 F 1 "GND" V 7355 2622 50  0000 R CNN
 F 2 "" H 7350 2750 50  0001 C CNN
@@
 $EndComp
 $Comp
-L power:GND #PWR0184
+L power:GND #PWR089
 U 1 1 60946F24
 P 4450 2650
-F 0 "#PWR0184" H 4450 2400 50  0001 C CNN
+F 0 "#PWR089" H 4450 2400 50  0001 C CNN
 F 1 "GND" V 4455 2522 50  0000 R CNN
 F 2 "" H 4450 2650 50  0001 C CNN
@@
 	7400 3950 7300 3950
 $Comp
-L Robin_lib:ADG706BRUZ U?
+L Robin_lib:ADG706BRUZ U23
 U 1 1 609480C8
 P 5100 2650
-F 0 "U?" H 6200 3037 60  0000 C CNN
+F 0 "U23" H 6200 3037 60  0000 C CNN
 F 1 "ADG706BRUZ" H 6200 2931 60  0000 C CNN
 F 2 "RU_28_ADI" H 6200 2890 60  0001 C CNN
@@
 $EndComp
 $Comp
-L power:+3.3V #PWR?
+L power:+3.3V #PWR093
 U 1 1 60948499
 P 7350 3650
-F 0 "#PWR?" H 7350 3500 50  0001 C CNN
+F 0 "#PWR093" H 7350 3500 50  0001 C CNN
 F 1 "+3.3V" V 7365 3778 50  0000 L CNN
 F 2 "" H 7350 3650 50  0001 C CNN
@@
 S12
 $Comp
-L power:GND #PWR?
+L power:GND #PWR091
 U 1 1 609489B0
 P 5000 3750
-F 0 "#PWR?" H 5000 3500 50  0001 C CNN
+F 0 "#PWR091" H 5000 3500 50  0001 C CNN
 F 1 "GND" V 5005 3622 50  0000 R CNN
 F 2 "" H 5000 3750 50  0001 C CNN

Commit message: best veel footprints ingevoegd
Parts:
- C56: footprint (none) -> Capacitor_SMD:C_1206_3216Metric_Pad1.42x1.75mm_HandSolder
Changed lines of the file:
@@
 EESchema Schematic File Version 4
-LIBS:PEE50_MPPT-cache
-EELAYER 26 0
+EELAYER 30 0
 EELAYER END
 $Descr A4 11693 8268
@@
 F 0 "C56" V 4448 2650 50  0000 C CNN
 F 1 "100n" V 4539 2650 50  0000 C CNN
-F 2 "" H 4738 2500 50  0001 C CNN
+F 2 "Capacitor_SMD:C_1206_3216Metric_Pad1.42x1.75mm_HandSolder" H 4738 2500 50  0001 C CNN
 F 3 "~" H 4700 2650 50  0001 C CNN
 	1    4700 2650

Commit message: footprints gemapt + 10x10 pcb rand getekend
Parts:
- U23: footprint RU_28_ADI -> AudioProject:ADG706BRUZ
Changed lines of the file:
@@
 EESchema Schematic File Version 4
-EELAYER 30 0
+LIBS:PEE50_MPPT-cache
+EELAYER 26 0
 EELAYER END
 $Descr A4 11693 8268
@@
 F 0 "U23" H 6200 3037 60  0000 C CNN
 F 1 "ADG706BRUZ" H 6200 2931 60  0000 C CNN
-F 2 "RU_28_ADI" H 6200 2890 60  0001 C CNN
+F 2 "AudioProject:ADG706BRUZ" H 6200 2890 60  0001 C CNN
 F 3 "" H 5100 2650 60  0000 C CNN
 	1    5100 2650

Commit message: maar opnieuw begonnen met mppt layouten ivm plugin regels
Parts:
- renumbered C56 to C6, U23 to U3
Changed lines of the file:
@@
 $Descr A4 11693 8268
 encoding utf-8
-Sheet 15 15
+Sheet 15 19
 Title ""
 Date ""
@@
 $EndDescr
 $Comp
-L power:+3.3V #PWR090
+L power:+3.3V #PWR013
 U 1 1 60946E3C
 P 4950 2600
-F 0 "#PWR090" H 4950 2450 50  0001 C CNN
+F 0 "#PWR013" H 4950 2450 50  0001 C CNN
 F 1 "+3.3V" H 4965 2773 50  0000 C CNN
 F 2 "" H 4950 2600 50  0001 C CNN
@@
 	4950 2650 5100 2650
 $Comp
-L Device:C C56
+L Device:C C6
 U 1 1 60946E6B
 P 4700 2650
-F 0 "C56" V 4448 2650 50  0000 C CNN
+F 0 "C6" V 4448 2650 50  0000 C CNN
 F 1 "100n" V 4539 2650 50  0000 C CNN
 F 2 "Capacitor_SMD:C_1206_3216Metric_Pad1.42x1.75mm_HandSolder" H 4738 2500 50  0001 C CNN
@@
 Connection ~ 4950 2650
 $Comp
-L power:GND #PWR092
+L power:GND #PWR015
 U 1 1 60946EFE
 P 7350 2750
-F 0 "#PWR092" H 7350 2500 50  0001 C CNN
+F 0 "#PWR015" H 7350 2500 50  0001 C CNN
 F 1 "GND" V 7355 2622 50  0000 R CNN
 F 2 "" H 7350 2750 50  0001 C CNN
@@
 $EndComp
 $Comp
-L power:GND #PWR089
+L power:GND #PWR012
 U 1 1 60946F24
 P 4450 2650
-F 0 "#PWR089" H 4450 2400 50  0001 C CNN
+F 0 "#PWR012" H 4450 2400 50  0001 C CNN
 F 1 "GND" V 4455 2522 50  0000 R CNN
 F 2 "" H 4450 2650 50  0001 C CNN
@@
 	7400 3950 7300 3950
 $Comp
-L Robin_lib:ADG706BRUZ U23
+L Robin_lib:ADG706BRUZ U3
 U 1 1 609480C8
 P 5100 2650
-F 0 "U23" H 6200 3037 60  0000 C CNN
+F 0 "U3" H 6200 3037 60  0000 C CNN
 F 1 "ADG706BRUZ" H 6200 2931 60  0000 C CNN
 F 2 "AudioProject:ADG706BRUZ" H 6200 2890 60  0001 C CNN
@@
 $EndComp
 $Comp
-L power:+3.3V #PWR093
+L power:+3.3V #PWR016
 U 1 1 60948499
 P 7350 3650
-F 0 "#PWR093" H 7350 3500 50  0001 C CNN
+F 0 "#PWR016" H 7350 3500 50  0001 C CNN
 F 1 "+3.3V" V 7365 3778 50  0000 L CNN
 F 2 "" H 7350 3650 50  0001 C CNN
@@
 S12
 $Comp
-L power:GND #PWR091
+L power:GND #PWR014
 U 1 1 609489B0
 P 5000 3750
-F 0 "#PWR091" H 5000 3500 50  0001 C CNN
+F 0 "#PWR014" H 5000 3500 50  0001 C CNN
 F 1 "GND" V 5005 3622 50  0000 R CNN
 F 2 "" H 5000 3750 50  0001 C CNN
