File: PEE50_MPPT/PEE50_MPPT.kicad_pcb (KiCad board)
At the start: 2 copper layers, 100 x 100 mm, 161 parts, among them J3 Conn_01x02_Female, J7 Conn_01x02_Female, J8 Conn_01x03_Female, Q1 BC547, Q2 BC547, Q3 BC547, Q4 BC547, U1 LM3480-3.3, U10 TPS552882QRPMRQ1, U11 MAX44284FAUT+T, U12 MAX44284FAUT+T, U13 CSD18514Q5A, U14 CSD18543Q3A, U15 TPS552882QRPMRQ1, U16 MAX44284FAUT+T, U17 MAX44284FAUT+T, U18 CSD18514Q5A, U19 CSD18543Q3A, U2 CSD18514Q5A, U20 TPS552882QRPMRQ1, U21 MAX44284FAUT+T, U22 MAX44284FAUT+T, U23 ADG706BRUZ, U24 NTA4151PT1G, U3 CSD18543Q3A, U4 TPS552882QRPMRQ1, U5 MSP430FR2353TDBT, U6 MAX44284FAUT+T, U7 MAX44284FAUT+T, U8 CSD18514Q5A, U9 CSD18543Q3A

Commit message: eerste MPPT gelay-out + een aantal sporen gelegd
Parts:
- added J1: PV_IN1, Connector_Phoenix_MSTB:PhoenixContact_MSTBA_2,5_2-G-5,08_1x02_P5.08mm_Horizontal, F.Cu at (105.4, 111.6)
- added J2: PV_IN2, Connector_Phoenix_MSTB:PhoenixContact_MSTBA_2,5_2-G-5,08_1x02_P5.08mm_Horizontal, F.Cu at (140.1, 75.5)
- added J4: Vout, Connector_Phoenix_MSTB:PhoenixContact_MSTBA_2,5_2-G-5,08_1x02_P5.08mm_Horizontal, F.Cu at (153.3, 62.0)
- added J5: PV_IN4, Connector_Phoenix_MSTB:PhoenixContact_MSTBA_2,5_2-G-5,08_1x02_P5.08mm_Horizontal, F.Cu at (166.5, 62.0)
- added J6: PV_IN3, Connector_Phoenix_MSTB:PhoenixContact_MSTBA_2,5_2-G-5,08_1x02_P5.08mm_Horizontal, F.Cu at (153.3, 75.5)
- moved L1 189.1 mm to (135.8, 111.0)
- moved R38 185.1 mm to (128.9, 136.4)
- moved C6 180.6 mm to (129.2, 131.3), turned to 180 degrees
- moved C4 176.5 mm to (113.7, 112.9), turned to 90 degrees
- moved R34 174.6 mm to (108.5, 131.5), turned to 270 degrees
- moved R39 164.2 mm to (126.4, 140.2)
- moved C10 156.4 mm to (119.6, 135.2), turned to 270 degrees
- moved R37 156.2 mm to (125.0, 131.1), turned to 270 degrees
- moved U4 155.1 mm to (118.5, 130.0)
- moved C9 154.3 mm to (122.2, 135.1), turned to 270 degrees
- moved C12 153.8 mm to (117.2, 135.2), turned to 270 degrees
- moved C11 152.7 mm to (124.8, 136.4), turned to 90 degrees
- moved U2 152.5 mm to (116.5, 122.0), turned to 180 degrees
- moved C13 151.5 mm to (114.4, 135.2), turned to 270 degrees
- moved R33 150.7 mm to (119.3, 116.4), turned to 90 degrees
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Routing:
- net /DC/DC_Converter/PVin+: track 0.00 -> 27.0 mm
- net Net-(C6-Pad1): track 0.00 -> 14.1 mm
- net /DC/DC_Converter/ISP: track 0.00 -> 8.04 mm
- net /current_Sense/R+: track 0.00 -> 5.97 mm
- net /DC/DC_Converter/FB: track 0.00 -> 3.10 mm
- net Net-(R31-Pad2): track 0.00 -> 3.06 mm
- net Net-(C11-Pad1): track 0.00 -> 2.44 mm
- net Net-(R33-Pad1): track 0.00 -> 1.98 mm
- net Pgnd: track 0.00 -> 0.95 mm
Other:
- net class power added: clearance 0.2, trace_width 1, via_dia 0.8, via_drill 0.4

Commit message: push
Routing:
- net Pgnd: track 0.95 -> 33.2 mm
- net /current_Sense/R+: track 5.97 -> 12.8 mm
Changed lines of the file:
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@@
-(kicad_pcb (version 20171130) (host pcbnew "(5.0.0)")
+(kicad_pcb (version 20171130) (host pcbnew "(5.1.5)-3")
   (general
     (thickness 1.6)
     (drawings 4)
-    (tracks 32)
+    (tracks 43)
     (zones 0)
     (modules 166)
@@
     (zone_45_only no)
     (trace_min 0.2)
-    (segment_width 0.2)
-    (edge_width 0.15)
     (via_size 0.8)
     (via_drill 0.4)
@@
     (uvia_min_size 0.2)
     (uvia_min_drill 0.1)
+    (edge_width 0.15)
+    (segment_width 0.2)
     (pcb_text_width 0.3)
     (pcb_text_size 1.5 1.5)
@@
     (pad_to_mask_clearance 0.2)
     (aux_axis_origin 0 0)
-    (visible_elements FFFFFF7F)
+    (visible_elements 7FFFFFFF)
     (pcbplotparams
       (layerselection 0x010fc_ffffffff)
@@
   (gr_line (start 100 100) (end 200 100) (layer Edge.Cuts) (width 0.15))
   (segment (start 122.976998 127.025999) (end 123.926001 127.025999) (width 1) (layer F.Cu) (net 1))
+  (segment (start 105.591 111.452) (end 105.41 111.633) (width 1) (layer F.Cu) (net 1))
+  (segment (start 116.586 111.452) (end 105.591 111.452) (width 1) (layer F.Cu) (net 1))
+  (segment (start 108.21 111.633) (end 109.343 110.5) (width 1) (layer F.Cu) (net 1))
+  (segment (start 105.41 111.633) (end 108.21 111.633) (width 1) (layer F.Cu) (net 1))
+  (segment (start 109.343 110.5) (end 116.95 110.5) (width 1) (layer F.Cu) (net 1))
+  (segment (start 108.21 111.633) (end 108.857 112.28) (width 1) (layer F.Cu) (net 1))
+  (segment (start 108.857 112.28) (end 116.98 112.28) (width 1) (layer F.Cu) (net 1))
   (segment (start 110.871 114.427) (end 116.586 114.427) (width 1) (layer F.Cu) (net 4))
   (segment (start 108.29 122.755) (end 108.363 122.682) (width 1) (layer F.Cu) (net 4))
@@
   (segment (start 139.954 133.095) (end 139.954 131.699) (width 1) (layer F.Cu) (net 48))
   (segment (start 105.41 116.713) (end 111.379 116.713) (width 1) (layer F.Cu) (net 58))
+  (segment (start 105.41 116.713) (end 107.573 116.713) (width 1) (layer F.Cu) (net 58))
+  (segment (start 107.573 116.713) (end 108.35 117.49) (width 1) (layer F.Cu) (net 58))
+  (segment (start 108.35 117.49) (end 109.7735 117.49) (width 1) (layer F.Cu) (net 58))
+  (segment (start 109.7735 117.49) (end 111.93 117.49) (width 1) (layer F.Cu) (net 58))
   (segment (start 104.521 125.6935) (end 107.5325 125.6935) (width 1) (layer F.Cu) (net 72))
   (segment (start 107.5325 125.6935) (end 107.569 125.73) (width 1) (layer F.Cu) (net 72))

Commit message: best veel al gedaan voor 1e mppt
Parts:
- U14, U19, U3, U9: footprint AudioProject:CSD18543Q3A -> Robin_Lib:DNH0008A
- moved U6 103.3 mm to (114.7, 116.8), turned to 270 degrees
- moved U9 89.8 mm to (69.0, 152.7)
- moved R13 71.1 mm to (119.1, 137.8), turned to 90 degrees
- moved U14 61.1 mm to (87.7, 145.5)
- moved U19 42.3 mm to (78.5, 152.7)
- moved U24 27.5 mm to (121.8, 149.6), turned to 180 degrees
- moved R9 24.9 mm to (117.2, 144.9)
- moved R67 22.6 mm to (125.9, 149.7), turned to 0 degrees
- moved Q1 21.1 mm to (121.3, 144.9), turned to 0 degrees
- moved R7 11.6 mm to (126.7, 144.4), turned to 270 degrees
- moved C9 10.9 mm to (114.2, 142.5), turned to 180 degrees
- moved C7 8.13 mm to (122.6, 130.0)
- moved C3 7.91 mm to (111.0, 105.0)
- moved C4 7.47 mm to (114.9, 105.6)
- moved C5 7.47 mm to (117.9, 105.6)
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Routing:
- net /DC/DC_Converter/ISP: track 8.04 -> 61.6 mm
- net Pgnd: track 33.2 -> 0.26 mm
- net Net-(C6-Pad1): track 14.1 -> 45.2 mm
- net /DC/DC_Converter/FB: track 3.10 -> 21.3 mm
- net Net-(R37-Pad2): track 0.00 -> 14.7 mm, vias 0 -> 2
- net Net-(R38-Pad1): track 0.00 -> 11.8 mm, vias 0 -> 2
- net Net-(R31-Pad2): track 3.06 -> 14.4 mm
- net /DC/DC_Converter/ISN: track 0.00 -> 10.4 mm
- net Net-(R34-Pad1): track 0.00 -> 9.98 mm
- net Net-(C11-Pad2): track 0.00 -> 8.69 mm
- net Net-(R36-Pad1): track 0.00 -> 6.62 mm
- net DAC1: track 0.00 -> 6.04 mm
- net Net-(R37-Pad1): track 0.00 -> 5.41 mm
- net Net-(Q1-Pad3): track 0.00 -> 5.36 mm
- net Net-(R67-Pad1): track 0.00 -> 5.26 mm
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
Commit message: 1e MPPT lijkt af, nou maar hopen dat copy + paste werkt
Parts:
- moved U7 145.6 mm to (124.0, 137.2), turned to 270 degrees
- moved C4 22.8 mm to (101.7, 124.2), turned to 270 degrees
- moved C3 20.4 mm to (110.1, 125.4), turned to 270 degrees
- moved R39 8.51 mm to (134.9, 139.4), turned to 90 degrees
- moved C11 7.73 mm to (131.1, 141.0), turned to 180 degrees
- moved C5 5.93 mm to (116.8, 111.4)
- moved L1 5.09 mm to (139.3, 114.7), turned to 270 degrees
- moved R38 2.26 mm to (131.1, 136.9), turned to 90 degrees
- moved R9 1.98 mm to (115.7, 146.2), turned to 270 degrees
- moved C8 0.81 mm to (121.0, 126.1)
Routing:
- net Net-(C6-Pad1): track 45.2 -> 178.3 mm
- net Net-(R33-Pad2): track 0.00 -> 17.1 mm, vias 0 -> 2
- net Net-(C6-Pad2): track 0.00 -> 15.7 mm, vias 0 -> 2
- net /DC/DC_Converter/PVin+: track 25.1 -> 39.7 mm
- net Net-(C8-Pad2): track 1.32 -> 12.5 mm
- net Net-(C11-Pad2): track 8.69 -> 17.4 mm
- net /DC/DC_Converter/FB: track 21.3 -> 29.2 mm, vias 0 -> 2
- net Net-(R38-Pad1): track 11.8 -> 16.9 mm
- net /DC/DC_Converter/ISN: track 10.4 -> 15.1 mm, vias 0 -> 2
- net Net-(C8-Pad1): track 0.59 -> 4.25 mm
- net /DC/DC_Converter/ISP: track 61.6 -> 64.6 mm
- net +3V3: track 2.92 -> 5.83 mm
- net /current_Sense/R+: track 17.2 -> 19.6 mm
- net Net-(R31-Pad2): track 14.4 -> 14.9 mm
Other:
- net class power: trace_width 1 -> 0.5

Commit message: maar opnieuw begonnen met mppt layouten ivm plugin regels
Parts:
- added R68: 1, Resistor_SMD:R_1206_3216Metric_Pad1.42x1.75mm_HandSolder, F.Cu at (141.2, 32.4)
- added R69: 21k, Resistor_SMD:R_1206_3216Metric_Pad1.42x1.75mm_HandSolder, F.Cu at (146.2, 25.8)
- added R70: 13k, Resistor_SMD:R_1206_3216Metric_Pad1.42x1.75mm_HandSolder, F.Cu at (136.3, 34.7)
- added U25: TPS552882QRPMRQ1, Robin_Lib:RPM0026A-MFG, F.Cu at (136.9, 24.1)
- added U26: MAX44284FAUT+T, Robin_Lib:21-0058I_MXM, F.Cu at (194.7, 27.1)
- added U27: MAX44284FAUT+T, Robin_Lib:21-0058I_MXM, F.Cu at (194.7, 18.3)
- C10, C19, C23, C32, C36, C45, C49: value 10u -> 100n
- C11: value 100n -> 4u7
- C12: value 39u -> 100n
- C13, C26, C27, C39, C40, C52, C53: value 39u -> 10u
- C14: value C -> 10u
- C16, C29, C42, C55, C56: value 100n -> 39u
- C17, C30, C43: value 150u -> 39u
- C18, C31, C4, C44: value 150u -> 100n
- C20, C33, C46, C8: value 100n -> 150u
- C21, C34, C47, C7: value 4u7 -> 150u
- C22, C35, C48: value 100n -> 10u
- C24, C37, C50: value 10u -> 4u7
- C3: value 150u -> 1u
- C5: value 10u -> C
- C57: value 1u -> 100n
- J1: value PV_IN1 -> Vout
- J2: value PV_IN2 -> Conn_01x02_Female; footprint Connector_Phoenix_MSTB:PhoenixContact_MSTBA_2,5_2-G-5,08_1x02_P5.08mm_Horizontal -> Connector_PinSocket_2.54mm:PinSocket_1x02_P2.54mm_Vertical
- J4: value Vout -> Conn_01x03_Female; footprint Connector_Phoenix_MSTB:PhoenixContact_MSTBA_2,5_2-G-5,08_1x02_P5.08mm_Horizontal -> Connector_PinSocket_2.54mm:PinSocket_1x03_P2.54mm_Vertical
- J5: value PV_IN4 -> PV_IN1
- J6: value PV_IN3 -> PV_IN1
- J7: value Conn_01x02_Female -> PV_IN1; footprint Connector_PinSocket_2.54mm:PinSocket_1x02_P2.54mm_Vertical -> Connector_Phoenix_MSTB:PhoenixContact_MSTBA_2,5_2-G-5,08_1x02_P5.08mm_Horizontal
- J8: value Conn_01x03_Female -> PV_IN1; footprint Connector_PinSocket_2.54mm:PinSocket_1x03_P2.54mm_Vertical -> Connector_Phoenix_MSTB:PhoenixContact_MSTBA_2,5_2-G-5,08_1x02_P5.08mm_Horizontal
- R10, R22: value R -> 0.01; footprint Resistor_SMD:R_1206_3216Metric_Pad1.42x1.75mm_HandSolder -> Resistor_SMD:R_2512_6332Metric_Pad1.52x3.35mm_HandSolder
- R11: value 10k -> 383k
- R12, R67: value R -> 100k
- R13, R17: value 0.01 -> 1; footprint Resistor_SMD:R_2512_6332Metric_Pad1.52x3.35mm_HandSolder -> Resistor_SMD:R_1206_3216Metric_Pad1.42x1.75mm_HandSolder
- R14: value 0.01 -> 100k; footprint Resistor_SMD:R_2512_6332Metric_Pad1.52x3.35mm_HandSolder -> Resistor_SMD:R_1206_3216Metric_Pad1.42x1.75mm_HandSolder
- R15: value 180k -> 66.5k
- R16: value 20k -> 100k
- R18: value 0.01 -> 21k; footprint Resistor_SMD:R_2512_6332Metric_Pad1.52x3.35mm_HandSolder -> Resistor_SMD:R_1206_3216Metric_Pad1.42x1.75mm_HandSolder
- R19: value 10k -> 13k
- R20: value R -> 180k
- R21: value 10k -> 20k
- R24, R7: value R -> 10k
- R25, R26, R6: value 0.01 -> R; footprint Resistor_SMD:R_2512_6332Metric_Pad1.52x3.35mm_HandSolder -> Resistor_SMD:R_1206_3216Metric_Pad1.42x1.75mm_HandSolder
- R27: value 180k -> 0.01; footprint Resistor_SMD:R_1206_3216Metric_Pad1.42x1.75mm_HandSolder -> Resistor_SMD:R_2512_6332Metric_Pad1.52x3.35mm_HandSolder
- R28: value 20k -> 383k
- R29: value 180k -> 100k
- R30: value 20k -> 1
- R31: value 383k -> 100k
- R32: value 100k -> 66.5k
- R33, R46: value 1 -> 100k
- R34: value 100k -> 1
- R35: value 66.5k -> 21k
- R36: value 100k -> 13k
- R37: value 1 -> 180k
- R38: value 21k -> 20k
- R39: value 13k -> 0.01; footprint Resistor_SMD:R_1206_3216Metric_Pad1.42x1.75mm_HandSolder -> Resistor_SMD:R_2512_6332Metric_Pad1.52x3.35mm_HandSolder
- R40: value 383k -> R
- R41: value 100k -> 10k
- R42, R60: value 1 -> R
- R43, R59: value 100k -> R
- R44: value 66.5k -> 0.01; footprint Resistor_SMD:R_1206_3216Metric_Pad1.42x1.75mm_HandSolder -> Resistor_SMD:R_2512_6332Metric_Pad1.52x3.35mm_HandSolder
- R45: value 100k -> 383k
- R47: value 21k -> 1
- R48: value 13k -> 100k
- R49: value 383k -> 66.5k
- R52: value 100k -> 21k
- R53: value 66.5k -> 13k
- R54: value 100k -> 180k
- R55: value 1 -> 20k
- R56: value 21k -> 0.01; footprint Resistor_SMD:R_1206_3216Metric_Pad1.42x1.75mm_HandSolder -> Resistor_SMD:R_2512_6332Metric_Pad1.52x3.35mm_HandSolder
- R57: value 13k -> R
- R58: value 383k -> 10k
- R61: value 100k -> 0.01; footprint Resistor_SMD:R_1206_3216Metric_Pad1.42x1.75mm_HandSolder -> Resistor_SMD:R_2512_6332Metric_Pad1.52x3.35mm_HandSolder
- R62: value 66.5k -> 383k
- R65: value 21k -> 100k
- R66: value 13k -> 66.5k
- R9: value 10k -> R
- U10, U4: value TPS552882QRPMRQ1 -> NTA4151PT1G; footprint AudioProject:TPS552882QRPMRQ1 -> AudioProject:NTA4151PT1G
- U11, U17: value MAX44284FAUT+T -> CSD18514Q5A; footprint Robin_Lib:21-0058I_MXM -> Robin_Lib:DQJ0008A
- U12, U6: value MAX44284FAUT+T -> CSD18543Q3A; footprint Robin_Lib:21-0058I_MXM -> Robin_Lib:DNH0008A
- U13: value CSD18514Q5A -> TPS552882QRPMRQ1; footprint AudioProject:CSD18514Q5A -> Robin_Lib:RPM0026A-MFG
- U14, U9: value CSD18543Q3A -> MAX44284FAUT+T; footprint Robin_Lib:DNH0008A -> Robin_Lib:21-0058I_MXM
- U15, U20: value TPS552882QRPMRQ1 -> MAX44284FAUT+T; footprint AudioProject:TPS552882QRPMRQ1 -> Robin_Lib:21-0058I_MXM
- U16: value MAX44284FAUT+T -> NTA4151PT1G; footprint Robin_Lib:21-0058I_MXM -> AudioProject:NTA4151PT1G
- U18: value CSD18514Q5A -> CSD18543Q3A; footprint AudioProject:CSD18514Q5A -> Robin_Lib:DNH0008A
- U19: value CSD18543Q3A -> TPS552882QRPMRQ1; footprint Robin_Lib:DNH0008A -> Robin_Lib:RPM0026A-MFG
- U2: value CSD18514Q5A -> MSP430FR2353TDBT; footprint AudioProject:CSD18514Q5A -> Robin_Lib:DBT38_TEX
- U21: footprint AudioProject:MAX44284FAUT&plus_T -> Robin_Lib:21-0058I_MXM
- U22: value MAX44284FAUT+T -> NTA4151PT1G; footprint AudioProject:MAX44284FAUT&plus_T -> AudioProject:NTA4151PT1G
- U23: value ADG706BRUZ -> CSD18514Q5A; footprint AudioProject:ADG706BRUZ -> Robin_Lib:DQJ0008A
- U24: value NTA4151PT1G -> CSD18543Q3A; footprint AudioProject:NTA4151PT1G -> Robin_Lib:DNH0008A
- U3: value CSD18543Q3A -> ADG706BRUZ; footprint Robin_Lib:DNH0008A -> AudioProject:ADG706BRUZ
- U5: value MSP430FR2353TDBT -> CSD18514Q5A; footprint Robin_Lib:DBT38_TEX -> Robin_Lib:DQJ0008A
- U7: value MAX44284FAUT+T -> TPS552882QRPMRQ1; footprint Robin_Lib:21-0058I_MXM -> Robin_Lib:RPM0026A-MFG
- U8: value CSD18514Q5A -> MAX44284FAUT+T; footprint AudioProject:CSD18514Q5A -> Robin_Lib:21-0058I_MXM
- moved J8 260.0 mm to (161.4, 37.7)
- moved U10 244.5 mm to (177.8, 30.1)
- moved U23 240.5 mm to (137.2, 19.2)
- moved C56 225.3 mm to (136.4, 29.7)
- moved C49 215.4 mm to (147.9, 17.7)
- moved U22 211.0 mm to (177.8, 48.4)
- moved U20 206.8 mm to (194.7, 35.9)
- moved R57 204.3 mm to (173.0, 43.7)
- moved C54 203.7 mm to (136.4, 32.0)
- moved C46 203.5 mm to (142.9, 19.9)
- moved R65 202.7 mm to (146.2, 29.0)
- moved C55 201.3 mm to (141.4, 27.4)
- moved R46 200.3 mm to (145.8, 63.6)
- moved U21 199.0 mm to (164.5, 69.1)
- moved R59 197.8 mm to (181.1, 40.7)
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Connections:
- C1 pad 1: Net-(C1-Pad1) -> +3V3
- C10 pad 1: /DC/DC_Converter/ISP -> Net-(C10-Pad1)
- C10 pad 2: Pgnd -> Net-(C10-Pad2)
- C11 pad 2: Net-(C11-Pad2) -> Pgnd
- C12 pad 1: /DC/DC_Converter/ISP -> Net-(C12-Pad1)
- C12 pad 2: Pgnd -> Net-(C12-Pad2)
- C13 pad 1: /DC/DC_Converter/ISP -> /Sheet609B465C/sheet609C6964/ISP
- C14 pad 1: Net-(C14-Pad1) -> /Sheet609B465C/sheet609C6964/ISP
- C15 pad 1: +3V3 -> Net-(C15-Pad1)
- C15 pad 2: Pgnd -> Net-(C15-Pad2)
- C16 pad 1: +3V3 -> /Sheet609B465C/sheet609C6964/ISP
- C17 pad 1: /sheet608C3AAC/PVin+ -> /Sheet609B465C/sheet609C6964/ISP
- C18 pad 1: /sheet608C3AAC/PVin+ -> +3V3
- C19 pad 1: /sheet608C3AAC/PVin+ -> +3V3
- C20 pad 1: Net-(C20-Pad1) -> /sheet609F26BA/sheet609C6964/PVin+
- C20 pad 2: Net-(C20-Pad2) -> Pgnd
- C21 pad 1: Net-(C21-Pad1) -> /sheet609F26BA/sheet609C6964/PVin+
- C22 pad 1: Net-(C22-Pad1) -> /sheet609F26BA/sheet609C6964/PVin+
- C22 pad 2: Net-(C22-Pad2) -> Pgnd
- C23 pad 1: /sheet608C3AAC/ISP -> Net-(C23-Pad1)
- C23 pad 2: Pgnd -> Net-(C23-Pad2)
- C24 pad 1: /sheet608C3AAC/ISP -> Net-(C24-Pad1)
- C26 pad 1: /sheet608C3AAC/ISP -> /sheet609F26BA/sheet609C6964/ISP
- C27 pad 1: /sheet608C3AAC/ISP -> /sheet609F26BA/sheet609C6964/ISP
- C28 pad 1: +3V3 -> Net-(C28-Pad1)
- C28 pad 2: Pgnd -> Net-(C28-Pad2)
- C29 pad 1: +3V3 -> /sheet609F26BA/sheet609C6964/ISP
- C3 pad 1: /DC/DC_Converter/PVin+ -> Net-(C3-Pad1)
- C30 pad 1: /sheet608C70A5/PVin+ -> /sheet609F26BA/sheet609C6964/ISP
- C31 pad 1: /sheet608C70A5/PVin+ -> +3V3
- C32 pad 1: /sheet608C70A5/PVin+ -> +3V3
- C33 pad 1: Net-(C33-Pad1) -> /sheet609F4756/sheet609C6964/PVin+
- C33 pad 2: Net-(C33-Pad2) -> Pgnd
- C34 pad 1: Net-(C34-Pad1) -> /sheet609F4756/sheet609C6964/PVin+
- C35 pad 1: Net-(C35-Pad1) -> /sheet609F4756/sheet609C6964/PVin+
- C35 pad 2: Net-(C35-Pad2) -> Pgnd
- C36 pad 1: /sheet608C70A5/ISP -> Net-(C36-Pad1)
- C36 pad 2: Pgnd -> Net-(C36-Pad2)
- C37 pad 1: /sheet608C70A5/ISP -> Net-(C37-Pad1)
- C39 pad 1: /sheet608C70A5/ISP -> /sheet609F4756/sheet609C6964/ISP
- C4 pad 1: /DC/DC_Converter/PVin+ -> +3V3
- C40 pad 1: /sheet608C70A5/ISP -> /sheet609F4756/sheet609C6964/ISP
- C41 pad 1: +3V3 -> Net-(C41-Pad1)
- C41 pad 2: Pgnd -> Net-(C41-Pad2)
- C42 pad 1: +3V3 -> /sheet609F4756/sheet609C6964/ISP
- C43 pad 1: /sheet608DD8EC/PVin+ -> /sheet609F4756/sheet609C6964/ISP
- C44 pad 1: /sheet608DD8EC/PVin+ -> +3V3
- C45 pad 1: /sheet608DD8EC/PVin+ -> +3V3
- C46 pad 1: Net-(C46-Pad1) -> /sheet609F5795/sheet609C6964/PVin+
- C46 pad 2: Net-(C46-Pad2) -> Pgnd
- C47 pad 1: Net-(C47-Pad1) -> /sheet609F5795/sheet609C6964/PVin+
- C48 pad 1: Net-(C48-Pad1) -> /sheet609F5795/sheet609C6964/PVin+
- C48 pad 2: Net-(C48-Pad2) -> Pgnd
- C49 pad 1: /sheet608DD8EC/ISP -> Net-(C49-Pad1)
- C49 pad 2: Pgnd -> Net-(C49-Pad2)
- C5 pad 1: /DC/DC_Converter/PVin+ -> Net-(C5-Pad1)
- C50 pad 1: /sheet608DD8EC/ISP -> Net-(C50-Pad1)
- C52 pad 1: /sheet608DD8EC/ISP -> /sheet609F5795/sheet609C6964/ISP
- C53 pad 1: /sheet608DD8EC/ISP -> /sheet609F5795/sheet609C6964/ISP
- C54 pad 1: +3V3 -> Net-(C54-Pad1)
- C54 pad 2: Pgnd -> Net-(C54-Pad2)
- C55 pad 1: +3V3 -> /sheet609F5795/sheet609C6964/ISP
- C56 pad 1: +3V3 -> /sheet609F5795/sheet609C6964/ISP
- C6 pad 1: Net-(C6-Pad1) -> +3V3
- C6 pad 2: Net-(C6-Pad2) -> Pgnd
- C7 pad 1: Net-(C7-Pad1) -> /Sheet609B465C/sheet609C6964/PVin+
- C8 pad 1: Net-(C8-Pad1) -> /Sheet609B465C/sheet609C6964/PVin+
- C8 pad 2: Net-(C8-Pad2) -> Pgnd
- C9 pad 1: /DC/DC_Converter/ISP -> /Sheet609B465C/sheet609C6964/PVin+
- J1 pad 1: Pgnd -> /Sheet609B465C/Vout
- J1 pad 2: /current_Sense/R+ -> Pgnd
- J2 pad 1: Pgnd -> +12V
- J2 pad 2: /sheet608C3AAE/R+ -> Pgnd
- J3 pad 1: +12V -> Net-(J3-Pad1)
- J3 pad 2: Pgnd -> Net-(J3-Pad2)
- J4 pad 1: /DC/DC_Converter/ISN -> Net-(J4-Pad1)
- J4 pad 2: Pgnd -> Net-(J4-Pad2)
- J5 pad 2: /sheet608C70A6/R+ -> /Sheet609B465C/sheet609C6965/R+
- J6 pad 2: /sheet608DD8ED/R+ -> /sheet609F26BA/sheet609C6965/R+
- J7 pad 1: Net-(J7-Pad1) -> Pgnd
- J7 pad 2: Net-(J7-Pad2) -> /sheet609F4756/sheet609C6965/R+
- J8 pad 1: Net-(J8-Pad1) -> Pgnd
- J8 pad 2: Net-(J8-Pad2) -> /sheet609F5795/sheet609C6965/R+
- JP1 pad 3: Net-(C1-Pad1) -> Net-(C3-Pad1)
- L1 pad 1: Net-(C6-Pad1) -> Net-(C10-Pad1)
- L1 pad 2: Net-(C8-Pad2) -> Net-(C12-Pad2)
- L2 pad 1: Net-(C20-Pad1) -> Net-(C23-Pad1)
- L2 pad 2: Net-(C22-Pad2) -> Net-(C25-Pad2)
- L3 pad 1: Net-(C33-Pad1) -> Net-(C36-Pad1)
- L3 pad 2: Net-(C35-Pad2) -> Net-(C38-Pad2)
- L4 pad 1: Net-(C46-Pad1) -> Net-(C49-Pad1)
- L4 pad 2: Net-(C48-Pad2) -> Net-(C51-Pad2)
- Q1 pad 1: /DC/DC_Converter/FB -> /Sheet609B465C/sheet609C6964/FB
- Q2 pad 1: /sheet608C3AAC/FB -> /sheet609F26BA/sheet609C6964/FB
- Q3 pad 1: /sheet608C70A5/FB -> /sheet609F4756/sheet609C6964/FB
- Q4 pad 1: /sheet608DD8EC/FB -> /sheet609F5795/sheet609C6964/FB
- R1 pad 1: /current_Sense/R+ -> /Sheet609B465C/Vout
- R1 pad 2: Vpv1 -> Vout
- R10 pad 1: Net-(Q1-Pad3) -> /Sheet609B465C/Vout
- R10 pad 2: Pgnd -> /Sheet609B465C/sheet609C6964/ISP
- R11 pad 1: /sheet608C3AAC/ISP -> /Sheet609B465C/sheet609C6964/PVin+
- R11 pad 2: /sheet608C3AAC/FB -> Net-(R11-Pad2)
- R12 pad 1: Net-(Q2-Pad3) -> Net-(R11-Pad2)
- R13 pad 1: /DC/DC_Converter/ISN -> Net-(R13-Pad1)
- R13 pad 2: /DC/DC_Converter/ISP -> Net-(R13-Pad2)
- R14 pad 1: /DC/DC_Converter/ISN -> Net-(R14-Pad1)
- R14 pad 2: /sheet608C3AAC/ISP -> Pgnd
- R15 pad 1: /DC/DC_Converter/ISN -> Net-(R15-Pad1)
- R15 pad 2: Vout -> Pgnd
- R16 pad 1: Vout -> Net-(R16-Pad1)
- R17 pad 1: /DC/DC_Converter/ISN -> Net-(R17-Pad1)
- R17 pad 2: /sheet608C70A5/ISP -> Net-(R17-Pad2)
- R18 pad 1: /DC/DC_Converter/ISN -> Net-(R18-Pad1)
- R18 pad 2: /sheet608DD8EC/ISP -> Pgnd
- R19 pad 1: /sheet608C70A5/ISP -> Net-(C15-Pad1)
- R19 pad 2: /sheet608C70A5/FB -> Pgnd
- R2 pad 1: Vpv1 -> Vout
- R20 pad 1: Net-(Q3-Pad3) -> /sheet609F26BA/sheet609C6965/R+
- R20 pad 2: Pgnd -> Vpv1
- R21 pad 1: /sheet608DD8EC/ISP -> Vpv1
- R21 pad 2: /sheet608DD8EC/FB -> Pgnd
- R22 pad 1: Net-(Q4-Pad3) -> /sheet609F26BA/sheet609C6964/PVin+
- R22 pad 2: Pgnd -> /sheet609F26BA/sheet609C6965/R+
- R23 pad 1: Net-(Q3-Pad2) -> Net-(Q2-Pad2)
- R23 pad 2: DAC4 -> DAC1
- R24 pad 1: Net-(Q4-Pad2) -> /sheet609F26BA/sheet609C6964/ISP
- R24 pad 2: DAC3 -> /sheet609F26BA/sheet609C6964/FB
- R25 pad 1: /sheet608C70A5/PVin+ -> Net-(Q2-Pad3)
- R25 pad 2: /sheet608C70A6/R+ -> Pgnd
- R26 pad 1: /sheet608DD8EC/PVin+ -> Net-(R26-Pad1)
- R26 pad 2: /sheet608DD8ED/R+ -> Pgnd
- R27 pad 1: /sheet608C70A6/R+ -> /Sheet609B465C/Vout
- R27 pad 2: Vpv4 -> /sheet609F26BA/sheet609C6964/ISP
- R28 pad 1: Vpv4 -> /sheet609F26BA/sheet609C6964/PVin+
- R28 pad 2: Pgnd -> Net-(R28-Pad2)
- R29 pad 1: /sheet608DD8ED/R+ -> Net-(R28-Pad2)
- R29 pad 2: Vpv3 -> Pgnd
- R3 pad 1: /sheet608C3AAE/R+ -> /Sheet609B465C/sheet609C6965/R+
- R3 pad 2: Vpv2 -> Vpv1
- R30 pad 1: Vpv3 -> Net-(R30-Pad1)
- R30 pad 2: Pgnd -> Net-(R30-Pad2)
- R31 pad 1: /DC/DC_Converter/PVin+ -> Net-(R31-Pad1)
- R31 pad 2: Net-(R31-Pad2) -> Pgnd
- R32 pad 1: Net-(R31-Pad2) -> Net-(R32-Pad1)
- R33 pad 2: Net-(R33-Pad2) -> Pgnd
- R34 pad 2: Pgnd -> Net-(R34-Pad2)
- R36 pad 1: Net-(R36-Pad1) -> Net-(C28-Pad1)
- R37 pad 1: Net-(R37-Pad1) -> /sheet609F4756/sheet609C6965/R+
- R37 pad 2: Net-(R37-Pad2) -> Vpv1
- R38 pad 1: Net-(R38-Pad1) -> Vpv1
- R39 pad 1: Net-(C11-Pad1) -> /sheet609F4756/sheet609C6964/PVin+
- R39 pad 2: Pgnd -> /sheet609F4756/sheet609C6965/R+
- R4 pad 1: Vpv2 -> Vpv1
- R40 pad 1: /sheet608C3AAC/PVin+ -> Net-(Q3-Pad2)
- R40 pad 2: Net-(R40-Pad2) -> DAC1
- R41 pad 1: Net-(R40-Pad2) -> /sheet609F4756/sheet609C6964/ISP
- R41 pad 2: Pgnd -> /sheet609F4756/sheet609C6964/FB
- R42 pad 1: Net-(R42-Pad1) -> Net-(Q3-Pad3)
- R42 pad 2: Net-(R42-Pad2) -> Pgnd
- R44 pad 1: Net-(R44-Pad1) -> /Sheet609B465C/Vout
- R44 pad 2: Pgnd -> /sheet609F4756/sheet609C6964/ISP
- R45 pad 1: Net-(R45-Pad1) -> /sheet609F4756/sheet609C6964/PVin+
- R45 pad 2: Pgnd -> Net-(R45-Pad2)
- R46 pad 1: Net-(R46-Pad1) -> Net-(R45-Pad2)
- R46 pad 2: Net-(R46-Pad2) -> Pgnd
- R47 pad 2: Pgnd -> Net-(R47-Pad2)
- R48 pad 1: Net-(C25-Pad1) -> Net-(R48-Pad1)
- R49 pad 1: /sheet608C70A5/PVin+ -> Net-(R49-Pad1)
- R49 pad 2: Net-(R49-Pad2) -> Pgnd
- R5 pad 1: /DC/DC_Converter/PVin+ -> /Sheet609B465C/sheet609C6964/PVin+
- R5 pad 2: /current_Sense/R+ -> /Sheet609B465C/sheet609C6965/R+
- R50 pad 1: Net-(R49-Pad2) -> Net-(R50-Pad1)
- R53 pad 1: Net-(R53-Pad1) -> Net-(C41-Pad1)
- R54 pad 1: Net-(R54-Pad1) -> /sheet609F5795/sheet609C6965/R+
- R54 pad 2: Pgnd -> Vpv1
- R55 pad 1: Net-(R55-Pad1) -> Vpv1
- R55 pad 2: Net-(R55-Pad2) -> Pgnd
- R56 pad 1: Net-(R56-Pad1) -> /sheet609F5795/sheet609C6964/PVin+
- R56 pad 2: Pgnd -> /sheet609F5795/sheet609C6965/R+
- R57 pad 1: Net-(C38-Pad1) -> Net-(Q4-Pad2)
- R57 pad 2: Pgnd -> DAC1
- R58 pad 1: /sheet608DD8EC/PVin+ -> /sheet609F5795/sheet609C6964/ISP
- R58 pad 2: Net-(R58-Pad2) -> /sheet609F5795/sheet609C6964/FB
- R59 pad 1: Net-(R58-Pad2) -> Net-(Q4-Pad3)
- R6 pad 1: /sheet608C3AAC/PVin+ -> Net-(Q1-Pad2)
- R6 pad 2: /sheet608C3AAE/R+ -> DAC1
- R60 pad 2: Net-(R60-Pad2) -> Pgnd
- R61 pad 1: Net-(R61-Pad1) -> /Sheet609B465C/Vout
- R61 pad 2: Pgnd -> /sheet609F5795/sheet609C6964/ISP
- R62 pad 1: Net-(R62-Pad1) -> /sheet609F5795/sheet609C6964/PVin+
- R62 pad 2: Pgnd -> Net-(R62-Pad2)
- R63 pad 1: Net-(R63-Pad1) -> Net-(R62-Pad2)
- R66 pad 1: Net-(C51-Pad1) -> Net-(R66-Pad1)
- R7 pad 1: Net-(Q1-Pad2) -> /Sheet609B465C/sheet609C6964/ISP
- R7 pad 2: DAC1 -> /Sheet609B465C/sheet609C6964/FB
- R8 pad 1: Net-(Q2-Pad2) -> Net-(Q1-Pad3)
- R8 pad 2: DAC2 -> Pgnd
- R9 pad 1: /DC/DC_Converter/ISP -> Net-(R9-Pad1)
- R9 pad 2: /DC/DC_Converter/FB -> Pgnd
- U1 pad 2: Net-(C1-Pad1) -> Net-(C3-Pad1)
- U10 pad 1: Net-(R46-Pad2) -> DAC1
- U10 pad 2: Net-(R42-Pad2) -> /sheet609F26BA/sheet609C6964/FB
- U10 pad 3: /sheet608C3AAC/PVin+ -> Net-(R26-Pad1)
- U11 pad 1: +3V3 -> Net-(C23-Pad1)
- U11 pad 2: Pgnd -> Net-(C23-Pad1)
- U11 pad 3: /sheet608C3AAE/R+ -> Net-(C23-Pad1)
- U11 pad 4: /sheet608C3AAC/PVin+ -> Net-(R30-Pad1)
- U11 pad 5: Ipv2 -> /sheet609F26BA/sheet609C6964/PVin+
- U11 pad 6: +3V3 -> /sheet609F26BA/sheet609C6964/PVin+
- U12 pad 1: +3V3 -> Pgnd
- U12 pad 3: /sheet608C3AAC/ISP -> Pgnd
- U12 pad 4: /DC/DC_Converter/ISN -> Net-(R34-Pad1)
- U12 pad 5: Imppt2 -> Net-(C23-Pad1)
- U12 pad 6: +3V3 -> Net-(C23-Pad1)
- U13 pad 1: Net-(C33-Pad1) -> Net-(R34-Pad2)
- U13 pad 2: Net-(C33-Pad1) -> Net-(R30-Pad2)
- U13 pad 3: Net-(C33-Pad1) -> /sheet609F26BA/sheet609C6964/PVin+
- U13 pad 4: Net-(R51-Pad1) -> Net-(R28-Pad2)
- U13 pad 5: /sheet608C70A5/PVin+ -> Net-(R31-Pad1)
- U13 pad 6: /sheet608C70A5/PVin+ -> Net-(R33-Pad1)
- U13 pad 7: /sheet608C70A5/PVin+ -> Pgnd
- U13 pad 8: /sheet608C70A5/PVin+ -> Net-(R32-Pad1)
- U13 pad 9: /sheet608C70A5/PVin+ -> Pgnd
- U14 pad 1: Pgnd -> +3V3
- U14 pad 3: Pgnd -> /sheet609F26BA/sheet609C6965/R+
- U14 pad 4: Net-(R55-Pad1) -> /sheet609F26BA/sheet609C6964/PVin+
- U14 pad 5: Net-(C33-Pad1) -> Ipv1
- U14 pad 6: Net-(C33-Pad1) -> +3V3
- U15 pad 1: Net-(R55-Pad2) -> +3V3
- U15 pad 2: Net-(R51-Pad2) -> Pgnd
- U15 pad 3: /sheet608C70A5/PVin+ -> /sheet609F26BA/sheet609C6964/ISP
- U15 pad 4: Net-(R49-Pad2) -> /Sheet609B465C/Vout
- U15 pad 5: Net-(R52-Pad1) -> Imppt1
- U15 pad 6: Net-(R54-Pad1) -> +3V3
- U16 pad 1: +3V3 -> DAC1
- U16 pad 2: Pgnd -> /sheet609F4756/sheet609C6964/FB
- U16 pad 3: /sheet608C70A6/R+ -> Net-(R43-Pad1)
- U17 pad 1: +3V3 -> Net-(C36-Pad1)
- U17 pad 2: Pgnd -> Net-(C36-Pad1)
- U17 pad 3: /sheet608C70A5/ISP -> Net-(C36-Pad1)
- U17 pad 4: /DC/DC_Converter/ISN -> Net-(R47-Pad1)
- U17 pad 5: Imppt4 -> /sheet609F4756/sheet609C6964/PVin+
- U17 pad 6: +3V3 -> /sheet609F4756/sheet609C6964/PVin+
- U18 pad 1: Net-(C46-Pad1) -> Pgnd
- U18 pad 2: Net-(C46-Pad1) -> Pgnd
- U18 pad 3: Net-(C46-Pad1) -> Pgnd
- U18 pad 4: Net-(R60-Pad1) -> Net-(R51-Pad1)
- U18 pad 5: /sheet608DD8EC/PVin+ -> Net-(C36-Pad1)
- U18 pad 6: /sheet608DD8EC/PVin+ -> Net-(C36-Pad1)
- U18 pad 7: /sheet608DD8EC/PVin+ -> Net-(C36-Pad1)
- U18 pad 8: /sheet608DD8EC/PVin+ -> Net-(C36-Pad1)
- U18 pad 9: /sheet608DD8EC/PVin+ -> Net-(C36-Pad1)
- U19 pad 1: Pgnd -> Net-(R51-Pad2)
- U19 pad 2: Pgnd -> Net-(R47-Pad2)
- U19 pad 3: Pgnd -> /sheet609F4756/sheet609C6964/PVin+
- U19 pad 4: Net-(R64-Pad1) -> Net-(R45-Pad2)
- U19 pad 5: Net-(C46-Pad1) -> Net-(R48-Pad1)
- U19 pad 6: Net-(C46-Pad1) -> Net-(R50-Pad1)
- U19 pad 7: Net-(C46-Pad1) -> Pgnd
- U19 pad 8: Net-(C46-Pad1) -> Net-(R49-Pad1)
- U19 pad 9: Net-(C46-Pad1) -> Pgnd
- U2 pad 1: Net-(C6-Pad1) -> (no net)
- U2 pad 2: Net-(C6-Pad1) -> (no net)
- U2 pad 3: Net-(C6-Pad1) -> (no net)
- U2 pad 4: Net-(R33-Pad1) -> (no net)
- U2 pad 5: /DC/DC_Converter/PVin+ -> (no net)
- U2 pad 6: /DC/DC_Converter/PVin+ -> DAC1
- U2 pad 7: /DC/DC_Converter/PVin+ -> /uC_MPPT/ADC
- U2 pad 8: /DC/DC_Converter/PVin+ -> Net-(J4-Pad1)
- U2 pad 9: /DC/DC_Converter/PVin+ -> Net-(J4-Pad2)
- U20 pad 1: Net-(R64-Pad2) -> +3V3
- U20 pad 2: Net-(R60-Pad2) -> Pgnd
- U20 pad 3: /sheet608DD8EC/PVin+ -> /sheet609F4756/sheet609C6965/R+
- U20 pad 4: Net-(R58-Pad2) -> /sheet609F4756/sheet609C6964/PVin+
- U20 pad 5: Net-(R61-Pad1) -> Ipv1
- U20 pad 6: Net-(R63-Pad1) -> +3V3
- U21 pad 3: /sheet608DD8ED/R+ -> /sheet609F4756/sheet609C6964/ISP
- U21 pad 4: /sheet608DD8EC/PVin+ -> /Sheet609B465C/Vout
- U21 pad 5: Ipv3 -> Imppt1
- U22 pad 1: +3V3 -> DAC1
- U22 pad 2: Pgnd -> /sheet609F5795/sheet609C6964/FB
- U22 pad 3: /sheet608DD8EC/ISP -> Net-(R60-Pad1)
- U23 pad 1: +3V3 -> Net-(C49-Pad1)
- U23 pad 2: Net-(U23-Pad2) -> Net-(C49-Pad1)
- U23 pad 3: Net-(U23-Pad3) -> Net-(C49-Pad1)
- U23 pad 4: Net-(U23-Pad4) -> Net-(R64-Pad1)
- U23 pad 5: Net-(U23-Pad5) -> /sheet609F5795/sheet609C6964/PVin+
- U23 pad 6: Net-(U23-Pad6) -> /sheet609F5795/sheet609C6964/PVin+
- U23 pad 7: Vout -> /sheet609F5795/sheet609C6964/PVin+
- U23 pad 8: Imppt4 -> /sheet609F5795/sheet609C6964/PVin+
- U23 pad 9: Imppt3 -> /sheet609F5795/sheet609C6964/PVin+
- U24 pad 1: DAC1 -> Pgnd
- U24 pad 2: /DC/DC_Converter/FB -> Pgnd
- U24 pad 3: Net-(R67-Pad1) -> Pgnd
- U3 pad 1: Pgnd -> +3V3
- U3 pad 2: Pgnd -> (no net)
- U3 pad 3: Pgnd -> (no net)
- U3 pad 4: Net-(R37-Pad1) -> (no net)
- U3 pad 5: Net-(C6-Pad1) -> (no net)
- U3 pad 6: Net-(C6-Pad1) -> (no net)
- U3 pad 7: Net-(C6-Pad1) -> Vout
- U3 pad 8: Net-(C6-Pad1) -> (no net)
- U3 pad 9: Net-(C6-Pad1) -> (no net)
- U4 pad 1: Net-(R37-Pad2) -> DAC1
- U4 pad 2: Net-(R33-Pad2) -> /Sheet609B465C/sheet609C6964/FB
- U4 pad 3: /DC/DC_Converter/PVin+ -> Net-(R9-Pad1)
- U5 pad 1: Net-(U5-Pad1) -> Net-(C10-Pad1)
- U5 pad 2: DAC3 -> Net-(C10-Pad1)
- U5 pad 3: Net-(U5-Pad3) -> Net-(C10-Pad1)
- U5 pad 4: Net-(U5-Pad4) -> Net-(R13-Pad1)
- U5 pad 5: Net-(U5-Pad5) -> /Sheet609B465C/sheet609C6964/PVin+
- U5 pad 6: DAC1 -> /Sheet609B465C/sheet609C6964/PVin+
- U5 pad 7: /uC_MPPT/ADC -> /Sheet609B465C/sheet609C6964/PVin+
- U5 pad 8: Net-(J8-Pad1) -> /Sheet609B465C/sheet609C6964/PVin+
- U5 pad 9: Net-(J8-Pad2) -> /Sheet609B465C/sheet609C6964/PVin+
- U6 pad 1: +3V3 -> Pgnd
- U6 pad 3: /current_Sense/R+ -> Pgnd
- U6 pad 4: /DC/DC_Converter/PVin+ -> Net-(R17-Pad1)
- U6 pad 5: Ipv1 -> Net-(C10-Pad1)
- U6 pad 6: +3V3 -> Net-(C10-Pad1)
- U7 pad 1: +3V3 -> Net-(R17-Pad2)
- U7 pad 2: Pgnd -> Net-(R13-Pad2)
- U7 pad 3: /DC/DC_Converter/ISP -> /Sheet609B465C/sheet609C6964/PVin+
- U7 pad 4: /DC/DC_Converter/ISN -> Net-(R11-Pad2)
- U7 pad 5: Imppt1 -> Net-(R14-Pad1)
- U7 pad 6: +3V3 -> Net-(R16-Pad1)
- U8 pad 1: Net-(C20-Pad1) -> +3V3
- U8 pad 2: Net-(C20-Pad1) -> Pgnd
- U8 pad 3: Net-(C20-Pad1) -> /Sheet609B465C/sheet609C6965/R+
- U8 pad 4: Net-(R42-Pad1) -> /Sheet609B465C/sheet609C6964/PVin+
- U8 pad 5: /sheet608C3AAC/PVin+ -> Ipv1
- U8 pad 6: /sheet608C3AAC/PVin+ -> +3V3
- U9 pad 1: Pgnd -> +3V3
- U9 pad 3: Pgnd -> /Sheet609B465C/sheet609C6964/ISP
- U9 pad 4: Net-(R46-Pad1) -> /Sheet609B465C/Vout
- U9 pad 5: Net-(C20-Pad1) -> Imppt1
- U9 pad 6: Net-(C20-Pad1) -> +3V3
Routing:
- net Net-(C6-Pad1): track 178.3 -> 0.00 mm
- net /DC/DC_Converter/ISP: track 64.6 -> 0.00 mm
- net /DC/DC_Converter/PVin+: track 39.7 -> 0.00 mm
- net /DC/DC_Converter/FB: track 29.2 -> 0.00 mm, vias 2 -> 0
- net /current_Sense/R+: track 19.6 -> 0.00 mm
- net Net-(C11-Pad2): track 17.4 -> 0.00 mm
- net Net-(R33-Pad2): track 17.1 -> 0.00 mm, vias 2 -> 0
- net Net-(R38-Pad1): track 16.9 -> 0.00 mm, vias 2 -> 0
- net Net-(C6-Pad2): track 15.7 -> 0.00 mm, vias 2 -> 0
- net /DC/DC_Converter/ISN: track 15.1 -> 0.00 mm, vias 2 -> 0
- net Net-(R31-Pad2): track 14.9 -> 0.00 mm
- net Net-(R37-Pad2): track 14.7 -> 0.00 mm, vias 2 -> 0
- net Net-(C8-Pad2): track 12.5 -> 0.00 mm
- net Net-(R34-Pad1): track 9.98 -> 0.00 mm
- net Net-(R36-Pad1): track 6.62 -> 0.00 mm
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
Commit message: 1e mppt klaar (nog een keer)
Parts:
- moved R9 10.00 mm to (144.5, 135.7)
- moved U4 9.22 mm to (138.8, 131.2)
- moved C11 5.93 mm to (127.0, 136.9), turned to 0 degrees
- moved C12 5.57 mm to (122.3, 134.0), turned to 90 degrees
- moved R18 3.49 mm to (127.1, 142.4)
- moved C15 3.20 mm to (127.1, 139.8)
- moved R6 3.18 mm to (141.6, 134.1), turned to 90 degrees
- moved R17 3.14 mm to (128.1, 133.3), turned to 90 degrees
- moved R19 2.10 mm to (130.9, 141.2), turned to 270 degrees
- moved R14 0.45 mm to (106.9, 137.3)
- moved R16 0.44 mm to (106.9, 140.0)
- moved C10 0.39 mm to (119.6, 133.3), turned to 270 degrees
- moved C8 0.38 mm to (113.3, 138.7)
- moved C9 0.38 mm to (115.7, 138.6)
- moved C7 0.25 mm to (110.9, 138.7)
Routing:
- net Net-(C12-Pad2): track 0.00 -> 94.7 mm, vias 0 -> 14
- net /Sheet609B465C/sheet609C6964/PVin+: track 0.00 -> 69.2 mm
- net /Sheet609B465C/sheet609C6964/ISP: track 0.00 -> 39.9 mm
- net Net-(C10-Pad1): track 0.00 -> 29.8 mm
- net /Sheet609B465C/sheet609C6964/FB: track 0.00 -> 28.8 mm, vias 0 -> 1
- net Pgnd: track 0.00 -> 27.1 mm, vias 0 -> 2
- net /Sheet609B465C/sheet609C6965/R+: track 0.00 -> 24.0 mm
- net Net-(R11-Pad2): track 0.00 -> 23.4 mm
- net Net-(R17-Pad2): track 0.00 -> 19.3 mm, vias 0 -> 2
- net /Sheet609B465C/Vout: track 0.00 -> 15.6 mm, vias 0 -> 2
- net Net-(R14-Pad1): track 0.00 -> 11.9 mm
- net Net-(R16-Pad1): track 0.00 -> 10.3 mm
- net +3V3: track 0.00 -> 9.80 mm
- net Net-(R13-Pad2): track 0.00 -> 9.11 mm
- net Net-(R13-Pad1): track 0.00 -> 7.48 mm
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- added copper zone on B.Cu, net Pgnd
- added copper zone on F.Cu, net Pgnd
Other:
- net class power: clearance 0.2 -> 0.1; trace_width 0.5 -> 0.25
