File: PEE50_MPPT/current_sense.sch (KiCad schematic (older format))
At the start: 2 parts, among them U5 MAX44284FAUT+T

Commit message: schakeling klaar (denk ik)
Changed lines of the file:
@@
 $Descr A4 11693 8268
 encoding utf-8
-Sheet 5 15
+Sheet 4 15
 Title ""
 Date ""
@@
 AR Path="/608DD930/608BDE84" Ref="U6"  Part="1"
 AR Path="/608DD944/608BDE84" Ref="U6"  Part="1"
-F 0 "U6" H 5500 3487 60  0000 C CNN
+F 0 "U5" H 5500 3487 60  0000 C CNN
 F 1 "MAX44284FAUT+T" H 5500 3381 60  0000 C CNN
 F 2 "21-0058I_MXM" H 5500 3340 60  0001 C CNN
@@
 AR Path="/608DD930/608BDFD5" Ref="#PWR0174"  Part="1"
 AR Path="/608DD944/608BDFD5" Ref="#PWR0178"  Part="1"
-F 0 "#PWR0178" H 4600 2850 50  0001 C CNN
+F 0 "#PWR0113" H 4600 2850 50  0001 C CNN
 F 1 "+3V3" H 4615 3173 50  0000 C CNN
 F 2 "" H 4600 3000 50  0001 C CNN
@@
 AR Path="/608DD930/608BE004" Ref="C14"  Part="1"
 AR Path="/608DD944/608BE004" Ref="C14"  Part="1"
-F 0 "C14" V 4098 3100 50  0000 C CNN
+F 0 "C13" V 4098 3100 50  0000 C CNN
 F 1 "100n" V 4189 3100 50  0000 C CNN
 F 2 "" H 4388 2950 50  0001 C CNN
@@
 AR Path="/608DD930/608BE067" Ref="#PWR0175"  Part="1"
 AR Path="/608DD944/608BE067" Ref="#PWR0179"  Part="1"
-F 0 "#PWR0179" H 4050 2900 50  0001 C CNN
+F 0 "#PWR0114" H 4050 2900 50  0001 C CNN
 F 1 "GND" H 4055 2977 50  0000 C CNN
 F 2 "" H 4050 3150 50  0001 C CNN
@@
 AR Path="/608DD930/608BE0AE" Ref="#PWR0176"  Part="1"
 AR Path="/608DD944/608BE0AE" Ref="#PWR0180"  Part="1"
-F 0 "#PWR0180" H 4500 2950 50  0001 C CNN
+F 0 "#PWR0115" H 4500 2950 50  0001 C CNN
 F 1 "GND" H 4505 3027 50  0000 C CNN
 F 2 "" H 4500 3200 50  0001 C CNN
@@
 AR Path="/608DD930/608BE366" Ref="#PWR0177"  Part="1"
 AR Path="/608DD944/608BE366" Ref="#PWR0181"  Part="1"
-F 0 "#PWR0181" H 6400 2900 50  0001 C CNN
+F 0 "#PWR0116" H 6400 2900 50  0001 C CNN
 F 1 "+3V3" H 6415 3223 50  0000 C CNN
 F 2 "" H 6400 3050 50  0001 C CNN

Commit message: maar opnieuw begonnen met mppt layouten ivm plugin regels
Parts:
- C18: renamed from C13; footprint (none) -> Capacitor_SMD:C_1206_3216Metric_Pad1.42x1.75mm_HandSolder
- U8: renamed from U5; footprint 21-0058I_MXM -> Robin_Lib:21-0058I_MXM
Changed lines of the file:
@@
 $Descr A4 11693 8268
 encoding utf-8
-Sheet 4 15
+Sheet 6 19
 Title ""
 Date ""
@@
 P 4700 3100
 AR Path="/608BDE84" Ref="U?"  Part="1"
-AR Path="/608BDD43/608BDE84" Ref="U5"  Part="1"
-AR Path="/608BF482/608BDE84" Ref="U6"  Part="1"
-AR Path="/608C3AF8/608BDE84" Ref="U6"  Part="1"
-AR Path="/608C3B0C/608BDE84" Ref="U6"  Part="1"
-AR Path="/608C70E9/608BDE84" Ref="U6"  Part="1"
-AR Path="/608C70FD/608BDE84" Ref="U6"  Part="1"
-AR Path="/608DD930/608BDE84" Ref="U6"  Part="1"
-AR Path="/608DD944/608BDE84" Ref="U6"  Part="1"
-F 0 "U5" H 5500 3487 60  0000 C CNN
+AR Path="/608BDD43/608BDE84" Ref="U?"  Part="1"
+AR Path="/608BF482/608BDE84" Ref="U?"  Part="1"
+AR Path="/608C3AF8/608BDE84" Ref="U?"  Part="1"
+AR Path="/608C3B0C/608BDE84" Ref="U?"  Part="1"
+AR Path="/608C70E9/608BDE84" Ref="U?"  Part="1"
+AR Path="/608C70FD/608BDE84" Ref="U?"  Part="1"
+AR Path="/608DD930/608BDE84" Ref="U?"  Part="1"
+AR Path="/608DD944/608BDE84" Ref="U?"  Part="1"
+AR Path="/609B465D/609C69AB/608BDE84" Ref="U8"  Part="1"
+AR Path="/609B465D/609C69BF/608BDE84" Ref="U?"  Part="1"
+AR Path="/609F26BD/609C69AB/608BDE84" Ref="U14"  Part="1"
+AR Path="/609F26BD/609C69BF/608BDE84" Ref="U?"  Part="1"
+AR Path="/609F4759/609C69AB/608BDE84" Ref="U20"  Part="1"
+AR Path="/609F4759/609C69BF/608BDE84" Ref="U?"  Part="1"
+AR Path="/609F5798/609C69AB/608BDE84" Ref="U26"  Part="1"
+AR Path="/609F5798/609C69BF/608BDE84" Ref="U?"  Part="1"
+F 0 "U8" H 5500 3487 60  0000 C CNN
 F 1 "MAX44284FAUT+T" H 5500 3381 60  0000 C CNN
-F 2 "21-0058I_MXM" H 5500 3340 60  0001 C CNN
+F 2 "Robin_Lib:21-0058I_MXM" H 5500 3340 60  0001 C CNN
 F 3 "" H 4700 3100 60  0000 C CNN
 	1    4700 3100
@@
 $EndComp
 $Comp
-L power:+3V3 #PWR0113
+L power:+3V3 #PWR?
 U 1 1 608BDFD5
 P 4600 3000
-AR Path="/608BDD43/608BDFD5" Ref="#PWR0113"  Part="1"
-AR Path="/608BF482/608BDFD5" Ref="#PWR0117"  Part="1"
-AR Path="/608C3AF8/608BDFD5" Ref="#PWR0142"  Part="1"
-AR Path="/608C3B0C/608BDFD5" Ref="#PWR0146"  Part="1"
-AR Path="/608C70E9/608BDFD5" Ref="#PWR0158"  Part="1"
-AR Path="/608C70FD/608BDFD5" Ref="#PWR0162"  Part="1"
-AR Path="/608DD930/608BDFD5" Ref="#PWR0174"  Part="1"
-AR Path="/608DD944/608BDFD5" Ref="#PWR0178"  Part="1"
-F 0 "#PWR0113" H 4600 2850 50  0001 C CNN
+AR Path="/608BDD43/608BDFD5" Ref="#PWR?"  Part="1"
+AR Path="/608BF482/608BDFD5" Ref="#PWR?"  Part="1"
+AR Path="/608C3AF8/608BDFD5" Ref="#PWR?"  Part="1"
+AR Path="/608C3B0C/608BDFD5" Ref="#PWR?"  Part="1"
+AR Path="/608C70E9/608BDFD5" Ref="#PWR?"  Part="1"
+AR Path="/608C70FD/608BDFD5" Ref="#PWR?"  Part="1"
+AR Path="/608DD930/608BDFD5" Ref="#PWR?"  Part="1"
+AR Path="/608DD944/608BDFD5" Ref="#PWR?"  Part="1"
+AR Path="/609B465D/609C69AB/608BDFD5" Ref="#PWR032"  Part="1"
+AR Path="/609B465D/609C69BF/608BDFD5" Ref="#PWR?"  Part="1"
+AR Path="/609F26BD/609C69AB/608BDFD5" Ref="#PWR053"  Part="1"
+AR Path="/609F26BD/609C69BF/608BDFD5" Ref="#PWR?"  Part="1"
+AR Path="/609F4759/609C69AB/608BDFD5" Ref="#PWR074"  Part="1"
+AR Path="/609F4759/609C69BF/608BDFD5" Ref="#PWR?"  Part="1"
+AR Path="/609F5798/609C69AB/608BDFD5" Ref="#PWR095"  Part="1"
+AR Path="/609F5798/609C69BF/608BDFD5" Ref="#PWR?"  Part="1"
+F 0 "#PWR095" H 4600 2850 50  0001 C CNN
 F 1 "+3V3" H 4615 3173 50  0000 C CNN
 F 2 "" H 4600 3000 50  0001 C CNN
@@
 	4600 3100 4700 3100
 $Comp
-L Device:C C13
+L Device:C C?
 U 1 1 608BE004
 P 4350 3100
-AR Path="/608BDD43/608BE004" Ref="C13"  Part="1"
-AR Path="/608BF482/608BE004" Ref="C14"  Part="1"
-AR Path="/608C3AF8/608BE004" Ref="C14"  Part="1"
-AR Path="/608C3B0C/608BE004" Ref="C14"  Part="1"
-AR Path="/608C70E9/608BE004" Ref="C14"  Part="1"
-AR Path="/608C70FD/608BE004" Ref="C14"  Part="1"
-AR Path="/608DD930/608BE004" Ref="C14"  Part="1"
-AR Path="/608DD944/608BE004" Ref="C14"  Part="1"
-F 0 "C13" V 4098 3100 50  0000 C CNN
+AR Path="/608BDD43/608BE004" Ref="C?"  Part="1"
+AR Path="/608BF482/608BE004" Ref="C?"  Part="1"
+AR Path="/608C3AF8/608BE004" Ref="C?"  Part="1"
+AR Path="/608C3B0C/608BE004" Ref="C?"  Part="1"
+AR Path="/608C70E9/608BE004" Ref="C?"  Part="1"
+AR Path="/608C70FD/608BE004" Ref="C?"  Part="1"
+AR Path="/608DD930/608BE004" Ref="C?"  Part="1"
+AR Path="/608DD944/608BE004" Ref="C?"  Part="1"
+AR Path="/609B465D/609C69AB/608BE004" Ref="C18"  Part="1"
+AR Path="/609B465D/609C69BF/608BE004" Ref="C?"  Part="1"
+AR Path="/609F26BD/609C69AB/608BE004" Ref="C31"  Part="1"
+AR Path="/609F26BD/609C69BF/608BE004" Ref="C?"  Part="1"
+AR Path="/609F4759/609C69AB/608BE004" Ref="C44"  Part="1"
+AR Path="/609F4759/609C69BF/608BE004" Ref="C?"  Part="1"
+AR Path="/609F5798/609C69AB/608BE004" Ref="C57"  Part="1"
+AR Path="/609F5798/609C69BF/608BE004" Ref="C?"  Part="1"
+F 0 "C18" V 4098 3100 50  0000 C CNN
 F 1 "100n" V 4189 3100 50  0000 C CNN
-F 2 "" H 4388 2950 50  0001 C CNN
+F 2 "Capacitor_SMD:C_1206_3216Metric_Pad1.42x1.75mm_HandSolder" H 4388 2950 50  0001 C CNN
 F 3 "~" H 4350 3100 50  0001 C CNN
 	1    4350 3100
@@
 Connection ~ 4600 3100
 $Comp
-L power:GND #PWR0114
+L power:GND #PWR?
 U 1 1 608BE067
 P 4050 3150
-AR Path="/608BDD43/608BE067" Ref="#PWR0114"  Part="1"
-AR Path="/608BF482/608BE067" Ref="#PWR0118"  Part="1"
-AR Path="/608C3AF8/608BE067" Ref="#PWR0143"  Part="1"
-AR Path="/608C3B0C/608BE067" Ref="#PWR0147"  Part="1"
-AR Path="/608C70E9/608BE067" Ref="#PWR0159"  Part="1"
-AR Path="/608C70FD/608BE067" Ref="#PWR0163"  Part="1"
-AR Path="/608DD930/608BE067" Ref="#PWR0175"  Part="1"
-AR Path="/608DD944/608BE067" Ref="#PWR0179"  Part="1"
-F 0 "#PWR0114" H 4050 2900 50  0001 C CNN
+AR Path="/608BDD43/608BE067" Ref="#PWR?"  Part="1"
+AR Path="/608BF482/608BE067" Ref="#PWR?"  Part="1"
+AR Path="/608C3AF8/608BE067" Ref="#PWR?"  Part="1"
+AR Path="/608C3B0C/608BE067" Ref="#PWR?"  Part="1"
+AR Path="/608C70E9/608BE067" Ref="#PWR?"  Part="1"
+AR Path="/608C70FD/608BE067" Ref="#PWR?"  Part="1"
+AR Path="/608DD930/608BE067" Ref="#PWR?"  Part="1"
+AR Path="/608DD944/608BE067" Ref="#PWR?"  Part="1"
+AR Path="/609B465D/609C69AB/608BE067" Ref="#PWR030"  Part="1"
+AR Path="/609B465D/609C69BF/608BE067" Ref="#PWR?"  Part="1"
+AR Path="/609F26BD/609C69AB/608BE067" Ref="#PWR051"  Part="1"
+AR Path="/609F26BD/609C69BF/608BE067" Ref="#PWR?"  Part="1"
+AR Path="/609F4759/609C69AB/608BE067" Ref="#PWR072"  Part="1"
+AR Path="/609F4759/609C69BF/608BE067" Ref="#PWR?"  Part="1"
+AR Path="/609F5798/609C69AB/608BE067" Ref="#PWR093"  Part="1"
+AR Path="/609F5798/609C69BF/608BE067" Ref="#PWR?"  Part="1"
+F 0 "#PWR093" H 4050 2900 50  0001 C CNN
 F 1 "GND" H 4055 2977 50  0000 C CNN
 F 2 "" H 4050 3150 50  0001 C CNN
@@
 	4050 3100 4200 3100
 $Comp
-L power:GND #PWR0115
+L power:GND #PWR?
 U 1 1 608BE0AE
 P 4500 3200
-AR Path="/608BDD43/608BE0AE" Ref="#PWR0115"  Part="1"
-AR Path="/608BF482/608BE0AE" Ref="#PWR0119"  Part="1"
-AR Path="/608C3AF8/608BE0AE" Ref="#PWR0144"  Part="1"
-AR Path="/608C3B0C/608BE0AE" Ref="#PWR0148"  Part="1"
-AR Path="/608C70E9/608BE0AE" Ref="#PWR0160"  Part="1"
-AR Path="/608C70FD/608BE0AE" Ref="#PWR0164"  Part="1"
-AR Path="/608DD930/608BE0AE" Ref="#PWR0176"  Part="1"
-AR Path="/608DD944/608BE0AE" Ref="#PWR0180"  Part="1"
-F 0 "#PWR0115" H 4500 2950 50  0001 C CNN
+AR Path="/608BDD43/608BE0AE" Ref="#PWR?"  Part="1"
+AR Path="/608BF482/608BE0AE" Ref="#PWR?"  Part="1"
+AR Path="/608C3AF8/608BE0AE" Ref="#PWR?"  Part="1"
+AR Path="/608C3B0C/608BE0AE" Ref="#PWR?"  Part="1"
+AR Path="/608C70E9/608BE0AE" Ref="#PWR?"  Part="1"
+AR Path="/608C70FD/608BE0AE" Ref="#PWR?"  Part="1"
+AR Path="/608DD930/608BE0AE" Ref="#PWR?"  Part="1"
+AR Path="/608DD944/608BE0AE" Ref="#PWR?"  Part="1"
+AR Path="/609B465D/609C69AB/608BE0AE" Ref="#PWR031"  Part="1"
+AR Path="/609B465D/609C69BF/608BE0AE" Ref="#PWR?"  Part="1"
+AR Path="/609F26BD/609C69AB/608BE0AE" Ref="#PWR052"  Part="1"
+AR Path="/609F26BD/609C69BF/608BE0AE" Ref="#PWR?"  Part="1"
+AR Path="/609F4759/609C69AB/608BE0AE" Ref="#PWR073"  Part="1"
+AR Path="/609F4759/609C69BF/608BE0AE" Ref="#PWR?"  Part="1"
+AR Path="/609F5798/609C69AB/608BE0AE" Ref="#PWR094"  Part="1"
+AR Path="/609F5798/609C69BF/608BE0AE" Ref="#PWR?"  Part="1"
+F 0 "#PWR094" H 4500 2950 50  0001 C CNN
 F 1 "GND" H 4505 3027 50  0000 C CNN
 F 2 "" H 4500 3200 50  0001 C CNN
@@
 	4500 3200 4700 3200
 $Comp
-L power:+3V3 #PWR0116
+L power:+3V3 #PWR?
 U 1 1 608BE366
 P 6400 3050
-AR Path="/608BDD43/608BE366" Ref="#PWR0116"  Part="1"
-AR Path="/608BF482/608BE366" Ref="#PWR0120"  Part="1"
-AR Path="/608C3AF8/608BE366" Ref="#PWR0145"  Part="1"
-AR Path="/608C3B0C/608BE366" Ref="#PWR0149"  Part="1"
-AR Path="/608C70E9/608BE366" Ref="#PWR0161"  Part="1"
-AR Path="/608C70FD/608BE366" Ref="#PWR0165"  Part="1"
-AR Path="/608DD930/608BE366" Ref="#PWR0177"  Part="1"
-AR Path="/608DD944/608BE366" Ref="#PWR0181"  Part="1"
-F 0 "#PWR0116" H 6400 2900 50  0001 C CNN
+AR Path="/608BDD43/608BE366" Ref="#PWR?"  Part="1"
+AR Path="/608BF482/608BE366" Ref="#PWR?"  Part="1"
+AR Path="/608C3AF8/608BE366" Ref="#PWR?"  Part="1"
+AR Path="/608C3B0C/608BE366" Ref="#PWR?"  Part="1"
+AR Path="/608C70E9/608BE366" Ref="#PWR?"  Part="1"
+AR Path="/608C70FD/608BE366" Ref="#PWR?"  Part="1"
+AR Path="/608DD930/608BE366" Ref="#PWR?"  Part="1"
+AR Path="/608DD944/608BE366" Ref="#PWR?"  Part="1"
+AR Path="/609B465D/609C69AB/608BE366" Ref="#PWR033"  Part="1"
+AR Path="/609B465D/609C69BF/608BE366" Ref="#PWR?"  Part="1"
+AR Path="/609F26BD/609C69AB/608BE366" Ref="#PWR054"  Part="1"
+AR Path="/609F26BD/609C69BF/608BE366" Ref="#PWR?"  Part="1"
+AR Path="/609F4759/609C69AB/608BE366" Ref="#PWR075"  Part="1"
+AR Path="/609F4759/609C69BF/608BE366" Ref="#PWR?"  Part="1"
+AR Path="/609F5798/609C69AB/608BE366" Ref="#PWR096"  Part="1"
+AR Path="/609F5798/609C69BF/608BE366" Ref="#PWR?"  Part="1"
+F 0 "#PWR096" H 6400 2900 50  0001 C CNN
 F 1 "+3V3" H 6415 3223 50  0000 C CNN
 F 2 "" H 6400 3050 50  0001 C CNN

Commit message: spinneweb aangemaakt
Changed lines of the file:
@@
 AR Path="/609F5798/609C69AB/608BDE84" Ref="U26"  Part="1"
 AR Path="/609F5798/609C69BF/608BDE84" Ref="U?"  Part="1"
-F 0 "U8" H 5500 3487 60  0000 C CNN
+F 0 "U26" H 5500 3487 60  0000 C CNN
 F 1 "MAX44284FAUT+T" H 5500 3381 60  0000 C CNN
 F 2 "Robin_Lib:21-0058I_MXM" H 5500 3340 60  0001 C CNN
@@
 AR Path="/609F5798/609C69AB/608BE004" Ref="C57"  Part="1"
 AR Path="/609F5798/609C69BF/608BE004" Ref="C?"  Part="1"
-F 0 "C18" V 4098 3100 50  0000 C CNN
+F 0 "C57" V 4098 3100 50  0000 C CNN
 F 1 "100n" V 4189 3100 50  0000 C CNN
 F 2 "Capacitor_SMD:C_1206_3216Metric_Pad1.42x1.75mm_HandSolder" H 4388 2950 50  0001 C CNN
