File: PEE50_MPPT/current_sense1.sch (KiCad schematic (older format))
At the start: 2 parts, among them U6 MAX44284FAUT+T

Commit message: best veel footprints ingevoegd
Parts:
- C15: footprint (none) -> Capacitor_SMD:C_1206_3216Metric_Pad1.42x1.75mm_HandSolder
Changed lines of the file:
@@
 EESchema Schematic File Version 4
-LIBS:PEE50_MPPT-cache
-EELAYER 26 0
+EELAYER 30 0
 EELAYER END
 $Descr A4 11693 8268
@@
 F 0 "C15" V 4098 3100 50  0000 C CNN
 F 1 "100n" V 4189 3100 50  0000 C CNN
-F 2 "" H 4388 2950 50  0001 C CNN
+F 2 "Capacitor_SMD:C_1206_3216Metric_Pad1.42x1.75mm_HandSolder" H 4388 2950 50  0001 C CNN
 F 3 "~" H 4350 3100 50  0001 C CNN
 	1    4350 3100

Commit message: footprints gemapt + 10x10 pcb rand getekend
Parts:
- U6: footprint 21-0058I_MXM -> Robin_Lib:21-0058I_MXM
Changed lines of the file:
@@
 EESchema Schematic File Version 4
-EELAYER 30 0
+LIBS:PEE50_MPPT-cache
+EELAYER 26 0
 EELAYER END
 $Descr A4 11693 8268
@@
 F 0 "U6" H 5500 3487 60  0000 C CNN
 F 1 "MAX44284FAUT+T" H 5500 3381 60  0000 C CNN
-F 2 "21-0058I_MXM" H 5500 3340 60  0001 C CNN
+F 2 "Robin_Lib:21-0058I_MXM" H 5500 3340 60  0001 C CNN
 F 3 "" H 4700 3100 60  0000 C CNN
 	1    4700 3100

Commit message: maar opnieuw begonnen met mppt layouten ivm plugin regels
Parts:
- renumbered C15 to C19, U6 to U9
Changed lines of the file:
@@
 $Descr A4 11693 8268
 encoding utf-8
-Sheet 4 15
+Sheet 7 19
 Title ""
 Date ""
@@
 P 4700 3100
 AR Path="/6099D7C1" Ref="U?"  Part="1"
-AR Path="/608BDD43/6099D7C1" Ref="U6"  Part="1"
+AR Path="/608BDD43/6099D7C1" Ref="U?"  Part="1"
 AR Path="/608BF482/6099D7C1" Ref="U?"  Part="1"
 AR Path="/608C3AF8/6099D7C1" Ref="U?"  Part="1"
@@
 AR Path="/608DD930/6099D7C1" Ref="U?"  Part="1"
 AR Path="/608DD944/6099D7C1" Ref="U?"  Part="1"
-F 0 "U6" H 5500 3487 60  0000 C CNN
+AR Path="/609B465D/609C69BF/6099D7C1" Ref="U9"  Part="1"
+AR Path="/609F26BD/609C69BF/6099D7C1" Ref="U15"  Part="1"
+AR Path="/609F4759/609C69BF/6099D7C1" Ref="U21"  Part="1"
+AR Path="/609F5798/609C69BF/6099D7C1" Ref="U27"  Part="1"
+F 0 "U9" H 5500 3487 60  0000 C CNN
 F 1 "MAX44284FAUT+T" H 5500 3381 60  0000 C CNN
 F 2 "Robin_Lib:21-0058I_MXM" H 5500 3340 60  0001 C CNN
@@
 $EndComp
 $Comp
-L power:+3V3 #PWR032
+L power:+3V3 #PWR?
 U 1 1 6099D7C5
 P 4600 3000
-AR Path="/608BDD43/6099D7C5" Ref="#PWR032"  Part="1"
+AR Path="/608BDD43/6099D7C5" Ref="#PWR?"  Part="1"
 AR Path="/608BF482/6099D7C5" Ref="#PWR?"  Part="1"
 AR Path="/608C3AF8/6099D7C5" Ref="#PWR?"  Part="1"
@@
 AR Path="/608DD930/6099D7C5" Ref="#PWR?"  Part="1"
 AR Path="/608DD944/6099D7C5" Ref="#PWR?"  Part="1"
-F 0 "#PWR032" H 4600 2850 50  0001 C CNN
+AR Path="/609B465D/609C69BF/6099D7C5" Ref="#PWR036"  Part="1"
+AR Path="/609F26BD/609C69BF/6099D7C5" Ref="#PWR057"  Part="1"
+AR Path="/609F4759/609C69BF/6099D7C5" Ref="#PWR078"  Part="1"
+AR Path="/609F5798/609C69BF/6099D7C5" Ref="#PWR099"  Part="1"
+F 0 "#PWR099" H 4600 2850 50  0001 C CNN
 F 1 "+3V3" H 4615 3173 50  0000 C CNN
 F 2 "" H 4600 3000 50  0001 C CNN
@@
 	4600 3100 4700 3100
 $Comp
-L Device:C C15
+L Device:C C?
 U 1 1 6099D7D2
 P 4350 3100
-AR Path="/608BDD43/6099D7D2" Ref="C15"  Part="1"
+AR Path="/608BDD43/6099D7D2" Ref="C?"  Part="1"
 AR Path="/608BF482/6099D7D2" Ref="C?"  Part="1"
 AR Path="/608C3AF8/6099D7D2" Ref="C?"  Part="1"
@@
 AR Path="/608DD930/6099D7D2" Ref="C?"  Part="1"
 AR Path="/608DD944/6099D7D2" Ref="C?"  Part="1"
-F 0 "C15" V 4098 3100 50  0000 C CNN
+AR Path="/609B465D/609C69BF/6099D7D2" Ref="C19"  Part="1"
+AR Path="/609F26BD/609C69BF/6099D7D2" Ref="C32"  Part="1"
+AR Path="/609F4759/609C69BF/6099D7D2" Ref="C45"  Part="1"
+AR Path="/609F5798/609C69BF/6099D7D2" Ref="C58"  Part="1"
+F 0 "C19" V 4098 3100 50  0000 C CNN
 F 1 "100n" V 4189 3100 50  0000 C CNN
 F 2 "Capacitor_SMD:C_1206_3216Metric_Pad1.42x1.75mm_HandSolder" H 4388 2950 50  0001 C CNN
@@
 Connection ~ 4600 3100
 $Comp
-L power:GND #PWR030
+L power:GND #PWR?
 U 1 1 6099D7D3
 P 4050 3150
-AR Path="/608BDD43/6099D7D3" Ref="#PWR030"  Part="1"
+AR Path="/608BDD43/6099D7D3" Ref="#PWR?"  Part="1"
 AR Path="/608BF482/6099D7D3" Ref="#PWR?"  Part="1"
 AR Path="/608C3AF8/6099D7D3" Ref="#PWR?"  Part="1"
@@
 AR Path="/608DD930/6099D7D3" Ref="#PWR?"  Part="1"
 AR Path="/608DD944/6099D7D3" Ref="#PWR?"  Part="1"
-F 0 "#PWR030" H 4050 2900 50  0001 C CNN
+AR Path="/609B465D/609C69BF/6099D7D3" Ref="#PWR034"  Part="1"
+AR Path="/609F26BD/609C69BF/6099D7D3" Ref="#PWR055"  Part="1"
+AR Path="/609F4759/609C69BF/6099D7D3" Ref="#PWR076"  Part="1"
+AR Path="/609F5798/609C69BF/6099D7D3" Ref="#PWR097"  Part="1"
+F 0 "#PWR097" H 4050 2900 50  0001 C CNN
 F 1 "GND" H 4055 2977 50  0000 C CNN
 F 2 "" H 4050 3150 50  0001 C CNN
@@
 	4050 3100 4200 3100
 $Comp
-L power:GND #PWR031
+L power:GND #PWR?
 U 1 1 6099D7DA
 P 4500 3200
-AR Path="/608BDD43/6099D7DA" Ref="#PWR031"  Part="1"
+AR Path="/608BDD43/6099D7DA" Ref="#PWR?"  Part="1"
 AR Path="/608BF482/6099D7DA" Ref="#PWR?"  Part="1"
 AR Path="/608C3AF8/6099D7DA" Ref="#PWR?"  Part="1"
@@
 AR Path="/608DD930/6099D7DA" Ref="#PWR?"  Part="1"
 AR Path="/608DD944/6099D7DA" Ref="#PWR?"  Part="1"
-F 0 "#PWR031" H 4500 2950 50  0001 C CNN
+AR Path="/609B465D/609C69BF/6099D7DA" Ref="#PWR035"  Part="1"
+AR Path="/609F26BD/609C69BF/6099D7DA" Ref="#PWR056"  Part="1"
+AR Path="/609F4759/609C69BF/6099D7DA" Ref="#PWR077"  Part="1"
+AR Path="/609F5798/609C69BF/6099D7DA" Ref="#PWR098"  Part="1"
+F 0 "#PWR098" H 4500 2950 50  0001 C CNN
 F 1 "GND" H 4505 3027 50  0000 C CNN
 F 2 "" H 4500 3200 50  0001 C CNN
@@
 	4500 3200 4700 3200
 $Comp
-L power:+3V3 #PWR033
+L power:+3V3 #PWR?
 U 1 1 6099D7E2
 P 6400 3050
-AR Path="/608BDD43/6099D7E2" Ref="#PWR033"  Part="1"
+AR Path="/608BDD43/6099D7E2" Ref="#PWR?"  Part="1"
 AR Path="/608BF482/6099D7E2" Ref="#PWR?"  Part="1"
 AR Path="/608C3AF8/6099D7E2" Ref="#PWR?"  Part="1"
@@
 AR Path="/608DD930/6099D7E2" Ref="#PWR?"  Part="1"
 AR Path="/608DD944/6099D7E2" Ref="#PWR?"  Part="1"
-F 0 "#PWR033" H 6400 2900 50  0001 C CNN
+AR Path="/609B465D/609C69BF/6099D7E2" Ref="#PWR037"  Part="1"
+AR Path="/609F26BD/609C69BF/6099D7E2" Ref="#PWR058"  Part="1"
+AR Path="/609F4759/609C69BF/6099D7E2" Ref="#PWR079"  Part="1"
+AR Path="/609F5798/609C69BF/6099D7E2" Ref="#PWR0100"  Part="1"
+F 0 "#PWR0100" H 6400 2900 50  0001 C CNN
 F 1 "+3V3" H 6415 3223 50  0000 C CNN
 F 2 "" H 6400 3050 50  0001 C CNN

Commit message: spinneweb aangemaakt
Changed lines of the file:
@@
 AR Path="/609F4759/609C69BF/6099D7C1" Ref="U21"  Part="1"
 AR Path="/609F5798/609C69BF/6099D7C1" Ref="U27"  Part="1"
-F 0 "U9" H 5500 3487 60  0000 C CNN
+F 0 "U27" H 5500 3487 60  0000 C CNN
 F 1 "MAX44284FAUT+T" H 5500 3381 60  0000 C CNN
 F 2 "Robin_Lib:21-0058I_MXM" H 5500 3340 60  0001 C CNN
@@
 AR Path="/609F4759/609C69BF/6099D7D2" Ref="C45"  Part="1"
 AR Path="/609F5798/609C69BF/6099D7D2" Ref="C58"  Part="1"
-F 0 "C19" V 4098 3100 50  0000 C CNN
+F 0 "C58" V 4098 3100 50  0000 C CNN
 F 1 "100n" V 4189 3100 50  0000 C CNN
 F 2 "Capacitor_SMD:C_1206_3216Metric_Pad1.42x1.75mm_HandSolder" H 4388 2950 50  0001 C CNN
