File: PEE50_MPPT/uC.sch (KiCad schematic (older format))
At the start: 4 parts, among them J3 Conn_01x03_Female, J4 Conn_01x03_Female, U2 MSP430FR2353TDBT

Commit message: reset pin en errors weggewerkt
Parts:
- added R71: 10k, Resistor_SMD:R_1206_3216Metric_Pad1.42x1.75mm_HandSolder, symbol Device:R
- added SW1: SW_DIP_x01, Button_Switch_THT:KSA_Tactile_SPST, symbol Switch:SW_DIP_x01
Connections:
- net +3V3: now also R71.1
- net GND: now also SW1.2
- net at J4.2 (Pin_2), U2.9 (*RST/NMI/SBWTDIO): now also R71.2, SW1.1
- no-connect marks 0 -> 23
Changed lines of the file:
@@
 Wire Wire Line
 	7500 3100 7600 3100
+NoConn ~ 3900 3250
+NoConn ~ 3900 3350
+NoConn ~ 3900 3450
+NoConn ~ 3900 3550
+NoConn ~ 3900 3650
+NoConn ~ 3900 3750
+NoConn ~ 3900 3850
+NoConn ~ 3900 3950
+NoConn ~ 3900 4200
+NoConn ~ 3900 4300
+NoConn ~ 7500 4850
+NoConn ~ 7500 4750
+NoConn ~ 7500 4550
+NoConn ~ 7500 4450
+NoConn ~ 7500 4350
+NoConn ~ 7500 4150
+NoConn ~ 7500 3950
+NoConn ~ 7500 3850
+NoConn ~ 7500 3750
+NoConn ~ 7500 3650
+NoConn ~ 7500 2700
+NoConn ~ 7500 2600
+NoConn ~ 7500 2500
+$Comp
+L Device:R R71
+U 1 1 60A5EFFF
+P 3800 1750
+F 0 "R71" H 3870 1796 50  0000 L CNN
+F 1 "10k" H 3870 1705 50  0000 L CNN
+F 2 "Resistor_SMD:R_1206_3216Metric_Pad1.42x1.75mm_HandSolder" V 3730 1750 50  0001 C CNN
+F 3 "~" H 3800 1750 50  0001 C CNN
+	1    3800 1750
+	1    0    0    -1
+$EndComp
+Wire Wire Line
+	3800 1900 3800 1950
+Connection ~ 3800 1950
+Wire Wire Line
+	3800 1600 4700 1600
+Wire Wire Line
+	4700 1600 4700 1800
+Wire Wire Line
+	4700 1800 5700 1800
+Connection ~ 5700 1800
+$Comp
+L Switch:SW_DIP_x01 SW1
+U 1 1 60A607C6
+P 3800 2500
+F 0 "SW1" V 3754 2630 50  0000 L CNN
+F 1 "SW_DIP_x01" V 3845 2630 50  0000 L CNN
+F 2 "Button_Switch_THT:KSA_Tactile_SPST" H 3800 2500 50  0001 C CNN
+F 3 "~" H 3800 2500 50  0001 C CNN
+	1    3800 2500
+	0    1    1    0
+$EndComp
+$Comp
+L power:GND #PWR0103
+U 1 1 60A60F26
+P 3800 2850
+F 0 "#PWR0103" H 3800 2600 50  0001 C CNN
+F 1 "GND" H 3805 2677 50  0000 C CNN
+F 2 "" H 3800 2850 50  0001 C CNN
+F 3 "" H 3800 2850 50  0001 C CNN
+	1    3800 2850
+	1    0    0    -1
+$EndComp
+Wire Wire Line
+	3800 2850 3800 2800
+Wire Wire Line
+	3800 2200 3800 2150
+Connection ~ 3800 2150
 $EndSCHEMATC
