File: PEE50-BatteryProtectionCircuit/PEE50-Schakeling.sch (KiCad schematic (older format))
At the start: 30 parts, among them U1 MAX17320G20+

Commit message: Vorige versie was outdated doordat of ik of kicad niet fatsoenlijk op ctrl+s kan klikken :) Nu wel de meest recente versie
Parts:
- removed C?: 0.47uF, symbol Device:C
- added C?: 0.1uF, symbol Device:C
- added D?: 4.7V Zener, symbol Device:D_Zener
- added R?: 150Ohm, symbol Device:R
- added R?: 10kOhm, symbol Device:R
- added R? (x2): 100 Ohm, symbol Device:R
- R? (x4): value 9 Ohm -> 50 Ohm
Connections:
- wire segments 99 -> 105
- no-connect marks 5 -> 6
Other:
- note removed: "Always on LDO\n(Eventueel voor externe apparaten)\nNiet geschikt voor uC"
Changed lines of the file:
@@
 	1    0    0    -1
 $EndComp
-Text GLabel 6650 4000 2    50   Input ~ 0
+Text GLabel 6650 4050 2    50   Input ~ 0
 NegativeTerminal
 Wire Wire Line
@@
 Wire Wire Line
 	2650 3250 2450 3250
-Wire Wire Line
-	2450 3250 2450 3750
-Wire Wire Line
-	2450 3750 2200 3750
-Wire Wire Line
-	2200 3750 2200 3800
-Connection ~ 2450 3750
-$Comp
-L Device:C C?
-U 1 1 608DCFEC
-P 2200 3950
-F 0 "C?" H 2315 3996 50  0000 L CNN
-F 1 "0.47uF" H 2315 3905 50  0000 L CNN
-F 2 "" H 2238 3800 50  0001 C CNN
-F 3 "~" H 2200 3950 50  0001 C CNN
-	1    2200 3950
-	1    0    0    -1
-$EndComp
-$Comp
-L power:GND #PWR?
-U 1 1 608DD5DA
-P 2200 4100
-F 0 "#PWR?" H 2200 3850 50  0001 C CNN
-F 1 "GND" H 2205 3927 50  0000 C CNN
-F 2 "" H 2200 4100 50  0001 C CNN
-F 3 "" H 2200 4100 50  0001 C CNN
-	1    2200 4100
-	1    0    0    -1
-$EndComp
-Wire Wire Line
-	2450 3750 2450 4250
 NoConn ~ 4250 2150
 $Comp
@@
 P 6050 1900
 F 0 "R?" V 5843 1900 50  0000 C CNN
-F 1 "9 Ohm" V 5934 1900 50  0000 C CNN
+F 1 "50 Ohm" V 5934 1900 50  0000 C CNN
 F 2 "" V 5980 1900 50  0001 C CNN
 F 3 "~" H 6050 1900 50  0001 C CNN
@@
 P 6050 1400
 F 0 "R?" V 5843 1400 50  0000 C CNN
-F 1 "9 Ohm" V 5934 1400 50  0000 C CNN
+F 1 "50 Ohm" V 5934 1400 50  0000 C CNN
 F 2 "" V 5980 1400 50  0001 C CNN
 F 3 "~" H 6050 1400 50  0001 C CNN
@@
 P 6050 2900
 F 0 "R?" V 5843 2900 50  0000 C CNN
-F 1 "9 Ohm" V 5934 2900 50  0000 C CNN
+F 1 "50 Ohm" V 5934 2900 50  0000 C CNN
 F 2 "" V 5980 2900 50  0001 C CNN
 F 3 "~" H 6050 2900 50  0001 C CNN
@@
 P 6050 2400
 F 0 "R?" V 5843 2400 50  0000 C CNN
-F 1 "9 Ohm" V 5934 2400 50  0000 C CNN
+F 1 "50 Ohm" V 5934 2400 50  0000 C CNN
 F 2 "" V 5980 2400 50  0001 C CNN
 F 3 "~" H 6050 2400 50  0001 C CNN
@@
 	1450 1800 1450 2450
 Wire Wire Line
-	1450 2450 2650 2450
-Wire Wire Line
 	1300 2350 1300 2250
 Wire Wire Line
-	1300 2350 2650 2350
+	1300 2350 1400 2350
 Wire Wire Line
 	1000 2450 1000 2500
@@
 Wire Wire Line
 	1700 2650 1400 2650
-Wire Wire Line
-	600  2750 2650 2750
 Wire Wire Line
 	650  2850 1350 2850
@@
 Text Notes 800  4250 0    50   ~ 0
 Communicatie Lijn \nvan MAX17320G20+ \nnaar MSP
-Wire Notes Line
-	2350 4200 2550 4200
-Wire Notes Line
-	2550 4200 2550 4350
-Wire Notes Line
-	2350 4350 2350 4200
-Text Notes 2550 4350 0    50   ~ 0
-Always on LDO\n(Eventueel voor externe apparaten)\nNiet geschikt voor uC
 Wire Wire Line
 	4650 4050 6650 4050
-Wire Wire Line
-	6650 4050 6650 4000
 Wire Wire Line
 	1700 1600 1700 750
@@
 Wire Wire Line
 	600  2750 600  6700
+$Comp
+L Device:R R?
+U 1 1 60958FF4
+P 1850 2750
+F 0 "R?" V 1643 2750 50  0000 C CNN
+F 1 "150Ohm" V 1734 2750 50  0000 C CNN
+F 2 "" V 1780 2750 50  0001 C CNN
+F 3 "~" H 1850 2750 50  0001 C CNN
+	1    1850 2750
+	0    1    1    0
+$EndComp
+Wire Wire Line
+	2650 2750 2100 2750
+Wire Wire Line
+	1700 2750 600  2750
+$Comp
+L Device:D_Zener D?
+U 1 1 60962CE8
+P 1950 3150
+F 0 "D?" V 1904 3229 50  0000 L CNN
+F 1 "4.7V Zener" V 1995 3229 50  0000 L CNN
+F 2 "" H 1950 3150 50  0001 C CNN
+F 3 "~" H 1950 3150 50  0001 C CNN
+	1    1950 3150
+	0    1    1    0
+$EndComp
+$Comp
+L power:GND #PWR?
+U 1 1 60962CEE
+P 1950 3300
+F 0 "#PWR?" H 1950 3050 50  0001 C CNN
+F 1 "GND" H 1955 3127 50  0000 C CNN
+F 2 "" H 1950 3300 50  0001 C CNN
+F 3 "" H 1950 3300 50  0001 C CNN
+	1    1950 3300
+	1    0    0    -1
+$EndComp
+Wire Wire Line
+	1950 3000 2100 3000
+Wire Wire Line
+	2100 3000 2100 2750
+Connection ~ 2100 2750
+Wire Wire Line
+	2100 2750 2000 2750
+NoConn ~ 2650 2550
+$Comp
+L Device:R R?
+U 1 1 609750BF
+P 2450 3650
+F 0 "R?" V 2243 3650 50  0000 C CNN
+F 1 "10kOhm" V 2334 3650 50  0000 C CNN
+F 2 "" V 2380 3650 50  0001 C CNN
+F 3 "~" H 2450 3650 50  0001 C CNN
+	1    2450 3650
+	1    0    0    -1
+$EndComp
+Wire Wire Line
+	2450 3250 2450 3500
+Wire Wire Line
+	2450 3800 2450 3900
+$Comp
+L power:GND #PWR?
+U 1 1 6097EC04
+P 2450 3900
+F 0 "#PWR?" H 2450 3650 50  0001 C CNN
+F 1 "GND" H 2455 3727 50  0000 C CNN
+F 2 "" H 2450 3900 50  0001 C CNN
+F 3 "" H 2450 3900 50  0001 C CNN
+	1    2450 3900
+	1    0    0    -1
+$EndComp
+$Comp
+L Device:C C?
+U 1 1 6098BD36
+P 1250 2500
+F 0 "C?" H 1365 2546 50  0000 L CNN
+F 1 "0.1uF" H 1365 2455 50  0000 L CNN
+F 2 "" H 1288 2350 50  0001 C CNN
+F 3 "~" H 1250 2500 50  0001 C CNN
+	1    1250 2500
+	0    -1   -1   0
+$EndComp
+Wire Wire Line
+	1000 2500 1100 2500
+Connection ~ 1000 2500
+Wire Wire Line
+	1400 2500 1400 2350
+$Comp
+L Device:R R?
+U 1 1 6099C999
+P 2400 2350
+F 0 "R?" V 2193 2350 50  0000 C CNN
+F 1 "100 Ohm" V 2284 2350 50  0000 C CNN
+F 2 "" V 2330 2350 50  0001 C CNN
+F 3 "~" H 2400 2350 50  0001 C CNN
+	1    2400 2350
+	0    1    1    0
+$EndComp
+$Comp
+L Device:R R?
+U 1 1 6099FEDF
+P 2000 2450
+F 0 "R?" V 1793 2450 50  0000 C CNN
+F 1 "100 Ohm" V 1884 2450 50  0000 C CNN
+F 2 "" V 1930 2450 50  0001 C CNN
+F 3 "~" H 2000 2450 50  0001 C CNN
+	1    2000 2450
+	0    1    1    0
+$EndComp
+Wire Wire Line
+	1450 2450 1850 2450
+Wire Wire Line
+	2150 2450 2650 2450
+Wire Wire Line
+	2650 2350 2550 2350
+Wire Wire Line
+	2250 2350 1400 2350
+Connection ~ 1400 2350
 $EndSCHEMATC

Commit message: CAN schema toegevoegd voor deel. Faissal en Mounir schema's gecombineerd.
Parts:
- removed IC?: TPS7A2433DBVR, SOT95P280X145-5N, symbol TPS7A2433DBVR:TPS7A2433DBVR
- removed U?: MSP430FR2353TDBT, DBT38_TEX, symbol msp430fr2353tdbt:MSP430FR2353TDBT
- added C1: 10uF, symbol Device:CP
- added C2, C? (x2): 100nF, symbol Device:C
- added C3: 1nF, symbol Device:C
- added C? (x2): C, symbol Device:C
- added IC?: TPS7A2433DBVR, SOT95P280X145-5N, symbol TPS7A2433DBVR:TPS7A2433DBVR
- added J1: Conn_02x07_Odd_Even, symbol Connector_Generic:Conn_02x07_Odd_Even
- added JP1: Jumper_NC_Dual, symbol Device:Jumper_NC_Dual
- added R1: 47k, symbol Device:R
- added U1: MSP430FR2353TDBT, DBT38_TEX, symbol msp430fr2353tdbt:MSP430FR2353TDBT
- added U?: ATA6561-GAQW, SOIC8_4P9X3P9MC_MCH, symbol 2021-05-06_15-34-10:ATA6561-GAQW
- added U?: MCP2515T-I_ST, TSSOP20_MC_MCH, symbol 2021-05-06_16-02-54:MCP2515T-I_ST
- added Y?: Crystal, symbol Device:Crystal
- U1: symbol 2021-04-28_10-27-17:MAX17320G20+ -> PEE50-Schakeling-rescue:MAX17320G20+-2021-04-28_10-27-17
Connections:
- net labels added: +12V
- wire segments 105 -> 188
- no-connect marks 6 -> 15
Other:
- moved on the sheet: C?, D?, J?, Q?, R?

Commit message: .
Parts:
- U?: symbol 2021-05-06_15-34-10:ATA6561-GAQW -> PEE50-Schakeling-rescue:ATA6561-GAQW-2021-05-06_15-34-10
- U?: symbol 2021-05-06_16-02-54:MCP2515T-I_ST -> PEE50-Schakeling-rescue:MCP2515T-I_ST-2021-05-06_16-02-54
Changed lines of the file:
@@
 	600  2700 600  7600
 $Comp
-L 2021-05-06_15-34-10:ATA6561-GAQW U?
+L PEE50-Schakeling-rescue:ATA6561-GAQW-2021-05-06_15-34-10 U?
 U 1 1 609DF1F8
 P 13800 7550
@@
 $EndComp
 $Comp
-L 2021-05-06_16-02-54:MCP2515T-I_ST U?
+L PEE50-Schakeling-rescue:MCP2515T-I_ST-2021-05-06_16-02-54 U?
 U 1 1 609E4D70
 P 10600 7450
