File: PEE50-BatteryProtectionCircuit/PEE50-Schakeling.sch (KiCad schematic (older format))
At the start: 48 parts, among them J1 Conn_02x07_Odd_Even, U1 MAX17320G20+, U1 MSP430FR2353TDBT

Commit message: Schakeling updated met nieuwe transceiver
Parts:
- removed U?: ATA6561-GAQW, SOIC8_4P9X3P9MC_MCH, symbol 2021-05-06_15-34-10:ATA6561-GAQW
- added C? (x2): 0.1uF, symbol Device:C
- added J?: Conn_01x02_Female, symbol Connector:Conn_01x02_Female
- added R?: 10k, symbol Device:R
- added U?: MAX3051ESA, SOIC127P600X175-8N, symbol MAX3051ESA:MAX3051ESA
- C? (x2): value C -> 30p
- Y?: value Crystal -> 8MHz
Connections:
- net labels added: 3.3V
- wire segments 188 -> 211
- no-connect marks 15 -> 16
Changed lines of the file:
@@
 Wire Wire Line
 	600  2700 600  7600
-$Comp
-L 2021-05-06_15-34-10:ATA6561-GAQW U?
-U 1 1 609DF1F8
-P 13800 7550
-F 0 "U?" H 15128 7153 60  0000 L CNN
-F 1 "ATA6561-GAQW" H 15128 7047 60  0000 L CNN
-F 2 "SOIC8_4P9X3P9MC_MCH" H 14600 7890 60  0001 C CNN
-F 3 "" H 13800 7550 60  0000 C CNN
-	1    13800 7550
-	1    0    0    -1
-$EndComp
+Wire Wire Line
+	13250 9600 10400 9600
+Wire Wire Line
+	10400 9600 10400 8250
+Wire Wire Line
+	10600 8650 10500 8650
+$Comp
+L Device:Crystal Y?
+U 1 1 60A08651
+P 12950 6200
+F 0 "Y?" V 12950 6350 50  0000 L CNN
+F 1 "8MHz" V 13100 6250 50  0000 L CNN
+F 2 "" H 12950 6200 50  0001 C CNN
+F 3 "~" H 12950 6200 50  0001 C CNN
+	1    12950 6200
+	0    1    1    0
+$EndComp
+$Comp
+L Device:C C?
+U 1 1 60A094EC
+P 12450 6000
+F 0 "C?" V 12198 6000 50  0000 C CNN
+F 1 "30p" V 12289 6000 50  0000 C CNN
+F 2 "" H 12488 5850 50  0001 C CNN
+F 3 "~" H 12450 6000 50  0001 C CNN
+	1    12450 6000
+	0    1    1    0
+$EndComp
+$Comp
+L Device:C C?
+U 1 1 60A0A27B
+P 12450 6450
+F 0 "C?" V 12198 6450 50  0000 C CNN
+F 1 "30p" V 12289 6450 50  0000 C CNN
+F 2 "" H 12488 6300 50  0001 C CNN
+F 3 "~" H 12450 6450 50  0001 C CNN
+	1    12450 6450
+	0    1    1    0
+$EndComp
+$Comp
+L power:GND #PWR?
+U 1 1 60A0A75F
+P 12100 6550
+F 0 "#PWR?" H 12100 6300 50  0001 C CNN
+F 1 "GND" H 12105 6377 50  0000 C CNN
+F 2 "" H 12100 6550 50  0001 C CNN
+F 3 "" H 12100 6550 50  0001 C CNN
+	1    12100 6550
+	1    0    0    -1
+$EndComp
+Wire Wire Line
+	12300 6000 12100 6000
+Wire Wire Line
+	12600 6000 12950 6000
+Wire Wire Line
+	12950 6000 12950 6050
+Wire Wire Line
+	12100 6550 12100 6450
+Wire Wire Line
+	12100 6450 12300 6450
+Wire Wire Line
+	12100 6450 12100 6000
+Connection ~ 12100 6450
+Wire Wire Line
+	12950 6350 12950 6450
+Wire Wire Line
+	12950 6450 12600 6450
+Wire Wire Line
+	9200 8550 9200 6450
+Wire Wire Line
+	9200 6450 8850 6450
+Wire Wire Line
+	9150 8450 9150 6350
+Wire Wire Line
+	9150 6350 8850 6350
+Wire Wire Line
+	13000 6450 12950 6450
+Connection ~ 12950 6450
+Wire Wire Line
+	13000 7650 13300 7650
+Wire Wire Line
+	13300 7650 13300 6000
+Wire Wire Line
+	13300 6000 12950 6000
+Connection ~ 12950 6000
+$Comp
+L MAX3051ESA:MAX3051ESA U?
+U 1 1 609BD471
+P 14950 8000
+F 0 "U?" H 14950 8970 50  0000 C CNN
+F 1 "MAX3051ESA" H 14950 8879 50  0000 C CNN
+F 2 "SOIC127P600X175-8N" H 14950 8000 50  0001 L BNN
+F 3 "" H 14950 8000 50  0001 L BNN
+	1    14950 8000
+	1    0    0    -1
+$EndComp
+Wire Wire Line
+	9100 8350 9100 6250
+Wire Wire Line
+	9100 6250 8850 6250
+Wire Wire Line
+	9250 7450 9250 6550
+Wire Wire Line
+	9250 6550 8850 6550
+Wire Wire Line
+	8850 6650 9050 6650
+Wire Wire Line
+	9050 6650 9050 7550
+Text GLabel 4500 5450 1    50   Output ~ 0
+3.3V
+Text GLabel 15800 7150 1    50   Input ~ 0
+3.3V
+Text GLabel 10600 8900 1    50   Input ~ 0
+3.3V
+$Comp
+L power:GND #PWR?
+U 1 1 609DDA70
+P 10550 9250
+F 0 "#PWR?" H 10550 9000 50  0001 C CNN
+F 1 "GND" H 10555 9077 50  0000 C CNN
+F 2 "" H 10550 9250 50  0001 C CNN
+F 3 "" H 10550 9250 50  0001 C CNN
+	1    10550 9250
+	1    0    0    -1
+$EndComp
+$Comp
+L power:GND #PWR?
+U 1 1 609DDE93
+P 15750 8750
+F 0 "#PWR?" H 15750 8500 50  0001 C CNN
+F 1 "GND" H 15755 8577 50  0000 C CNN
+F 2 "" H 15750 8750 50  0001 C CNN
+F 3 "" H 15750 8750 50  0001 C CNN
+	1    15750 8750
+	1    0    0    -1
+$EndComp
+Wire Wire Line
+	15650 7300 15800 7300
+Wire Wire Line
+	15800 7300 15800 7150
+Wire Wire Line
+	15750 8750 15750 8700
+Wire Wire Line
+	15750 8700 15650 8700
+Wire Wire Line
+	13650 7500 14250 7500
+Wire Wire Line
+	13450 7700 14250 7700
+Wire Wire Line
+	10500 9450 14250 9450
+Wire Wire Line
+	14250 8500 14250 9450
+Wire Wire Line
+	13450 6800 13450 7700
+$Comp
+L Connector:Conn_01x02_Female J?
+U 1 1 60A3068A
+P 15100 6800
+F 0 "J?" H 15128 6776 50  0000 L CNN
+F 1 "Conn_01x02_Female" H 15128 6685 50  0000 L CNN
+F 2 "" H 15100 6800 50  0001 C CNN
+F 3 "~" H 15100 6800 50  0001 C CNN
+	1    15100 6800
+	1    0    0    -1
+$EndComp
+Wire Wire Line
+	13450 6800 14900 6800
+Wire Wire Line
+	14900 6900 13650 6900
+Wire Wire Line
+	13650 6900 13650 7500
+Wire Wire Line
+	14250 8100 13250 8100
+Wire Wire Line
+	13250 8100 13250 9600
+$Comp
+L power:GND #PWR?
+U 1 1 60A519AC
+P 14150 7900
+F 0 "#PWR?" H 14150 7650 50  0001 C CNN
+F 1 "GND" H 14155 7727 50  0000 C CNN
+F 2 "" H 14150 7900 50  0001 C CNN
+F 3 "" H 14150 7900 50  0001 C CNN
+	1    14150 7900
+	1    0    0    -1
+$EndComp
+Wire Wire Line
+	14150 7900 14250 7900
+NoConn ~ 14250 8300
+$Comp
+L Device:C C?
+U 1 1 60A7182B
+P 15800 7650
+F 0 "C?" H 16000 7550 50  0000 C CNN
+F 1 "0.1uF" H 16000 7650 50  0000 C CNN
+F 2 "" H 15838 7500 50  0001 C CNN
+F 3 "~" H 15800 7650 50  0001 C CNN
+	1    15800 7650
+	-1   0    0    1
+$EndComp
+Wire Wire Line
+	15800 7300 15800 7500
+Connection ~ 15800 7300
+Wire Wire Line
+	15800 7800 15800 8700
+Wire Wire Line
+	15800 8700 15750 8700
+Connection ~ 15750 8700
+Wire Wire Line
+	10600 8900 10600 8950
+Wire Wire Line
+	10600 9150 10550 9150
+Wire Wire Line
+	10550 9150 10550 9250
+$Comp
+L Device:R R?
+U 1 1 60A9E176
+P 10250 7800
+F 0 "R?" H 10320 7846 50  0000 L CNN
+F 1 "10k" H 10320 7755 50  0000 L CNN
+F 2 "" V 10180 7800 50  0001 C CNN
+F 3 "~" H 10250 7800 50  0001 C CNN
+	1    10250 7800
+	1    0    0    -1
+$EndComp
+Wire Wire Line
+	10250 8950 10250 7950
+$Comp
+L Device:C C?
+U 1 1 60ABFED0
+P 10250 9100
+F 0 "C?" H 10450 9000 50  0000 C CNN
+F 1 "0.1uF" H 10450 9100 50  0000 C CNN
+F 2 "" H 10288 8950 50  0001 C CNN
+F 3 "~" H 10250 9100 50  0001 C CNN
+	1    10250 9100
+	-1   0    0    1
+$EndComp
+Connection ~ 10250 8950
+Wire Wire Line
+	10250 9250 10550 9250
+Connection ~ 10550 9250
+Connection ~ 10600 8950
+Connection ~ 13000 7350
+Wire Wire Line
+	13000 7350 13000 6450
+Wire Wire Line
+	13000 7550 13000 7350
+Wire Wire Line
+	10600 8950 10250 8950
+Wire Wire Line
+	10600 8550 9200 8550
+Wire Wire Line
+	10600 8450 9150 8450
+Wire Wire Line
+	10600 8350 9100 8350
+Wire Wire Line
+	10400 8250 10600 8250
+Wire Wire Line
+	10250 7650 10600 7650
+Wire Wire Line
+	9050 7550 10600 7550
+Wire Wire Line
+	10600 7450 9250 7450
+Wire Wire Line
+	10500 8650 10500 9450
 $Comp
 L 2021-05-06_16-02-54:MCP2515T-I_ST U?
@@
 	1    0    0    -1
 $EndComp
-Wire Wire Line
-	13800 7750 13250 7750
-Wire Wire Line
-	13250 7750 13250 9600
-Wire Wire Line
-	13250 9600 10400 9600
-Wire Wire Line
-	10400 9600 10400 8250
-Wire Wire Line
-	10400 8250 10600 8250
-Wire Wire Line
-	10600 8650 10500 8650
-Wire Wire Line
-	10500 8650 10500 9450
-Wire Wire Line
-	10500 9450 13550 9450
-Wire Wire Line
-	13550 9450 13550 7950
-Wire Wire Line
-	13550 7950 13800 7950
-Wire Wire Line
-	13800 7550 13650 7550
-Wire Wire Line
-	13650 7550 13650 6950
-Wire Wire Line
-	13650 6950 14750 6950
-Wire Wire Line
-	13800 7650 13450 7650
-Wire Wire Line
-	13450 7650 13450 6800
-Wire Wire Line
-	13450 6800 14750 6800
-$Comp
-L Device:Crystal Y?
-U 1 1 60A08651
-P 12950 6200
-F 0 "Y?" V 12950 6350 50  0000 L CNN
-F 1 "Crystal" V 13100 6250 50  0000 L CNN
-F 2 "" H 12950 6200 50  0001 C CNN
-F 3 "~" H 12950 6200 50  0001 C CNN
-	1    12950 6200
-	0    1    1    0
-$EndComp
-$Comp
-L Device:C C?
-U 1 1 60A094EC
-P 12450 6000
-F 0 "C?" V 12198 6000 50  0000 C CNN
-F 1 "C" V 12289 6000 50  0000 C CNN
-F 2 "" H 12488 5850 50  0001 C CNN
-F 3 "~" H 12450 6000 50  0001 C CNN
-	1    12450 6000
-	0    1    1    0
-$EndComp
-$Comp
-L Device:C C?
-U 1 1 60A0A27B
-P 12450 6450
-F 0 "C?" V 12198 6450 50  0000 C CNN
-F 1 "C" V 12289 6450 50  0000 C CNN
-F 2 "" H 12488 6300 50  0001 C CNN
-F 3 "~" H 12450 6450 50  0001 C CNN
-	1    12450 6450
-	0    1    1    0
-$EndComp
-$Comp
-L power:GND #PWR?
-U 1 1 60A0A75F
-P 12100 6550
-F 0 "#PWR?" H 12100 6300 50  0001 C CNN
-F 1 "GND" H 12105 6377 50  0000 C CNN
-F 2 "" H 12100 6550 50  0001 C CNN
-F 3 "" H 12100 6550 50  0001 C CNN
-	1    12100 6550
-	1    0    0    -1
-$EndComp
-Wire Wire Line
-	12300 6000 12100 6000
-Wire Wire Line
-	12600 6000 12950 6000
-Wire Wire Line
-	12950 6000 12950 6050
-Wire Wire Line
-	12100 6550 12100 6450
-Wire Wire Line
-	12100 6450 12300 6450
-Wire Wire Line
-	12100 6450 12100 6000
-Connection ~ 12100 6450
-Wire Wire Line
-	12950 6350 12950 6450
-Wire Wire Line
-	12950 6450 12600 6450
-Wire Wire Line
-	10600 8550 9200 8550
-Wire Wire Line
-	9200 8550 9200 6450
-Wire Wire Line
-	9200 6450 8850 6450
-Wire Wire Line
-	10600 8450 9150 8450
-Wire Wire Line
-	9150 8450 9150 6350
-Wire Wire Line
-	9150 6350 8850 6350
-Wire Wire Line
-	13000 7550 13000 7350
-Wire Wire Line
-	13000 6450 12950 6450
-Connection ~ 13000 7350
-Wire Wire Line
-	13000 7350 13000 6450
-Connection ~ 12950 6450
-Wire Wire Line
-	13000 7650 13300 7650
-Wire Wire Line
-	13300 7650 13300 6000
-Wire Wire Line
-	13300 6000 12950 6000
-Connection ~ 12950 6000
 $EndSCHEMATC
