File: PEE50-BatteryProtectionCircuit/PEE50-Schakeling.sch (KiCad schematic (older format))
At the start: 52 parts, among them J1 Conn_02x07_Odd_Even, U1 MAX17320G20+, U1 MSP430FR2353TDBT

Commit message: Pinout FETs verwisseld
Parts:
- U?: symbol MAX3051ESA:MAX3051ESA -> PEE50-Schakeling-rescue:MAX3051ESA-MAX3051ESA
- U?: symbol 2021-05-06_16-02-54:MCP2515T-I_ST -> PEE50-Schakeling-rescue:MCP2515T-I_ST-2021-05-06_16-02-54
Changed lines of the file:
@@
 	10500 8650 10500 9450
 $Comp
-L 2021-05-06_16-02-54:MCP2515T-I_ST U?
+L PEE50-Schakeling-rescue:MCP2515T-I_ST-2021-05-06_16-02-54 U?
 U 1 1 609E4D70
 P 10600 7450
@@
 $EndComp
 $Comp
-L MAX3051ESA:MAX3051ESA U?
+L PEE50-Schakeling-rescue:MAX3051ESA-MAX3051ESA U?
 U 1 1 609BD471
 P 14950 8000

Commit message: Een aantal footprints gekozen
Parts:
- removed J1: Conn_02x07_Odd_Even, symbol Connector_Generic:Conn_02x07_Odd_Even
- removed U?: MCP2515T-I_ST, TSSOP20_MC_MCH, symbol PEE50-Schakeling-rescue:MCP2515T-I_ST-2021-05-06_16-02-54
- added J5: Conn_02x03_Odd_Even, Connector_PinHeader_2.54mm:PinHeader_2x03_P2.54mm_Vertical, symbol Connector_Generic:Conn_02x03_Odd_Even
- added U3, U4: MCP2515T-I_ST, symbol PEE50-Schakeling-rescue:MCP2515T-I_ST-2021-05-06_16-02-54
- C1, C10, C11, C15, C16, C17, C18, C2, C3, C4, C5, C6, C7, C8, C9: renamed from C?; footprint (none) -> Capacitor_SMD:C_0603_1608Metric
- C12: renamed from C2; footprint (none) -> Capacitor_SMD:C_0603_1608Metric
- C13: renamed from C1; footprint (none) -> Capacitor_SMD:C_0603_1608Metric
- C14: renamed from C3; footprint (none) -> Capacitor_SMD:C_0603_1608Metric
- D1, D2, D3: renamed from D?; footprint (none) -> Diode_SMD:D_0603_1608Metric_Castellated
- IC1: renamed from IC?; footprint SOT95P280X145-5N -> Package_TO_SOT_SMD:SOT-23-5
- J1, J2, J3, J4, J6: renamed from J?; footprint (none) -> Connector_Phoenix_MSTB:PhoenixContact_MSTBA_2,5_2-G-5,08_1x02_P5.08mm_Horizontal
- Q1, Q2: renamed from Q?; footprint (none) -> Package_TO_SOT_SMD:TO-263-2; symbol Device:Q_NMOS_DGS -> PEE50-Schakeling-rescue:Q_NMOS_DGS-Device
- U2: renamed from U1; footprint DBT38_TEX -> (none)
- U5: renamed from U?; footprint SOIC127P600X175-8N -> (none)
- gave numbers to parts that had none: 16
- renumbered R1 to R11
Connections:
- wire segments 211 -> 209
- no-connect marks 16 -> 8

Commit message: PCB V1.0 finish
Parts:
- removed U4: MCP2515T-I_ST, symbol PEE50-Schakeling-rescue:MCP2515T-I_ST-2021-05-06_16-02-54
- added BT1: BH1000G, CAN_control:BAT_BH1000G, symbol BH1000G:BH1000G
- added D4, D5: D_Schottky, Diode_SMD:D_0603_1608Metric, symbol Device:D_Schottky
- added J7: Conn_01x02_Male, Connector_Phoenix_MSTB:PhoenixContact_MSTBA_2,5_2-G-5,08_1x02_P5.08mm_Horizontal, symbol Connector:Conn_01x02_Male
- added R17: 120, Resistor_SMD:R_0603_1608Metric, symbol Device:R
- IC1: footprint Package_TO_SOT_SMD:SOT-23-5 -> CAN_control:SOT95P280X145-5N
- J6: footprint Connector_Phoenix_MSTB:PhoenixContact_MSTBA_2,5_2-G-5,08_1x02_P5.08mm_Horizontal -> Connector_Molex:Molex_Mini-Fit_Jr_5566-04A2_2x02_P4.20mm_Vertical
- JP1: footprint (none) -> Connector_PinHeader_2.54mm:PinHeader_1x03_P2.54mm_Vertical
- Q1, Q2: footprint Package_TO_SOT_SMD:TO-263-2 -> Package_SON:VSONP-8-1EP_5x6_P1.27mm; symbol PEE50-Schakeling-rescue:Q_NMOS_DGS-Device -> PEE50-Schakeling-rescue:Q_NMOS_DGS-Device-PEE50-Schakeling-rescue
- R1, R10, R11, R12, R13, R14, R15, R16, R2, R3, R4, R5, R6, R7, R8, R9: footprint (none) -> Resistor_SMD:R_0603_1608Metric
- U1: footprint MAXim:MAX17320G20&plus_ -> CAN_control:MAX17320G20&plus_
- U2: footprint (none) -> CAN_control:MSP430FR2353TDBT
- U3: footprint (none) -> CAN_control:MCP2515T-I&slash_ST
- U5: footprint (none) -> CAN_control:SOIC127P600X175-8N
- Y1: footprint (none) -> Crystal:Crystal_HC49-4H_Vertical
Connections:
- net +12V: now also D5.2 (A); no longer C4.2, IC1.1 (IN), IC1.3 (EN)
- net GND: now also BT1.N
- net NegativeTerminal: now also J7.1 (Pin_1)
- net PositiveTerminal: now also Q1.1 (S), J7.2 (Pin_2); no longer Q1.3 (S)
- net at C1.1, J1.2 (Pin_2), R12.1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: now also Q2.1 (S); no longer Q2.3 (S)
- net at R5.2: now also Q1.2 (G); no longer Q1.1 (G)
- net at Q2.2 (G): now also C1.2, R8.2; no longer Q1.2 (D)
- net +3V3: now reaches C12.1, C13.1, JP1.2, R11.1, U2.10 (DVCC)
- net +3V3: now also C15.2, C18.2, C5.2, IC1.5 (OUT), R16.2, U3.20 (VDD), U5.3 (VCC)
- net at U2.15 (P2-4/COMP1-1): now also U3.7 (*TX2RTS)
- net at U2.24 (P2-3/TB1TRG): now also U3.5 (*TX1RTS)
- net at U2.25 (P2-2/TB1CLK): now also U3.4 (*TX0RTS)
- net at U2.26 (P2-1/TB1-2/COMP1-O): now also U3.11 (*RX1BF)
- net at U2.27 (P2-0/TB1-1/COMP0-O): now also U3.12 (*RX0BF)
- net at U2.29 (P1-6/UCA0RXD/UCA0SOMI/TB0-1/TDI/TCLK/OA1-/A6): now also R16.1, U3.19 (*RESET)
- net at J6.1 (Pin_1), U5.6 (CANL): now also R17.2
- net at J6.2 (Pin_2), U5.7 (CANH): now also R17.1
- removed net 3.3V: C15.2, C18.2, C5.2, IC1.5 (OUT), J5.4 (Pin_4), JP1.1, R16.2, U3.20 (VDD), U5.3 (VCC)
- new net: Q1.3 (D), Q2.3 (D)
- new net: C4.2, D4.1 (K), D5.1 (K), IC1.1 (IN), IC1.3 (EN)
- new net: BT1.P, D4.2 (A)
- new net Ext3.3V: J5.4 (Pin_4), JP1.1
- no-connect marks 8 -> 10
Other:
- note added: "External 3.3V"
- note added: "JTAG connector"
- note added: "Reset"
- note added: "Test"
- note added: "Vin"

Commit message: Connector voor 12V toegevoegd aan PCB en schema
Parts:
- added J8: Conn_01x02_Male, Connector_Phoenix_MSTB:PhoenixContact_MSTBA_2,5_2-G-5,08_1x02_P5.08mm_Horizontal, symbol Connector:Conn_01x02_Male
Connections:
- net GND: now also J8.2 (Pin_2)
- net +12V: no longer names the net of D5.2 (A)
- net +12V: now also J8.1 (Pin_1)
Changed lines of the file:
@@
 	10650 6100 10850 6100
-$Comp
-L power:+12V #PWR05
-U 1 1 6093D50F
-P 2300 5050
-F 0 "#PWR05" H 2300 4900 50  0001 C CNN
-F 1 "+12V" H 2315 5223 50  0000 C CNN
-F 2 "" H 2300 5050 50  0001 C CNN
-F 3 "" H 2300 5050 50  0001 C CNN
-	1    2300 5050
-	1    0    0    -1
-$EndComp
 $Comp
 L Device:CP C13
@@
 	9250 7500 8850 7500
 $Comp
-L power:+3.3V #PWR?
+L power:+3.3V #PWR0101
 U 1 1 60D3825E
 P 10600 8900
-F 0 "#PWR?" H 10600 8750 50  0001 C CNN
+F 0 "#PWR0101" H 10600 8750 50  0001 C CNN
 F 1 "+3.3V" H 10615 9073 50  0000 C CNN
 F 2 "" H 10600 8900 50  0001 C CNN
@@
 	1    0    0    -1
 $EndComp
+$Comp
+L Connector:Conn_01x02_Male J8
+U 1 1 60A7424D
+P 2300 4850
+F 0 "J8" V 2300 5000 50  0000 R CNN
+F 1 "Conn_01x02_Male" V 2400 5550 50  0000 R CNN
+F 2 "Connector_Phoenix_MSTB:PhoenixContact_MSTBA_2,5_2-G-5,08_1x02_P5.08mm_Horizontal" H 2300 4850 50  0001 C CNN
+F 3 "~" H 2300 4850 50  0001 C CNN
+	1    2300 4850
+	0    1    1    0
+$EndComp
+$Comp
+L power:GND #PWR05
+U 1 1 60A753A1
+P 2050 5200
+F 0 "#PWR05" H 2050 4950 50  0001 C CNN
+F 1 "GND" H 2055 5027 50  0000 C CNN
+F 2 "" H 2050 5200 50  0001 C CNN
+F 3 "" H 2050 5200 50  0001 C CNN
+	1    2050 5200
+	1    0    0    -1
+$EndComp
+Wire Wire Line
+	2050 5200 2050 5050
+Wire Wire Line
+	2050 5050 2200 5050
 $EndSCHEMATC

Commit message: 2de coincell batterij holder toegevoegd.
Parts:
- added BT2: BH1000G, CAN_control:BAT_BH1000G, symbol BH1000G:BH1000G
Connections:
- net GND: now also BT2.N; no longer BT1.N
- new net: BT1.N, BT2.P
Changed lines of the file:
@@
 Connection ~ 2300 5550
 Wire Wire Line
-	3000 5950 4150 5950
+	3000 5950 3200 5950
 Wire Wire Line
 	1800 6300 1800 6600
@@
 Wire Wire Line
 	1800 6600 1850 6600
-Wire Wire Line
-	2450 6600 2450 5950
-Wire Wire Line
-	2450 5950 3000 5950
 Text GLabel 11350 6200 2    50   Output ~ 0
 Ext3.3V
@@
 Wire Wire Line
 	2050 5050 2200 5050
+$Comp
+L BH1000G:BH1000G BT2
+U 1 1 60A95410
+P 2850 6600
+F 0 "BT2" H 2850 6867 50  0000 C CNN
+F 1 "BH1000G" H 2850 6776 50  0000 C CNN
+F 2 "CAN_control:BAT_BH1000G" H 2850 6600 50  0001 L BNN
+F 3 "" H 2850 6600 50  0001 L BNN
+F 4 "Manufacturer Recommendations" H 2850 6600 50  0001 L BNN "STANDARD"
+F 5 "E" H 2850 6600 50  0001 L BNN "PARTREV"
+F 6 "MPD" H 2850 6600 50  0001 L BNN "MANUFACTURER"
+F 7 "12.6mm" H 2850 6600 50  0001 L BNN "MAXIMUM_PACKAGE_HEIGHT"
+	1    2850 6600
+	1    0    0    -1
+$EndComp
+Wire Wire Line
+	2450 6600 2550 6600
+Wire Wire Line
+	3150 6600 3200 6600
+Wire Wire Line
+	3200 6600 3200 5950
+Connection ~ 3200 5950
+Wire Wire Line
+	3200 5950 4150 5950
 $EndSCHEMATC
