File: CurrentProtectionTemplate/PEE50-CurrentProtectionTemplate.kicad_pcb (KiCad board)
At the start: 2 copper layers, 100 x 100 mm, 37 parts, among them J1 CAN_IN, J2 CAN_OUT, J3 4-Wire_JTAG_Programming, J4 CAN_IN, J5 CAN_OUT, Q1 IRLML6346TRPBF, SW1 SW_Push, U1 TPS7A2433DBVR, U2 MSP430FR2353TDBT, U3 MAX44284EAUT+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

Commit message: Routed everything
Parts:
- removed the J5 at (58.5, 62.6)
- removed the TP2 at (73.5, 74.0)
- removed the TP4 at (78.1, 73.6)
- added C14: 22nF, Capacitor_SMD:C_1206_3216Metric, F.Cu at (56.9, 32.6)
- added J2: CAN_IN, Connector_PinHeader_2.54mm:PinHeader_1x04_P2.54mm_Vertical, F.Cu at (16.9, 37.5)
- added R4: 1.8k, Resistor_SMD:R_1206_3216Metric, F.Cu at (56.9, 30.2)
- added TP1: SPI_SlaveIn, TestPoint:TestPoint_Loop_D1.80mm_Drill1.0mm_Beaded, F.Cu at (57.0, 46.2)
- added TP3: SPI_ChipSel, TestPoint:TestPoint_Loop_D1.80mm_Drill1.0mm_Beaded, F.Cu at (49.6, 46.1)
- C1: value 1uF -> 100nF
- C10: value 18pF -> 4.7uF
- C2: value 100nF -> 1uF
- C7: value 100nF -> 18pF
- C8: value 18pF -> 100nF
- C9: value 4.7uF -> 18pF
- J4: value CAN_IN -> CAN_OUT
- Q1: moved to B.Cu
- Y2: footprint Crystal:Crystal_SMD_HC49-SD_HandSoldering -> Crystal:Crystal_SMD_HC49-SD
- moved R3 70.0 mm to (16.4, 25.0), turned to 270 degrees
- moved TP7 64.1 mm to (27.1, 31.1)
- moved J5 62.2 mm to (19.1, 60.4), turned to 180 degrees
- moved C10 58.8 mm to (69.7, 26.0), turned to 90 degrees
- moved TP6 58.6 mm to (34.8, 27.6)
- moved C13 55.3 mm to (31.3, 30.1), turned to 180 degrees
- moved C2 55.2 mm to (48.8, 27.1), turned to 90 degrees
- moved C4 54.0 mm to (52.3, 24.5)
- moved C7 52.1 mm to (25.3, 43.1), turned to 90 degrees
- moved C8 51.9 mm to (66.6, 22.5), turned to 180 degrees
- moved U5 51.3 mm to (31.2, 26.4), turned to 90 degrees
- moved C9 49.9 mm to (25.3, 36.6), turned to 90 degrees
- moved TP5 49.4 mm to (35.7, 45.3)
- moved R1 49.4 mm to (22.2, 54.5), turned to 270 degrees
- moved J4 49.1 mm to (20.9, 37.5), turned to 180 degrees
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- renumbered J2 to J3, J3 to J5, TP3 to TP2, TP5 to TP4, TP1 to TP5
Connections:
- net /CANH renamed /Beveiliging/CANH
- net /CANL renamed /Beveiliging/CANL
- net /RS_STBY_CAN renamed /Beveiliging/RS_STBY_CAN
- net /RXD renamed /Beveiliging/RXD
- net /SBWTCK renamed /Beveiliging/SBWTCK
- net /SBWTDIO renamed /Beveiliging/SBWTDIO
- net /SHDN_CAN renamed /Beveiliging/SHDN_CAN
- net /SlaveIn renamed /Beveiliging/SlaveIn
- net /SlaveOut renamed /Beveiliging/SlaveOut
- net /SysClk renamed /Beveiliging/SysClk
- net /TXD renamed /Beveiliging/TXD
- net /XIN renamed /Beveiliging/XIN
- net /XOUT renamed /Beveiliging/XOUT
- net /~ChipSel renamed /Beveiliging/~ChipSel
- net /~ENABLE renamed /Beveiliging/~ENABLE
- net /~INT renamed /Beveiliging/~INT
- net /~RST_CAN renamed /Beveiliging/~RST_CAN
- net /~RX0INT renamed /Beveiliging/~RX0INT
- net /~RX1INT renamed /Beveiliging/~RX1INT
- net /~TX0RTS renamed /Beveiliging/~TX0RTS
- net /~TX1RTS renamed /Beveiliging/~TX1RTS
- net /~TX2RTS renamed /Beveiliging/~TX2RTS
- C1 pad 1: +12V -> GNDPWR
- C1 pad 2: GNDPWR -> +3V3
- C10 pad 1: /OSC2 -> +3V3
- C11 pad 1: +3V3 -> GNDPWR
- C11 pad 2: GNDPWR -> +3V3
- C12 pad 1: +3V3 -> GNDPWR
- C12 pad 2: GNDPWR -> +3V3
- C2 pad 1: +3V3 -> GNDPWR
- C2 pad 2: GNDPWR -> +12V
- C4 pad 1: +3V3 -> GNDPWR
- C4 pad 2: GNDPWR -> +3V3
- C7 pad 1: +3V3 -> /Beveiliging/OSC1
- C8 pad 1: /OSC1 -> +3V3
- C9 pad 1: +3V3 -> GNDPWR
- C9 pad 2: GNDPWR -> /Beveiliging/OSC2
- J5 pad 6: (no net) -> Net-(J5-Pad6)
- Q1 pad 3: (no net) -> GND
- R2 pad 4: (no net) -> +12P
- U1 pad 4: (no net) -> Net-(U1-Pad4)
- U2 pad 1: (no net) -> Net-(U2-Pad1)
- U2 pad 14: (no net) -> Net-(U2-Pad14)
- U2 pad 15: (no net) -> Net-(U2-Pad15)
- U2 pad 2: (no net) -> Net-(U2-Pad2)
- U2 pad 22: (no net) -> Net-(U2-Pad22)
- U2 pad 23: (no net) -> Net-(U2-Pad23)
- U2 pad 27: (no net) -> Net-(U2-Pad27)
- U2 pad 32: (no net) -> Net-(U2-Pad32)
- U2 pad 33: (no net) -> Net-(U2-Pad33)
- U2 pad 34: (no net) -> Net-(U2-Pad34)
- U2 pad 35: (no net) -> Net-(U2-Pad35)
- U2 pad 38: (no net) -> Net-(U2-Pad38)
- U2 pad 4: (no net) -> Net-(U2-Pad4)
- U2 pad 5: (no net) -> Net-(U2-Pad5)
- U2 pad 6: (no net) -> Net-(U2-Pad6)
- U2 pad 7: /Vcurrent -> /Beveiliging/Vcurrent
- U3 pad 5: /Vcurrent -> Net-(R4-Pad2)
- U4 pad 7: /OSC2 -> /Beveiliging/OSC2
- U4 pad 8: /OSC1 -> /Beveiliging/OSC1
- Y2 pad 1: /OSC1 -> /Beveiliging/OSC1
- Y2 pad 2: /OSC2 -> /Beveiliging/OSC2
Routing:
- net /Beveiliging/SBWTDIO: track 0.00 -> 71.4 mm
- net GNDPWR: track 0.00 -> 69.5 mm, vias 0 -> 14
- net /Beveiliging/RXD: track 0.00 -> 67.6 mm
- net +3V3: track 0.00 -> 66.9 mm, vias 0 -> 2
- net /Beveiliging/TXD: track 0.00 -> 62.9 mm
- net /Beveiliging/SBWTCK: track 0.00 -> 57.6 mm
- net /Beveiliging/~ENABLE: track 0.00 -> 54.2 mm, vias 0 -> 1
- net /Beveiliging/CANH: track 0.00 -> 53.2 mm
- net /Beveiliging/CANL: track 0.00 -> 50.5 mm
- net /Beveiliging/RS_STBY_CAN: track 0.00 -> 31.9 mm, vias 0 -> 2
- net +12V: track 0.00 -> 29.1 mm
- net /Beveiliging/SHDN_CAN: track 0.00 -> 28.6 mm, vias 0 -> 2
- net /Beveiliging/SlaveOut: track 0.00 -> 25.6 mm, vias 0 -> 1
- net /Beveiliging/~RST_CAN: track 0.00 -> 25.1 mm, vias 0 -> 4
- net /Beveiliging/~TX2RTS: track 0.00 -> 24.3 mm, vias 0 -> 2
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- added copper zone on F.Cu, net +12P
- added copper zone on F.Cu, net +12V
- added copper zone on F.Cu, net +3V3
- added copper zone on B.Cu, net GND
- added copper zone on B.Cu, net GNDPWR
Other:
- rule trace_min: 0.2 -> 0.127
- rule via_min_drill: 0.3 -> 0.2
- board text added: "GND 5V 3V3 >>RXD <<TXD SBWTDIO SBWTCK"

Commit message: Ready for order
Routing:
- net /Beveiliging/~RX0INT: track 18.9 -> 26.1 mm
- net /Beveiliging/~RX1INT: track 19.0 -> 25.6 mm
- net /Beveiliging/~INT: track 23.0 -> 28.8 mm

Commit message: PCB as ordered
Parts:
- J5: value 4-Wire_JTAG_Programming -> Launchpad_Programming
- Q1: value IRLML6346TRPBF -> RFD14N05L; footprint footprints:IRLML6346TRPBF -> Package_TO_SOT_THT:TO-251-3-1EP_Horizontal_TabDown; moved to F.Cu
- moved Q1 23.8 mm to (77.0, 17.4), turned to 180 degrees
Connections:
- Q1 pad 2: GNDPWR -> GND
- Q1 pad 3: GND -> GNDPWR
Routing:
- net /Beveiliging/CANL: track 50.5 -> 79.1 mm
- net /Beveiliging/CANH: track 53.2 -> 77.6 mm
- net /Beveiliging/~ENABLE: track 54.2 -> 46.7 mm
- net GND: track 0.00 -> 7.43 mm
- net /Beveiliging/SBWTCK: track 57.6 -> 53.7 mm
- net /Beveiliging/SBWTDIO: track 71.4 -> 67.6 mm
- net /Beveiliging/RS_STBY_CAN: track 31.9 -> 32.5 mm
- net /Beveiliging/SHDN_CAN: track 28.6 -> 29.1 mm
